File: CAN.sch (KiCad schematic (older format))
At the start: 12 parts

Commit message: ready for first rev
Changed lines of the file:
@@
 $Descr A4 11693 8268
 encoding utf-8
-Sheet 6 8
+Sheet 5 8
 Title ""
 Date ""
@@
 Text HLabel 2350 3850 0    60   BiDi ~ 0
 MS_CAN_LO
-Text HLabel 5450 2700 0    60   BiDi ~ 0
+Text HLabel 5950 3100 2    60   BiDi ~ 0
 SW_CAN
 Text HLabel 4700 1950 2    60   Output ~ 0
@@
 	1700 2850 2000 2850
 Wire Wire Line
-	3350 2550 3400 2550
-Wire Wire Line
-	3400 2550 3450 2550
+	3350 2550 3450 2550
 Wire Wire Line
 	3400 2650 3400 2550
 Connection ~ 3400 2550
 Wire Wire Line
-	3400 3200 3400 3250
-Wire Wire Line
-	3400 3250 3400 3350
-Wire Wire Line
-	3350 1600 3350 1650
-Wire Wire Line
-	3350 1650 3350 1750
-Wire Wire Line
-	3400 4150 3450 4150
-Wire Wire Line
-	3450 4150 3500 4150
+	3400 3200 3400 3350
+Wire Wire Line
+	3350 1600 3350 1750
+Wire Wire Line
+	3400 4150 3500 4150
 Wire Wire Line
 	3450 4250 3450 4150
@@
 	2350 3850 2900 3850
 Wire Wire Line
-	3850 1950 4400 1950
-Wire Wire Line
-	4400 1950 4700 1950
-Wire Wire Line
-	3850 2050 4600 2050
-Wire Wire Line
-	4600 2050 4700 2050
-Wire Wire Line
-	3900 3550 4400 3550
-Wire Wire Line
-	4400 3550 4750 3550
-Wire Wire Line
-	3900 3650 4600 3650
-Wire Wire Line
-	4600 3650 4750 3650
+	3850 1950 4700 1950
+Wire Wire Line
+	3850 2050 4700 2050
+Wire Wire Line
+	3900 3550 4750 3550
+Wire Wire Line
+	3900 3650 4750 3650
 $Comp
 L +3.3V #PWR?
@@
 	4400 4600 4400 4700
 Wire Wire Line
-	4400 4700 4500 4700
-Wire Wire Line
-	4500 4700 4600 4700
+	4400 4700 4600 4700
 Wire Wire Line
 	4600 4700 4600 4600
@@
 	4400 2900 4400 3000
 Wire Wire Line
-	4400 3000 4500 3000
-Wire Wire Line
-	4500 3000 4600 3000
+	4400 3000 4600 3000
 Wire Wire Line
 	4600 3000 4600 2900

Commit message: fixed some ports errors
Parts:
- gave numbers to parts that had none: 12
Changed lines of the file:
@@
 SW_CAN_LOAD
 $Comp
-L MCP2562-E/MF U?
+L MCP2562-E/MF U2
 U 1 1 5AFD0533
 P 3350 2150
-F 0 "U?" H 2950 2500 50  0000 L CNN
+F 0 "U2" H 2950 2500 50  0000 L CNN
 F 1 "MCP2562-E/MF" H 3450 2500 50  0000 L CNN
 F 2 "Housings_DFN_QFN:DFN-8-1EP_3x3mm_Pitch0.65mm" H 3350 1650 50  0001 C CIN
@@
 $EndComp
 $Comp
-L MCP2562-E/MF U?
+L MCP2562-E/MF U3
 U 1 1 5AFD05D8
 P 3400 3750
-F 0 "U?" H 3000 4100 50  0000 L CNN
+F 0 "U3" H 3000 4100 50  0000 L CNN
 F 1 "MCP2562-E/MF" H 3500 4100 50  0000 L CNN
 F 2 "Housings_DFN_QFN:DFN-8-1EP_3x3mm_Pitch0.65mm" H 3400 3250 50  0001 C CIN
@@
 3.3V
 $Comp
-L +5V #PWR?
+L +5V #PWR056
 U 1 1 5AFD0678
 P 1800 2700
-F 0 "#PWR?" H 1800 2550 50  0001 C CNN
+F 0 "#PWR056" H 1800 2550 50  0001 C CNN
 F 1 "+5V" H 1800 2840 50  0000 C CNN
 F 2 "" H 1800 2700 50  0001 C CNN
@@
 $EndComp
 $Comp
-L +3.3V #PWR?
+L +3.3V #PWR057
 U 1 1 5AFD0692
 P 2000 2850
-F 0 "#PWR?" H 2000 2700 50  0001 C CNN
+F 0 "#PWR057" H 2000 2700 50  0001 C CNN
 F 1 "+3.3V" H 2000 2990 50  0000 C CNN
 F 2 "" H 2000 2850 50  0001 C CNN
@@
 $EndComp
 $Comp
-L GND #PWR?
+L GND #PWR058
 U 1 1 5AFD06C6
 P 3400 2650
-F 0 "#PWR?" H 3400 2400 50  0001 C CNN
+F 0 "#PWR058" H 3400 2400 50  0001 C CNN
 F 1 "GND" H 3400 2500 50  0000 C CNN
 F 2 "" H 3400 2650 50  0001 C CNN
@@
 $EndComp
 $Comp
-L GND #PWR?
+L GND #PWR059
 U 1 1 5AFD06DE
 P 3450 4250
-F 0 "#PWR?" H 3450 4000 50  0001 C CNN
+F 0 "#PWR059" H 3450 4000 50  0001 C CNN
 F 1 "GND" H 3450 4100 50  0000 C CNN
 F 2 "" H 3450 4250 50  0001 C CNN
@@
 $EndComp
 $Comp
-L +5V #PWR?
+L +5V #PWR060
 U 1 1 5AFD0701
 P 3350 1600
-F 0 "#PWR?" H 3350 1450 50  0001 C CNN
+F 0 "#PWR060" H 3350 1450 50  0001 C CNN
 F 1 "+5V" H 3350 1740 50  0000 C CNN
 F 2 "" H 3350 1600 50  0001 C CNN
@@
 $EndComp
 $Comp
-L +5V #PWR?
+L +5V #PWR061
 U 1 1 5AFD0712
 P 3400 3200
-F 0 "#PWR?" H 3400 3050 50  0001 C CNN
+F 0 "#PWR061" H 3400 3050 50  0001 C CNN
 F 1 "+5V" H 3400 3340 50  0000 C CNN
 F 2 "" H 3400 3200 50  0001 C CNN
@@
 	3900 3650 4750 3650
 $Comp
-L +3.3V #PWR?
+L +3.3V #PWR062
 U 1 1 5AFD09DE
 P 4100 3850
-F 0 "#PWR?" H 4100 3700 50  0001 C CNN
+F 0 "#PWR062" H 4100 3700 50  0001 C CNN
 F 1 "+3.3V" H 4100 3990 50  0000 C CNN
 F 2 "" H 4100 3850 50  0001 C CNN
@@
 	3900 3850 4100 3850
 $Comp
-L +3.3V #PWR?
+L +3.3V #PWR063
 U 1 1 5AFD0A66
 P 4100 2250
-F 0 "#PWR?" H 4100 2100 50  0001 C CNN
+F 0 "#PWR063" H 4100 2100 50  0001 C CNN
 F 1 "+3.3V" H 4100 2390 50  0000 C CNN
 F 2 "" H 4100 2250 50  0001 C CNN
@@
 REVIZAR PIN 8 DATASHEET
 $Comp
-L R R?
+L R R18
 U 1 1 5AFD0A96
 P 4400 2350
-F 0 "R?" V 4480 2350 50  0000 C CNN
+F 0 "R18" V 4480 2350 50  0000 C CNN
 F 1 "100" V 4400 2350 50  0000 C CNN
 F 2 "" V 4330 2350 50  0001 C CNN
@@
 $EndComp
 $Comp
-L R R?
+L R R20
 U 1 1 5AFD0AD6
 P 4600 2350
-F 0 "R?" V 4680 2350 50  0000 C CNN
+F 0 "R20" V 4680 2350 50  0000 C CNN
 F 1 "100" V 4600 2350 50  0000 C CNN
 F 2 "" V 4530 2350 50  0001 C CNN
@@
 $EndComp
 $Comp
-L R R?
+L R R19
 U 1 1 5AFD0B26
 P 4400 4050
-F 0 "R?" V 4480 4050 50  0000 C CNN
+F 0 "R19" V 4480 4050 50  0000 C CNN
 F 1 "100" V 4400 4050 50  0000 C CNN
 F 2 "" V 4330 4050 50  0001 C CNN
@@
 $EndComp
 $Comp
-L R R?
+L R R21
 U 1 1 5AFD0B52
 P 4600 4050
-F 0 "R?" V 4680 4050 50  0000 C CNN
+F 0 "R21" V 4680 4050 50  0000 C CNN
 F 1 "100" V 4600 4050 50  0000 C CNN
 F 2 "" V 4530 4050 50  0001 C CNN
@@
 $EndComp
 $Comp
-L C C?
+L C C11
 U 1 1 5AFD0B74
 P 4400 4450
-F 0 "C?" H 4300 4550 50  0000 L CNN
+F 0 "C11" H 4300 4550 50  0000 L CNN
 F 1 "560p" H 4200 4350 50  0000 L CNN
 F 2 "" H 4438 4300 50  0001 C CNN
@@
 $EndComp
 $Comp
-L C C?
+L C C13
 U 1 1 5AFD0BBE
 P 4600 4450
-F 0 "C?" H 4625 4550 50  0000 L CNN
+F 0 "C13" H 4625 4550 50  0000 L CNN
 F 1 "560p" H 4625 4350 50  0000 L CNN
 F 2 "" H 4638 4300 50  0001 C CNN
@@
 $EndComp
 $Comp
-L C C?
+L C C10
 U 1 1 5AFD0BEE
 P 4400 2750
-F 0 "C?" H 4300 2850 50  0000 L CNN
+F 0 "C10" H 4300 2850 50  0000 L CNN
 F 1 "560p" H 4200 2650 50  0000 L CNN
 F 2 "" H 4438 2600 50  0001 C CNN
@@
 $EndComp
 $Comp
-L C C?
+L C C12
 U 1 1 5AFD0C57
 P 4600 2750
-F 0 "C?" H 4625 2850 50  0000 L CNN
+F 0 "C12" H 4625 2850 50  0000 L CNN
 F 1 "560p" H 4625 2650 50  0000 L CNN
 F 2 "" H 4638 2600 50  0001 C CNN
@@
 $EndComp
 $Comp
-L GND #PWR?
+L GND #PWR064
 U 1 1 5AFD0CF3
 P 4500 4700
-F 0 "#PWR?" H 4500 4450 50  0001 C CNN
+F 0 "#PWR064" H 4500 4450 50  0001 C CNN
 F 1 "GND" H 4500 4550 50  0000 C CNN
 F 2 "" H 4500 4700 50  0001 C CNN
@@
 $EndComp
 $Comp
-L GND #PWR?
+L GND #PWR065
 U 1 1 5AFD0D44
 P 4500 3000
-F 0 "#PWR?" H 4500 2750 50  0001 C CNN
+F 0 "#PWR065" H 4500 2750 50  0001 C CNN
 F 1 "GND" H 4500 2850 50  0000 C CNN
 F 2 "" H 4500 3000 50  0001 C CNN
@@
 Connection ~ 4600 2050
 $Comp
-L C C?
+L C C9
 U 1 1 5AFD1564
 P 3700 3250
-F 0 "C?" H 3600 3350 50  0000 L CNN
+F 0 "C9" H 3600 3350 50  0000 L CNN
 F 1 "1u" V 3550 3200 50  0000 L CNN
 F 2 "" H 3738 3100 50  0001 C CNN
@@
 $EndComp
 $Comp
-L C C?
+L C C8
 U 1 1 5AFD1622
 P 3650 1650
-F 0 "C?" H 3550 1750 50  0000 L CNN
+F 0 "C8" H 3550 1750 50  0000 L CNN
 F 1 "1u" V 3500 1550 50  0000 L CNN
 F 2 "" H 3688 1500 50  0001 C CNN
@@
 $EndComp
 $Comp
-L GND #PWR?
+L GND #PWR066
 U 1 1 5AFD172E
 P 3950 1650
-F 0 "#PWR?" H 3950 1400 50  0001 C CNN
+F 0 "#PWR066" H 3950 1400 50  0001 C CNN
 F 1 "GND" H 3950 1500 50  0000 C CNN
 F 2 "" H 3950 1650 50  0001 C CNN
@@
 $EndComp
 $Comp
-L GND #PWR?
+L GND #PWR067
 U 1 1 5AFD175D
 P 4000 3250
-F 0 "#PWR?" H 4000 3000 50  0001 C CNN
+F 0 "#PWR067" H 4000 3000 50  0001 C CNN
 F 1 "GND" H 4000 3100 50  0000 C CNN
 F 2 "" H 4000 3250 50  0001 C CNN
