File: HOST.sch (KiCad schematic (older format))
At the start: 8 parts

Commit message: ready for first rev
Other:
- note added: "Speed Grades & Supply\n4MHz @ 1.8V -> NO\n10MHz @ 3.3V -> LOW POWER\n20MHz @ 5V -> SEGURA"
- note added: "Unconnected Pins -> 15.2.6.\na VCC o GND"
- note removed: "Speed Grades\n– 0 - 4MHz @ 1.8V - 5.5V -> NO\n– 0 - 10MHz @ 2.7V - 5.5V -> LOW POWER\n– 0 - 20MHz @ 4.5 - 5.5V -> SEGURA"
Changed lines of the file:
@@
 3.3V
 Text Notes 1800 1450 0    60   ~ 0
-Speed Grades\n– 0 - 4MHz @ 1.8V - 5.5V -> NO\n– 0 - 10MHz @ 2.7V - 5.5V -> LOW POWER\n– 0 - 20MHz @ 4.5 - 5.5V -> SEGURA
+Speed Grades & Supply\n4MHz  @ 1.8V -> NO\n10MHz @ 3.3V -> LOW POWER\n20MHz @ 5V   -> SEGURA
 Text HLabel 7200 4450 2    60   Input ~ 0
 MASTER_BT_RX
@@
 	4300 1250 4300 1350
 Wire Wire Line
-	4300 1650 4300 1750
+	4300 1750 4300 1650
 Wire Wire Line
 	3250 1750 4500 1750
@@
 Wire Wire Line
 	6500 4950 7200 4950
+Text Notes 5850 1250 0    60   ~ 0
+Unconnected Pins -> 15.2.6.\na VCC o GND
 $EndSCHEMATC

Commit message: fixed some ports errors
Parts:
- gave numbers to parts that had none: 8
Connections:
- net GND: now also U4.15 ((PCINT30/OC2B/ICP)PD6), U4.16 ((PCINT31/OC2A)PD7), U4.25 ((PCINT22/TOSC1)PC6), U4.26 ((PCINT23/TOSC2)PC7), U4.29 (AREF), U4.30 ((PCINT7/ADC7)PA7), U4.31 ((PCINT6/ADC6)PA6), U4.32 ((PCINT5/ADC5)PA5), U4.33 ((PCINT4/ADC4)PA4), U4.34 ((PCINT3/ADC3)PA3), U4.35 ((PCINT2/ADC2)PA2), U4.36 ((PCINT1/ADC1)PA1), U4.37 ((PCINT0/ADC0)PA0), U4.40 ((PCINT8/T0/XCK)PB0), U4.41 ((PCINT9/CLKO/T1)PB1), U4.42 ((PCINT10/AIN0/INT2)PB2), U4.43 ((PCINT11/AIN1/OC0)PB3), U4.44 ((PCINT12/OC0B/~SS~)PB4)
Changed lines of the file:
@@
 $EndDescr
 $Comp
-L ATMEGA164A-AU U?
+L ATMEGA164A-AU U4
 U 1 1 5B069CFB
 P 5500 3450
-F 0 "U?" H 4650 5330 50  0000 L BNN
+F 0 "U4" H 4650 5330 50  0000 L BNN
 F 1 "ATMEGA164A-AU" H 5900 1500 50  0000 L BNN
 F 2 "TQFP44" H 5500 3450 50  0001 C CIN
@@
 Text HLabel 2000 1650 0    60   UnSpc ~ 0
 5V
-Text HLabel 2000 1800 0    60   UnSpc ~ 0
-3.3V
 Text Notes 1800 1450 0    60   ~ 0
 Speed Grades & Supply\n4MHz  @ 1.8V -> NO\n10MHz @ 3.3V -> LOW POWER\n20MHz @ 5V   -> SEGURA
@@
 Connection ~ 5400 5450
 $Comp
-L GND #PWR?
+L GND #PWR095
 U 1 1 5B057F0C
 P 5350 5550
-F 0 "#PWR?" H 5350 5300 50  0001 C CNN
+F 0 "#PWR095" H 5350 5300 50  0001 C CNN
 F 1 "GND" H 5350 5400 50  0000 C CNN
 F 2 "" H 5350 5550 50  0001 C CNN
@@
 Connection ~ 5300 1450
 $Comp
-L R R?
+L R R44
 U 1 1 5B057F90
 P 4300 1500
-F 0 "R?" V 4380 1500 50  0000 C CNN
+F 0 "R44" V 4380 1500 50  0000 C CNN
 F 1 "50k" V 4300 1500 50  0000 C CNN
 F 2 "" V 4230 1500 50  0001 C CNN
@@
 $EndComp
 $Comp
-L +5V #PWR?
+L +5V #PWR096
 U 1 1 5B058075
 P 2150 1650
-F 0 "#PWR?" H 2150 1500 50  0001 C CNN
+F 0 "#PWR096" H 2150 1500 50  0001 C CNN
 F 1 "+5V" H 2150 1790 50  0000 C CNN
 F 2 "" H 2150 1650 50  0001 C CNN
@@
 $EndComp
 $Comp
-L +5V #PWR?
+L +5V #PWR097
 U 1 1 5B05808D
 P 4300 1250
-F 0 "#PWR?" H 4300 1100 50  0001 C CNN
+F 0 "#PWR097" H 4300 1100 50  0001 C CNN
 F 1 "+5V" H 4300 1390 50  0000 C CNN
 F 2 "" H 4300 1250 50  0001 C CNN
@@
 $EndComp
 $Comp
-L +5V #PWR?
+L +5V #PWR098
 U 1 1 5B05809E
 P 5400 1300
-F 0 "#PWR?" H 5400 1150 50  0001 C CNN
+F 0 "#PWR098" H 5400 1150 50  0001 C CNN
 F 1 "+5V" H 5400 1440 50  0000 C CNN
 F 2 "" H 5400 1300 50  0001 C CNN
@@
 	5400 1300 5400 1450
 $Comp
-L Crystal Y?
+L Crystal Y2
 U 1 1 5B05818A
 P 4350 2350
-F 0 "Y?" H 4350 2500 50  0000 C CNN
+F 0 "Y2" H 4350 2500 50  0000 C CNN
 F 1 "16MHz" H 4350 2200 50  0000 C CNN
 F 2 "" H 4350 2350 50  0001 C CNN
@@
 $EndComp
 $Comp
-L C C?
+L C C22
 U 1 1 5B0581EF
 P 3950 2150
-F 0 "C?" H 3975 2250 50  0000 L CNN
+F 0 "C22" H 3975 2250 50  0000 L CNN
 F 1 "22p" V 4100 2100 50  0000 L CNN
 F 2 "" H 3988 2000 50  0001 C CNN
@@
 $EndComp
 $Comp
-L C C?
+L C C23
 U 1 1 5B058228
 P 3950 2550
-F 0 "C?" H 3975 2650 50  0000 L CNN
+F 0 "C23" H 3975 2650 50  0000 L CNN
 F 1 "22p" V 4100 2500 50  0000 L CNN
 F 2 "" H 3988 2400 50  0001 C CNN
@@
 	3800 2150 3800 2550
 $Comp
-L GND #PWR?
+L GND #PWR099
 U 1 1 5B0583D3
 P 3600 2400
-F 0 "#PWR?" H 3600 2150 50  0001 C CNN
+F 0 "#PWR099" H 3600 2150 50  0001 C CNN
 F 1 "GND" H 3600 2250 50  0000 C CNN
 F 2 "" H 3600 2400 50  0001 C CNN
@@
 PROTECCION PARA LA DIFERENCIA ENTRE \nLOS Vcc DE PLACA ENCHUFADA AL AUTO\nY Vcc DE COMPU, ETC
 $Comp
-L C C?
+L C C21
 U 1 1 5B058BE1
 P 2400 2450
-F 0 "C?" H 2425 2550 50  0000 L CNN
+F 0 "C21" H 2425 2550 50  0000 L CNN
 F 1 "100n" H 2425 2350 50  0000 L CNN
 F 2 "" H 2438 2300 50  0001 C CNN
@@
 $EndComp
 $Comp
-L +5V #PWR?
+L +5V #PWR0100
 U 1 1 5B058C84
 P 2400 2200
-F 0 "#PWR?" H 2400 2050 50  0001 C CNN
+F 0 "#PWR0100" H 2400 2050 50  0001 C CNN
 F 1 "+5V" H 2400 2340 50  0000 C CNN
 F 2 "" H 2400 2200 50  0001 C CNN
@@
 $EndComp
 $Comp
-L GND #PWR?
+L GND #PWR0101
 U 1 1 5B058CBF
 P 2400 2700
-F 0 "#PWR?" H 2400 2450 50  0001 C CNN
+F 0 "#PWR0101" H 2400 2450 50  0001 C CNN
 F 1 "GND" H 2400 2550 50  0000 C CNN
 F 2 "" H 2400 2700 50  0001 C CNN
@@
 Connection ~ 4350 2550
 $Comp
-L SW_Push SW?
+L SW_Push SW1
 U 1 1 5B05974A
 P 3500 1950
-F 0 "SW?" H 3550 2050 50  0000 L CNN
+F 0 "SW1" H 3550 2050 50  0000 L CNN
 F 1 "SW_Push" H 3500 1890 50  0000 C CNN
 F 2 "" H 3500 2150 50  0001 C CNN
@@
 $EndComp
 $Comp
-L GND #PWR?
+L GND #PWR0102
 U 1 1 5B0597BA
 P 3500 2150
-F 0 "#PWR?" H 3500 1900 50  0001 C CNN
+F 0 "#PWR0102" H 3500 1900 50  0001 C CNN
 F 1 "GND" H 3500 2000 50  0000 C CNN
 F 2 "" H 3500 2150 50  0001 C CNN
@@
 Connection ~ 3500 1750
 $Comp
-L R R?
+L R R45
 U 1 1 5B075F2E
 P 6900 4400
-F 0 "R?" V 6980 4400 50  0000 C CNN
+F 0 "R45" V 6980 4400 50  0000 C CNN
 F 1 "4.7K" V 6900 4400 50  0000 C CNN
 F 2 "" V 6830 4400 50  0001 C CNN
@@
 Connection ~ 6900 4550
 $Comp
-L +5V #PWR?
+L +5V #PWR0103
 U 1 1 5B0760B5
 P 6900 4250
-F 0 "#PWR?" H 6900 4100 50  0001 C CNN
+F 0 "#PWR0103" H 6900 4100 50  0001 C CNN
 F 1 "+5V" H 6900 4390 50  0000 C CNN
 F 2 "" H 6900 4250 50  0001 C CNN
@@
 Text Notes 5850 1250 0    60   ~ 0
 Unconnected Pins -> 15.2.6.\na VCC o GND
+$Comp
+L GND #PWR0104
+U 1 1 5B221FAD
+P 4500 2950
+F 0 "#PWR0104" H 4500 2700 50  0001 C CNN
+F 1 "GND" H 4500 2800 50  0000 C CNN
+F 2 "" H 4500 2950 50  0001 C CNN
+F 3 "" H 4500 2950 50  0001 C CNN
+	1    4500 2950
+	1    0    0    -1
+$EndComp
+Wire Wire Line
+	6500 1750 6500 3050
+Connection ~ 6500 2950
+Connection ~ 6500 2850
+Connection ~ 6500 2750
+Connection ~ 6500 2650
+Connection ~ 6500 2450
+Connection ~ 6500 2350
+Connection ~ 6500 2250
+Connection ~ 6500 2150
+Connection ~ 6500 2050
+Connection ~ 6500 1950
+Connection ~ 6500 1850
+Wire Wire Line
+	6500 4250 6500 4150
+Wire Wire Line
+	6500 5050 6500 5150
+$Comp
+L GND #PWR0105
+U 1 1 5B222469
+P 6700 5150
+F 0 "#PWR0105" H 6700 4900 50  0001 C CNN
+F 1 "GND" H 6700 5000 50  0000 C CNN
+F 2 "" H 6700 5150 50  0001 C CNN
+F 3 "" H 6700 5150 50  0001 C CNN
+	1    6700 5150
+	1    0    0    -1
+$EndComp
+$Comp
+L GND #PWR0106
+U 1 1 5B22248C
+P 6700 2550
+F 0 "#PWR0106" H 6700 2300 50  0001 C CNN
+F 1 "GND" H 6700 2400 50  0000 C CNN
+F 2 "" H 6700 2550 50  0001 C CNN
+F 3 "" H 6700 2550 50  0001 C CNN
+	1    6700 2550
+	1    0    0    -1
+$EndComp
+Wire Wire Line
+	6500 2550 6700 2550
+Connection ~ 6500 2550
+Wire Wire Line
+	6500 5100 6700 5100
+Wire Wire Line
+	6700 5100 6700 5150
+Connection ~ 6500 5100
+$Comp
+L GND #PWR0107
+U 1 1 5B2225C1
+P 6700 4200
+F 0 "#PWR0107" H 6700 3950 50  0001 C CNN
+F 1 "GND" H 6700 4050 50  0000 C CNN
+F 2 "" H 6700 4200 50  0001 C CNN
+F 3 "" H 6700 4200 50  0001 C CNN
+	1    6700 4200
+	1    0    0    -1
+$EndComp
+Wire Wire Line
+	6500 4200 6700 4200
+Connection ~ 6500 4200
 $EndSCHEMATC
