File: J1850_BUS.sch (KiCad schematic (older format))
At the start: 28 parts

Commit message: fixed some ports errors
Parts:
- gave numbers to parts that had none: 26
Connections:
- net +5V: now also U1.3 (V+), U1.3 (V+)
- no-connect marks 3 -> 8
