File: OBD2_CONNECTOR.sch (KiCad schematic (older format))
At the start: 10 parts

Commit message: fixed some ports errors
Parts:
- gave numbers to parts that had none: 8
- renumbered S2A to S2A1
Changed lines of the file:
@@
 $EndDescr
 $Comp
-L CONN_01X16 J?
+L CONN_01X16 J5
 U 1 1 5AFCB095
 P 2450 3650
-F 0 "J?" H 2450 4500 50  0000 C CNN
+F 0 "J5" H 2450 4500 50  0000 C CNN
 F 1 "OBD2_CONNECTOR" V 2550 3650 50  0000 C CNN
 F 2 "" H 2450 3650 50  0001 C CNN
@@
 $EndComp
 $Comp
-L GND #PWR?
+L GND #PWR043
 U 1 1 5AFCB20C
 P 2750 4000
-F 0 "#PWR?" H 2750 3750 50  0001 C CNN
+F 0 "#PWR043" H 2750 3750 50  0001 C CNN
 F 1 "GND" H 2750 3850 50  0000 C CNN
 F 2 "" H 2750 4000 50  0001 C CNN
@@
 NoConn ~ 2650 3200
 $Comp
-L PESD1CAN D?
+L PESD1CAN D6
 U 1 1 5AFD7B19
 P 2800 5100
-F 0 "D?" H 2800 5551 50  0000 L BNN
+F 0 "D6" H 2800 5551 50  0000 L BNN
 F 1 "PESD1CAN" H 2800 5000 50  0000 L BNN
 F 2 "SOT23-3" H 2800 5100 50  0001 L BNN
@@
 $EndComp
 $Comp
-L PESD1CAN D?
+L PESD1CAN D7
 U 1 1 5AFD7C20
 P 3500 5100
-F 0 "D?" H 3500 5551 50  0000 L BNN
+F 0 "D7" H 3500 5551 50  0000 L BNN
 F 1 "PESD1CAN" H 3500 5000 50  0000 L BNN
 F 2 "SOT23-3" H 3500 5100 50  0001 L BNN
@@
 $EndComp
 $Comp
-L GND #PWR?
+L GND #PWR044
 U 1 1 5AFD7C77
 P 3300 5750
-F 0 "#PWR?" H 3300 5500 50  0001 C CNN
+F 0 "#PWR044" H 3300 5500 50  0001 C CNN
 F 1 "GND" H 3300 5600 50  0000 C CNN
 F 2 "" H 3300 5750 50  0001 C CNN
@@
 11
 $Comp
-L D_Schottky_x2_ACom_KKA D?
+L D_Schottky_x2_ACom_KKA D8
 U 1 1 5AFD819A
 P 4850 5250
-F 0 "D?" H 4900 5150 50  0000 C CNN
+F 0 "D8" H 4900 5150 50  0000 C CNN
 F 1 "MMBZ27VAL" H 4850 5350 50  0000 C CNN
 F 2 "" H 4850 5250 50  0001 C CNN
@@
 $EndComp
 $Comp
-L D_Schottky_x2_ACom_KKA D?
+L D_Schottky_x2_ACom_KKA D9
 U 1 1 5AFD8202
 P 5950 5250
-F 0 "D?" H 6000 5150 50  0000 C CNN
+F 0 "D9" H 6000 5150 50  0000 C CNN
 F 1 "MMBZ27VAL" H 5950 5350 50  0000 C CNN
 F 2 "" H 5950 5250 50  0001 C CNN
@@
 $EndComp
 $Comp
-L D_Schottky_x2_ACom_KKA D?
+L D_Schottky_x2_ACom_KKA D10
 U 1 1 5AFD828F
 P 7100 5400
-F 0 "D?" H 7150 5300 50  0000 C CNN
+F 0 "D10" H 7150 5300 50  0000 C CNN
 F 1 "MMBZ27VAL" H 7100 5500 50  0000 C CNN
 F 2 "" H 7100 5400 50  0001 C CNN
@@
 $EndComp
 $Comp
-L GND #PWR?
+L GND #PWR045
 U 1 1 5AFD853B
 P 5950 5550
-F 0 "#PWR?" H 5950 5300 50  0001 C CNN
+F 0 "#PWR045" H 5950 5300 50  0001 C CNN
 F 1 "GND" H 5950 5400 50  0000 C CNN
 F 2 "" H 5950 5550 50  0001 C CNN
@@
 $EndComp
 $Comp
-L GND #PWR?
+L GND #PWR046
 U 1 1 5AFD8558
 P 4850 5550
-F 0 "#PWR?" H 4850 5300 50  0001 C CNN
+F 0 "#PWR046" H 4850 5300 50  0001 C CNN
 F 1 "GND" H 4850 5400 50  0000 C CNN
 F 2 "" H 4850 5550 50  0001 C CNN
@@
 $EndComp
 $Comp
-L GND #PWR?
+L GND #PWR047
 U 1 1 5AFD85BB
 P 7100 5850
-F 0 "#PWR?" H 7100 5600 50  0001 C CNN
+F 0 "#PWR047" H 7100 5600 50  0001 C CNN
 F 1 "GND" H 7100 5700 50  0000 C CNN
 F 2 "" H 7100 5850 50  0001 C CNN
@@
 	7100 5100 7100 4850
 $Comp
-L Polyfuse F?
+L Polyfuse F1
 U 1 1 5AFD97C6
 P 6300 3100
-F 0 "F?" V 6200 3100 50  0000 C CNN
+F 0 "F1" V 6200 3100 50  0000 C CNN
 F 1 "PTS181230V020" V 6400 3100 50  0000 C CNN
 F 2 "" H 6350 2900 50  0001 L CNN
@@
 $EndComp
 $Comp
-L D S2A
+L D S2A1
 U 1 1 5AFD981B
 P 6900 3100
-F 0 "S2A" H 6900 3200 50  0000 C CNN
+F 0 "S2A1" H 6900 3200 50  0000 C CNN
 F 1 "D" H 6900 3000 50  0000 C CNN
 F 2 "" H 6900 3100 50  0001 C CNN
@@
 $EndComp
 $Comp
-L C C?
+L C C3
 U 1 1 5AFD98BC
 P 5850 3450
-F 0 "C?" H 5875 3550 50  0000 L CNN
+F 0 "C3" H 5875 3550 50  0000 L CNN
 F 1 "10n 100V" H 5875 3350 50  0000 L CNN
 F 2 "" H 5888 3300 50  0001 C CNN
@@
 Connection ~ 6650 3100
 $Comp
-L GND #PWR?
+L GND #PWR048
 U 1 1 5AFDA018
 P 6300 3700
-F 0 "#PWR?" H 6300 3450 50  0001 C CNN
+F 0 "#PWR048" H 6300 3450 50  0001 C CNN
 F 1 "GND" H 6300 3550 50  0000 C CNN
 F 2 "" H 6300 3700 50  0001 C CNN
@@
 Imax = 200mA
 $Comp
-L VCC #PWR?
+L VCC #PWR049
 U 1 1 5AFE2824
 P 7200 3000
-F 0 "#PWR?" H 7200 2850 50  0001 C CNN
+F 0 "#PWR049" H 7200 2850 50  0001 C CNN
 F 1 "VCC" H 7200 3150 50  0000 C CNN
 F 2 "" H 7200 3000 50  0001 C CNN
