File: KiCad Proyecto/CAN.sch (KiCad schematic (older format))
At the start: 12 parts, among them U2 MCP2562-E/MF, U3 MCP2562-E/MF

Commit message: git commit -m se usa para dejar un mensaje al commitear
Connections:
- net HS_CAN_LO: now also R20.1
- net HS_CAN_RX_STN: no longer R20.1
- net HS_CAN_TX: now also R18.1
- net HS_CAN_TX_STN: no longer R18.1
- net MS_CAN_HI: now also R19.1
- net MS_CAN_LO: now also R21.1
- net MS_CAN_RX_STN: no longer R21.1
- net MS_CAN_TX_STN: no longer R19.1
Other:
- note added: "REVIZAR de RUSIA PIN 8 DATASHEET"
- note removed: "REVIZAR PIN 8 DATASHEET"
- moved on the sheet: C10, C11, C12, C13, R18, R19, R20, R21
Changed lines of the file:
@@
 	3850 2250 4100 2250
 Text Notes 2950 2950 0    60   ~ 0
-REVIZAR PIN 8 DATASHEET
+REVIZAR de RUSIA PIN 8 DATASHEET
 $Comp
 L R R18
 U 1 1 5AFD0A96
-P 4400 2350
-F 0 "R18" V 4480 2350 50  0000 C CNN
-F 1 "100" V 4400 2350 50  0000 C CNN
-F 2 "" V 4330 2350 50  0001 C CNN
-F 3 "" H 4400 2350 50  0001 C CNN
-	1    4400 2350
+P 2550 2550
+F 0 "R18" V 2630 2550 50  0000 C CNN
+F 1 "100" V 2550 2550 50  0000 C CNN
+F 2 "" V 2480 2550 50  0001 C CNN
+F 3 "" H 2550 2550 50  0001 C CNN
+	1    2550 2550
 	1    0    0    -1
 $EndComp
@@
 L R R20
 U 1 1 5AFD0AD6
-P 4600 2350
-F 0 "R20" V 4680 2350 50  0000 C CNN
-F 1 "100" V 4600 2350 50  0000 C CNN
-F 2 "" V 4530 2350 50  0001 C CNN
-F 3 "" H 4600 2350 50  0001 C CNN
-	1    4600 2350
+P 2750 2550
+F 0 "R20" V 2830 2550 50  0000 C CNN
+F 1 "100" V 2750 2550 50  0000 C CNN
+F 2 "" V 2680 2550 50  0001 C CNN
+F 3 "" H 2750 2550 50  0001 C CNN
+	1    2750 2550
 	1    0    0    -1
 $EndComp
@@
 L R R19
 U 1 1 5AFD0B26
-P 4400 4050
-F 0 "R19" V 4480 4050 50  0000 C CNN
-F 1 "100" V 4400 4050 50  0000 C CNN
-F 2 "" V 4330 4050 50  0001 C CNN
-F 3 "" H 4400 4050 50  0001 C CNN
-	1    4400 4050
+P 2500 4250
+F 0 "R19" V 2580 4250 50  0000 C CNN
+F 1 "100" V 2500 4250 50  0000 C CNN
+F 2 "" V 2430 4250 50  0001 C CNN
+F 3 "" H 2500 4250 50  0001 C CNN
+	1    2500 4250
 	1    0    0    -1
 $EndComp
@@
 L R R21
 U 1 1 5AFD0B52
-P 4600 4050
-F 0 "R21" V 4680 4050 50  0000 C CNN
-F 1 "100" V 4600 4050 50  0000 C CNN
-F 2 "" V 4530 4050 50  0001 C CNN
-F 3 "" H 4600 4050 50  0001 C CNN
-	1    4600 4050
+P 2700 4250
+F 0 "R21" V 2780 4250 50  0000 C CNN
+F 1 "100" V 2700 4250 50  0000 C CNN
+F 2 "" V 2630 4250 50  0001 C CNN
+F 3 "" H 2700 4250 50  0001 C CNN
+	1    2700 4250
 	1    0    0    -1
 $EndComp
@@
 L C C11
 U 1 1 5AFD0B74
-P 4400 4450
-F 0 "C11" H 4300 4550 50  0000 L CNN
-F 1 "560p" H 4200 4350 50  0000 L CNN
-F 2 "" H 4438 4300 50  0001 C CNN
-F 3 "" H 4400 4450 50  0001 C CNN
-	1    4400 4450
+P 2500 4650
+F 0 "C11" H 2400 4750 50  0000 L CNN
+F 1 "560p" H 2300 4550 50  0000 L CNN
+F 2 "" H 2538 4500 50  0001 C CNN
+F 3 "" H 2500 4650 50  0001 C CNN
+	1    2500 4650
 	1    0    0    -1
 $EndComp
@@
 L C C13
 U 1 1 5AFD0BBE
-P 4600 4450
-F 0 "C13" H 4625 4550 50  0000 L CNN
-F 1 "560p" H 4625 4350 50  0000 L CNN
-F 2 "" H 4638 4300 50  0001 C CNN
-F 3 "" H 4600 4450 50  0001 C CNN
-	1    4600 4450
+P 2700 4650
+F 0 "C13" H 2725 4750 50  0000 L CNN
+F 1 "560p" H 2725 4550 50  0000 L CNN
+F 2 "" H 2738 4500 50  0001 C CNN
+F 3 "" H 2700 4650 50  0001 C CNN
+	1    2700 4650
 	1    0    0    -1
 $EndComp
@@
 L C C10
 U 1 1 5AFD0BEE
-P 4400 2750
-F 0 "C10" H 4300 2850 50  0000 L CNN
-F 1 "560p" H 4200 2650 50  0000 L CNN
-F 2 "" H 4438 2600 50  0001 C CNN
-F 3 "" H 4400 2750 50  0001 C CNN
-	1    4400 2750
+P 2550 2950
+F 0 "C10" H 2450 3050 50  0000 L CNN
+F 1 "560p" H 2350 2850 50  0000 L CNN
+F 2 "" H 2588 2800 50  0001 C CNN
+F 3 "" H 2550 2950 50  0001 C CNN
+	1    2550 2950
 	1    0    0    -1
 $EndComp
@@
 L C C12
 U 1 1 5AFD0C57
-P 4600 2750
-F 0 "C12" H 4625 2850 50  0000 L CNN
-F 1 "560p" H 4625 2650 50  0000 L CNN
-F 2 "" H 4638 2600 50  0001 C CNN
-F 3 "" H 4600 2750 50  0001 C CNN
-	1    4600 2750
+P 2750 2950
+F 0 "C12" H 2775 3050 50  0000 L CNN
+F 1 "560p" H 2775 2850 50  0000 L CNN
+F 2 "" H 2788 2800 50  0001 C CNN
+F 3 "" H 2750 2950 50  0001 C CNN
+	1    2750 2950
 	1    0    0    -1
 $EndComp
@@
 L GND #PWR064
 U 1 1 5AFD0CF3
-P 4500 4700
-F 0 "#PWR064" H 4500 4450 50  0001 C CNN
-F 1 "GND" H 4500 4550 50  0000 C CNN
-F 2 "" H 4500 4700 50  0001 C CNN
-F 3 "" H 4500 4700 50  0001 C CNN
-	1    4500 4700
+P 2600 4900
+F 0 "#PWR064" H 2600 4650 50  0001 C CNN
+F 1 "GND" H 2600 4750 50  0000 C CNN
+F 2 "" H 2600 4900 50  0001 C CNN
+F 3 "" H 2600 4900 50  0001 C CNN
+	1    2600 4900
 	1    0    0    -1
 $EndComp
@@
 L GND #PWR065
 U 1 1 5AFD0D44
-P 4500 3000
-F 0 "#PWR065" H 4500 2750 50  0001 C CNN
-F 1 "GND" H 4500 2850 50  0000 C CNN
-F 2 "" H 4500 3000 50  0001 C CNN
-F 3 "" H 4500 3000 50  0001 C CNN
-	1    4500 3000
-	1    0    0    -1
-$EndComp
-Wire Wire Line
-	4400 3900 4400 3550
-Connection ~ 4400 3550
-Wire Wire Line
-	4600 3900 4600 3650
-Connection ~ 4600 3650
-Wire Wire Line
-	4400 4200 4400 4300
-Wire Wire Line
-	4600 4200 4600 4300
-Wire Wire Line
-	4400 4600 4400 4700
-Wire Wire Line
-	4400 4700 4600 4700
-Wire Wire Line
-	4600 4700 4600 4600
-Connection ~ 4500 4700
-Wire Wire Line
-	4400 2500 4400 2600
-Wire Wire Line
-	4600 2500 4600 2600
-Wire Wire Line
-	4400 2900 4400 3000
-Wire Wire Line
-	4400 3000 4600 3000
-Wire Wire Line
-	4600 3000 4600 2900
-Connection ~ 4500 3000
-Wire Wire Line
-	4400 2200 4400 1950
-Connection ~ 4400 1950
-Wire Wire Line
-	4600 2200 4600 2050
-Connection ~ 4600 2050
+P 2650 3200
+F 0 "#PWR065" H 2650 2950 50  0001 C CNN
+F 1 "GND" H 2650 3050 50  0000 C CNN
+F 2 "" H 2650 3200 50  0001 C CNN
+F 3 "" H 2650 3200 50  0001 C CNN
+	1    2650 3200
+	1    0    0    -1
+$EndComp
+Wire Wire Line
+	2500 3650 2500 4100
+Wire Wire Line
+	2700 4100 2700 3850
+Wire Wire Line
+	2500 4400 2500 4500
+Wire Wire Line
+	2700 4400 2700 4500
+Wire Wire Line
+	2500 4800 2500 4900
+Wire Wire Line
+	2500 4900 2700 4900
+Wire Wire Line
+	2700 4900 2700 4800
+Connection ~ 2600 4900
+Wire Wire Line
+	2550 2700 2550 2800
+Wire Wire Line
+	2750 2700 2750 2800
+Wire Wire Line
+	2550 3100 2550 3200
+Wire Wire Line
+	2550 3200 2750 3200
+Wire Wire Line
+	2750 3200 2750 3100
+Connection ~ 2650 3200
+Wire Wire Line
+	2550 2050 2550 2400
+Wire Wire Line
+	2750 2400 2750 2250
 $Comp
 L C C9
@@
 Wire Wire Line
 	3800 1650 3950 1650
+Connection ~ 2700 3850
+Connection ~ 2500 3650
+Connection ~ 2550 2050
+Connection ~ 2750 2250
 $EndSCHEMATC

Commit message: mensaje generado de forma aleatoria
Other:
- note added: "REVIZAR de RUSIA PIN 8 DATASHEET\nSTBY esta conectado internamente a un PULL UP a VDD"
- note removed: "REVIZAR de RUSIA PIN 8 DATASHEET"
Changed lines of the file:
@@
 	1    0    0    -1
 $EndComp
-Wire Wire Line
-	1700 2750 1800 2750
-Wire Wire Line
-	1800 2750 1800 2700
-Wire Wire Line
-	1700 2850 2000 2850
-Wire Wire Line
-	3350 2550 3450 2550
-Wire Wire Line
-	3400 2650 3400 2550
-Connection ~ 3400 2550
-Wire Wire Line
-	3400 3200 3400 3350
-Wire Wire Line
-	3350 1600 3350 1750
-Wire Wire Line
-	3400 4150 3500 4150
-Wire Wire Line
-	3450 4250 3450 4150
-Connection ~ 3450 4150
-Wire Wire Line
-	2400 2050 2850 2050
-Wire Wire Line
-	2400 2250 2850 2250
-Wire Wire Line
-	2350 3650 2900 3650
-Wire Wire Line
-	2350 3850 2900 3850
-Wire Wire Line
-	3850 1950 4700 1950
-Wire Wire Line
-	3850 2050 4700 2050
-Wire Wire Line
-	3900 3550 4750 3550
-Wire Wire Line
-	3900 3650 4750 3650
 $Comp
 L +3.3V #PWR062
@@
 	1    0    0    -1
 $EndComp
-Wire Wire Line
-	3900 3850 4100 3850
 $Comp
 L +3.3V #PWR063
@@
 	1    0    0    -1
 $EndComp
-Wire Wire Line
-	3850 2250 4100 2250
 Text Notes 2950 2950 0    60   ~ 0
-REVIZAR de RUSIA PIN 8 DATASHEET
+REVIZAR de RUSIA PIN 8 DATASHEET\nSTBY esta conectado internamente a un PULL UP a VDD
 $Comp
 L R R18
@@
 	1    0    0    -1
 $EndComp
-Wire Wire Line
-	2500 3650 2500 4100
-Wire Wire Line
-	2700 4100 2700 3850
-Wire Wire Line
-	2500 4400 2500 4500
-Wire Wire Line
-	2700 4400 2700 4500
-Wire Wire Line
-	2500 4800 2500 4900
-Wire Wire Line
-	2500 4900 2700 4900
-Wire Wire Line
-	2700 4900 2700 4800
-Connection ~ 2600 4900
-Wire Wire Line
-	2550 2700 2550 2800
-Wire Wire Line
-	2750 2700 2750 2800
-Wire Wire Line
-	2550 3100 2550 3200
-Wire Wire Line
-	2550 3200 2750 3200
-Wire Wire Line
-	2750 3200 2750 3100
-Connection ~ 2650 3200
-Wire Wire Line
-	2550 2050 2550 2400
-Wire Wire Line
-	2750 2400 2750 2250
 $Comp
 L C C9
@@
 $EndComp
 Wire Wire Line
+	1700 2750 1800 2750
+Wire Wire Line
+	1800 2750 1800 2700
+Wire Wire Line
+	1700 2850 2000 2850
+Wire Wire Line
+	3350 2550 3450 2550
+Wire Wire Line
+	3400 2650 3400 2550
+Connection ~ 3400 2550
+Wire Wire Line
+	3400 3200 3400 3350
+Wire Wire Line
+	3350 1600 3350 1750
+Wire Wire Line
+	3400 4150 3500 4150
+Wire Wire Line
+	3450 4250 3450 4150
+Connection ~ 3450 4150
+Wire Wire Line
+	2400 2050 2850 2050
+Wire Wire Line
+	2400 2250 2850 2250
+Wire Wire Line
+	2350 3650 2900 3650
+Wire Wire Line
+	2350 3850 2900 3850
+Wire Wire Line
+	3850 1950 4700 1950
+Wire Wire Line
+	3850 2050 4700 2050
+Wire Wire Line
+	3900 3550 4750 3550
+Wire Wire Line
+	3900 3650 4750 3650
+Wire Wire Line
+	3900 3850 4100 3850
+Wire Wire Line
+	3850 2250 4100 2250
+Wire Wire Line
+	2500 3650 2500 4100
+Wire Wire Line
+	2700 4100 2700 3850
+Wire Wire Line
+	2500 4400 2500 4500
+Wire Wire Line
+	2700 4400 2700 4500
+Wire Wire Line
+	2500 4800 2500 4900
+Wire Wire Line
+	2500 4900 2700 4900
+Wire Wire Line
+	2700 4900 2700 4800
+Connection ~ 2600 4900
+Wire Wire Line
+	2550 2700 2550 2800
+Wire Wire Line
+	2750 2700 2750 2800
+Wire Wire Line
+	2550 3100 2550 3200
+Wire Wire Line
+	2550 3200 2750 3200
+Wire Wire Line
+	2750 3200 2750 3100
+Connection ~ 2650 3200
+Wire Wire Line
+	2550 2050 2550 2400
+Wire Wire Line
+	2750 2400 2750 2250
+Wire Wire Line
 	3550 3250 3400 3250
