File: KiCad Proyecto/HOST.sch (KiCad schematic (older format))
At the start: 8 parts, among them SW1 SW_Push, U4 ATMEGA164A-AU, Y2 16MHz

Commit message: Esto es un comentario escrito en una consola
Parts:
- added R46: 50k, symbol R
Connections:
- net GND: now also R46.2; no longer U4.30 ((PCINT7/ADC7)PA7), U4.31 ((PCINT6/ADC6)PA6), U4.32 ((PCINT5/ADC5)PA5), U4.33 ((PCINT4/ADC4)PA4), U4.34 ((PCINT3/ADC3)PA3), U4.35 ((PCINT2/ADC2)PA2), U4.36 ((PCINT1/ADC1)PA1), U4.37 ((PCINT0/ADC0)PA0), U4.40 ((PCINT8/T0/XCK)PB0), U4.41 ((PCINT9/CLKO/T1)PB1), U4.42 ((PCINT10/AIN0/INT2)PB2), U4.43 ((PCINT11/AIN1/OC0)PB3), U4.44 ((PCINT12/OC0B/~SS~)PB4)
- new net: R46.1, U4.30 ((PCINT7/ADC7)PA7), U4.31 ((PCINT6/ADC6)PA6), U4.32 ((PCINT5/ADC5)PA5), U4.33 ((PCINT4/ADC4)PA4), U4.34 ((PCINT3/ADC3)PA3), U4.35 ((PCINT2/ADC2)PA2), U4.36 ((PCINT1/ADC1)PA1), U4.37 ((PCINT0/ADC0)PA0), U4.40 ((PCINT8/T0/XCK)PB0), U4.41 ((PCINT9/CLKO/T1)PB1), U4.42 ((PCINT10/AIN0/INT2)PB2), U4.43 ((PCINT11/AIN1/OC0)PB3), U4.44 ((PCINT12/OC0B/~SS~)PB4)
Changed lines of the file:
@@
 L GND #PWR0106
 U 1 1 5B22248C
-P 6700 2550
-F 0 "#PWR0106" H 6700 2300 50  0001 C CNN
-F 1 "GND" H 6700 2400 50  0000 C CNN
-F 2 "" H 6700 2550 50  0001 C CNN
-F 3 "" H 6700 2550 50  0001 C CNN
-	1    6700 2550
+P 6850 2850
+F 0 "#PWR0106" H 6850 2600 50  0001 C CNN
+F 1 "GND" H 6850 2700 50  0000 C CNN
+F 2 "" H 6850 2850 50  0001 C CNN
+F 3 "" H 6850 2850 50  0001 C CNN
+	1    6850 2850
 	1    0    0    -1
 $EndComp
 Wire Wire Line
-	6500 2550 6700 2550
+	6500 2550 6850 2550
 Connection ~ 6500 2550
 Wire Wire Line
@@
 	6500 4200 6700 4200
 Connection ~ 6500 4200
+$Comp
+L R R46
+U 1 1 5B2C890B
+P 6850 2700
+F 0 "R46" V 6930 2700 50  0000 C CNN
+F 1 "50k" V 6850 2700 50  0000 C CNN
+F 2 "" V 6780 2700 50  0001 C CNN
+F 3 "" H 6850 2700 50  0001 C CNN
+	1    6850 2700
+	1    0    0    -1
+$EndComp
 $EndSCHEMATC
