File: KiCad Proyecto/J1850_BUS.sch (KiCad schematic (older format))
At the start: 26 parts, among them Q1 2N7002, Q2 2N7002, Q3 3904, Q4 RSU002P03, U1 LM339

Commit message: Japon de mierda me cagaste el Prode, la fafafa no ayudó
Parts:
- removed Q4: RSU002P03, symbol Q_NMOS_DGS
- added Q4: RSU002P03, symbol Q_PMOS_SGD
Connections:
- wire segments 60 -> 61
Changed lines of the file:
@@
 Text HLabel 7200 2200 0    60   Input ~ 0
 J1850_BUS+_TX
-Text HLabel 4100 2350 0    60   Input ~ 0
+Text HLabel 4250 2300 0    60   Input ~ 0
 J1850_BUS+_VH
 Text HLabel 6900 5050 0    60   Input ~ 0
@@
 U 1 1 5AFCEA62
 P 7750 2150
+AR Path="/5AFCEA62" Ref="Q2"  Part="1"
+AR Path="/5AFB6308/5AFCEA62" Ref="Q2"  Part="1"
 F 0 "Q2" H 7950 2225 50  0000 L CNN
 F 1 "2N7002" H 7950 2150 50  0000 L CNN
@@
 $EndComp
 $Comp
-L 2N7002 Q1
-U 1 1 5AFD20A7
-P 4550 2300
-F 0 "Q1" H 4750 2375 50  0000 L CNN
-F 1 "2N7002" H 4500 2050 50  0000 L CNN
-F 2 "TO_SOT_Packages_SMD:SOT-23" H 4750 2225 50  0001 L CIN
-F 3 "" H 4550 2300 50  0001 L CNN
-	1    4550 2300
-	1    0    0    -1
-$EndComp
-$Comp
 L VCC #PWR033
 U 1 1 5AFD253B
@@
 V_J1850
 Wire Wire Line
-	5000 1500 5000 1600
-Wire Wire Line
-	5000 1600 4800 1600
+	5000 1600 5000 1500
+Wire Wire Line
+	4800 1600 5000 1600
 $Comp
 L R R9
@@
 	4900 2700 4900 2600
 Connection ~ 4900 2600
-Wire Wire Line
-	4100 2350 4350 2350
 Text Notes 3700 850  0    60   ~ 0
 CAP CERCA DE LM
@@
 EL ARDU USA \nBSS138
 Wire Wire Line
-	7850 1950 7850 1800
+	7850 1800 7850 1950
 Text Label 7850 1250 0    60   ~ 0
 V_J1850
 Wire Wire Line
-	7850 1500 7850 1250
-$Comp
-L Q_NMOS_DGS Q4
-U 1 1 5AFD6A72
-P 8350 1550
-F 0 "Q4" V 8600 1600 50  0000 L CNN
-F 1 "RSU002P03" V 8600 1100 50  0000 L CNN
-F 2 "" H 8550 1650 50  0001 C CNN
-F 3 "" H 8350 1550 50  0001 C CNN
-	1    8350 1550
-	0    -1   -1   0
-$EndComp
+	7850 1250 7850 1500
 Wire Wire Line
 	7850 1450 8150 1450
@@
 	7450 5050 7700 5050
 Wire Wire Line
-	8000 4850 8000 4650
+	8000 4650 8000 4850
 Wire Wire Line
 	8000 4350 8000 4200
@@
 Wire Wire Line
 	4500 5350 4500 5450
+Wire Wire Line
+	4250 2300 4350 2300
+$Comp
+L 2N7002 Q1
+U 1 1 5AFD20A7
+P 4550 2300
+AR Path="/5AFD20A7" Ref="Q1"  Part="1"
+AR Path="/5AFB6308/5AFD20A7" Ref="Q1"  Part="1"
+F 0 "Q1" H 4750 2375 50  0000 L CNN
+F 1 "2N7002" H 4500 2050 50  0000 L CNN
+F 2 "TO_SOT_Packages_SMD:SOT-23" H 4750 2225 50  0001 L CIN
+F 3 "" H 4550 2300 50  0001 L CNN
+	1    4550 2300
+	1    0    0    -1
+$EndComp
+Wire Wire Line
+	7550 2200 7550 2150
+$Comp
+L Q_PMOS_SGD Q4
+U 1 1 5B2CE066
+P 8350 1550
+F 0 "Q4" H 8550 1600 50  0000 L CNN
+F 1 "RSU002P03" H 8550 1500 50  0000 L CNN
+F 2 "" H 8550 1650 50  0001 C CNN
+F 3 "" H 8350 1550 50  0001 C CNN
+	1    8350 1550
+	0    1    -1   0
+$EndComp
 $EndSCHEMATC

Commit message: Esto es un comentario escrito en una consola
Connections:
- net +5V: no longer U1.3 (V+), U1.3 (V+)
- net VCC: now also U1.3 (V+), U1.3 (V+)
Changed lines of the file:
@@
 Text Notes 8450 5200 0    60   ~ 0
 EL ARDU USA \nMBT2222
-$Comp
-L +5V #PWR041
-U 1 1 5B231989
-P 4500 5350
-F 0 "#PWR041" H 4500 5200 50  0001 C CNN
-F 1 "+5V" H 4500 5490 50  0000 C CNN
-F 2 "" H 4500 5350 50  0001 C CNN
-F 3 "" H 4500 5350 50  0001 C CNN
-	1    4500 5350
-	1    0    0    -1
-$EndComp
-$Comp
-L +5V #PWR042
-U 1 1 5B2319E8
-P 4500 4150
-F 0 "#PWR042" H 4500 4000 50  0001 C CNN
-F 1 "+5V" H 4500 4290 50  0000 C CNN
-F 2 "" H 4500 4150 50  0001 C CNN
-F 3 "" H 4500 4150 50  0001 C CNN
-	1    4500 4150
-	1    0    0    -1
-$EndComp
 NoConn ~ 2000 1800
 NoConn ~ 1600 1500
@@
 	0    1    -1   0
 $EndComp
+$Comp
+L VCC #PWR?
+U 1 1 5B30334A
+P 4500 4150
+F 0 "#PWR?" H 4500 4000 50  0001 C CNN
+F 1 "VCC" H 4500 4300 50  0000 C CNN
+F 2 "" H 4500 4150 50  0001 C CNN
+F 3 "" H 4500 4150 50  0001 C CNN
+	1    4500 4150
+	1    0    0    -1
+$EndComp
+$Comp
+L VCC #PWR?
+U 1 1 5B3043A1
+P 4500 5350
+F 0 "#PWR?" H 4500 5200 50  0001 C CNN
+F 1 "VCC" H 4500 5500 50  0000 C CNN
+F 2 "" H 4500 5350 50  0001 C CNN
+F 3 "" H 4500 5350 50  0001 C CNN
+	1    4500 5350
+	1    0    0    -1
+$EndComp
 $EndSCHEMATC

Commit message: added some footprints
Parts:
- D3, D4, D5: value BAT46 -> BAT46W-7-F
Changed lines of the file:
@@
 LIBS:stn2120
 LIBS:switches
-LIBS:PF_APINER-cache
 EELAYER 25 0
 EELAYER END
@@
 P 9000 1450
 F 0 "D4" H 9000 1550 50  0000 C CNN
-F 1 "BAT46" H 9000 1350 50  0000 C CNN
+F 1 "BAT46W-7-F" H 9000 1350 50  0000 C CNN
 F 2 "" H 9000 1450 50  0001 C CNN
 F 3 "" H 9000 1450 50  0001 C CNN
@@
 P 9350 2100
 F 0 "D5" V 9350 2200 50  0000 C CNN
-F 1 "BAT46" V 9350 1900 50  0000 C CNN
+F 1 "BAT46W-7-F" V 9200 1850 50  0000 C CNN
 F 2 "" H 9350 2100 50  0001 C CNN
 F 3 "" H 9350 2100 50  0001 C CNN
@@
 P 8000 4050
 F 0 "D3" V 8000 4150 50  0000 C CNN
-F 1 "BAT46" V 8000 3850 50  0000 C CNN
+F 1 "BAT46W-7-F" V 7850 4050 50  0000 C CNN
 F 2 "" H 8000 4050 50  0001 C CNN
 F 3 "" H 8000 4050 50  0001 C CNN
@@
 $EndComp
 $Comp
-L VCC #PWR?
+L VCC #PWR041
 U 1 1 5B30334A
 P 4500 4150
-F 0 "#PWR?" H 4500 4000 50  0001 C CNN
+F 0 "#PWR041" H 4500 4000 50  0001 C CNN
 F 1 "VCC" H 4500 4300 50  0000 C CNN
 F 2 "" H 4500 4150 50  0001 C CNN
@@
 $EndComp
 $Comp
-L VCC #PWR?
+L VCC #PWR042
 U 1 1 5B3043A1
 P 4500 5350
-F 0 "#PWR?" H 4500 5200 50  0001 C CNN
+F 0 "#PWR042" H 4500 5200 50  0001 C CNN
 F 1 "VCC" H 4500 5500 50  0000 C CNN
 F 2 "" H 4500 5350 50  0001 C CNN
