File: KiCad Proyecto/K_L_LINE.sch (KiCad schematic (older format))
At the start: 11 parts, among them Q5 3904, Q6 3904, U1 LM339

Commit message: Esto es un comentario escrito en una consola
Connections:
- net GND: now also U1.12 (V-)
- net VCC: now also U1.3 (V+)
Changed lines of the file:
@@
 Wire Wire Line
 	4100 4400 4250 4400
+$Comp
+L VCC #PWR?
+U 1 1 5B2BCFD5
+P 3700 2600
+F 0 "#PWR?" H 3700 2450 50  0001 C CNN
+F 1 "VCC" H 3700 2750 50  0000 C CNN
+F 2 "" H 3700 2600 50  0001 C CNN
+F 3 "" H 3700 2600 50  0001 C CNN
+	1    3700 2600
+	1    0    0    -1
+$EndComp
+$Comp
+L GND #PWR?
+U 1 1 5B2BD001
+P 3700 3400
+F 0 "#PWR?" H 3700 3150 50  0001 C CNN
+F 1 "GND" H 3700 3250 50  0000 C CNN
+F 2 "" H 3700 3400 50  0001 C CNN
+F 3 "" H 3700 3400 50  0001 C CNN
+	1    3700 3400
+	1    0    0    -1
+$EndComp
+Wire Wire Line
+	3700 2700 3700 2600
+Wire Wire Line
+	3700 3300 3700 3400
 $EndSCHEMATC
