File: KiCad Proyecto/STN2120.sch (KiCad schematic (older format))
At the start: 27 parts, among them Y1 16MHz

Commit message: Esto es un comentario escrito en una consola
Parts:
- stn1: value stn2220 -> stn2120
Connections:
- net +3V3: now also R34.1
- net +5V: no longer R34.1
- net SW_CAN_MODE0: now also R42.2, stn1.35 (SW_CAN_MODE0); no longer R40.2, stn1.36 (SW_CAN_MODE1)
- net SW_CAN_MODE1: now also R40.2, stn1.36 (SW_CAN_MODE1); no longer R42.2, stn1.35 (SW_CAN_MODE0)
Other:
- note removed: "UART TX es 5v tolerant\nsacar 3.3V y pull-up?"
Changed lines of the file:
@@
 P 5450 3450
 F 0 "stn1" H 5450 1700 60  0000 C CNN
-F 1 "stn2220" H 5450 4650 60  0000 C CNN
+F 1 "stn2120" H 5450 4650 60  0000 C CNN
 F 2 "" H 7700 2450 60  0001 C CNN
 F 3 "" H 7700 2450 60  0001 C CNN
@@
 Text HLabel 7950 4550 2    60   Input ~ 0
 SW_CAN_RX
+Text HLabel 7950 4800 2    60   Output ~ 0
+SW_CAN_MODE0
 Text HLabel 7950 4700 2    60   Output ~ 0
-SW_CAN_MODE0
-Text HLabel 7950 4800 2    60   Output ~ 0
 SW_CAN_MODE1
 Text HLabel 6350 4900 2    60   Output ~ 0
@@
 Wire Wire Line
 	3300 5500 3300 5250
-Text Notes 5850 1600 0    60   ~ 0
-UART TX es 5v tolerant\nsacar 3.3V y pull-up?
-$Comp
-L +5V #PWR091
-U 1 1 5B06FB2A
-P 4350 2450
-F 0 "#PWR091" H 4350 2300 50  0001 C CNN
-F 1 "+5V" H 4350 2590 50  0000 C CNN
-F 2 "" H 4350 2450 50  0001 C CNN
-F 3 "" H 4350 2450 50  0001 C CNN
-	1    4350 2450
-	1    0    0    -1
-$EndComp
 Wire Wire Line
 	6200 4550 7950 4550
 Wire Wire Line
-	4550 2450 4700 2450
+	4350 2450 4700 2450
 Connection ~ 4700 2450
 Text HLabel 1600 3650 0    60   UnSpc ~ 0
@@
 	1    0    0    -1
 $EndComp
+Connection ~ 4550 2450
 $EndSCHEMATC

Commit message: added some footprints
Parts:
- stn1: footprint (none) -> Housings_DFN_QFN:QFN-44-1EP_8x8mm_Pitch0.65mm
Changed lines of the file:
@@
 LIBS:stn2120
 LIBS:switches
-LIBS:PF_APINER-cache
 EELAYER 25 0
 EELAYER END
@@
 F 0 "stn1" H 5450 1700 60  0000 C CNN
 F 1 "stn2120" H 5450 4650 60  0000 C CNN
-F 2 "" H 7700 2450 60  0001 C CNN
+F 2 "Housings_DFN_QFN:QFN-44-1EP_8x8mm_Pitch0.65mm" H 7700 2450 60  0001 C CNN
 F 3 "" H 7700 2450 60  0001 C CNN
 	1    5450 3450
@@
 Connection ~ 4700 4950
 $Comp
-L GND #PWR077
+L GND #PWR079
 U 1 1 5AFECC5B
 P 4700 5050
-F 0 "#PWR077" H 4700 4800 50  0001 C CNN
+F 0 "#PWR079" H 4700 4800 50  0001 C CNN
 F 1 "GND" H 4700 4900 50  0000 C CNN
 F 2 "" H 4700 5050 50  0001 C CNN
@@
 Connection ~ 4700 4100
 $Comp
-L GND #PWR078
+L GND #PWR080
 U 1 1 5AFEDC33
 P 4700 4200
-F 0 "#PWR078" H 4700 3950 50  0001 C CNN
+F 0 "#PWR080" H 4700 3950 50  0001 C CNN
 F 1 "GND" H 4700 4050 50  0000 C CNN
 F 2 "" H 4700 4200 50  0001 C CNN
@@
 V_BAT
 $Comp
-L GND #PWR079
+L GND #PWR081
 U 1 1 5AFEDEED
 P 1500 5100
-F 0 "#PWR079" H 1500 4850 50  0001 C CNN
+F 0 "#PWR081" H 1500 4850 50  0001 C CNN
 F 1 "GND" H 1500 4950 50  0000 C CNN
 F 2 "" H 1500 5100 50  0001 C CNN
@@
 Connection ~ 1500 5050
 $Comp
-L +3.3V #PWR080
+L +3.3V #PWR082
 U 1 1 5AFEE0D8
 P 1800 4000
-F 0 "#PWR080" H 1800 3850 50  0001 C CNN
+F 0 "#PWR082" H 1800 3850 50  0001 C CNN
 F 1 "+3.3V" H 1800 4140 50  0000 C CNN
 F 2 "" H 1800 4000 50  0001 C CNN
@@
 	4700 2300 4700 2650
 $Comp
-L +3.3V #PWR081
+L +3.3V #PWR083
 U 1 1 5AFEEB48
 P 4700 2300
-F 0 "#PWR081" H 4700 2150 50  0001 C CNN
+F 0 "#PWR083" H 4700 2150 50  0001 C CNN
 F 1 "+3.3V" H 4700 2440 50  0000 C CNN
 F 2 "" H 4700 2300 50  0001 C CNN
@@
 Connection ~ 4700 2550
 $Comp
-L +3.3V #PWR082
+L +3.3V #PWR084
 U 1 1 5AFEEBBD
 P 3200 2400
-F 0 "#PWR082" H 3200 2250 50  0001 C CNN
+F 0 "#PWR084" H 3200 2250 50  0001 C CNN
 F 1 "+3.3V" H 3200 2540 50  0000 C CNN
 F 2 "" H 3200 2400 50  0001 C CNN
@@
 $EndComp
 $Comp
-L GND #PWR083
+L GND #PWR085
 U 1 1 5AFEED91
 P 3200 2900
-F 0 "#PWR083" H 3200 2650 50  0001 C CNN
+F 0 "#PWR085" H 3200 2650 50  0001 C CNN
 F 1 "GND" H 3200 2750 50  0000 C CNN
 F 2 "" H 3200 2900 50  0001 C CNN
@@
 CADA UNO CERCA DE\nVDD Y AVDD
 $Comp
-L +3.3V #PWR084
+L +3.3V #PWR086
 U 1 1 5AFEF9F2
 P 6500 1900
-F 0 "#PWR084" H 6500 1750 50  0001 C CNN
+F 0 "#PWR086" H 6500 1750 50  0001 C CNN
 F 1 "+3.3V" H 6500 2040 50  0000 C CNN
 F 2 "" H 6500 1900 50  0001 C CNN
@@
 	6200 3200 7950 3200
 $Comp
-L +3.3V #PWR085
+L +3.3V #PWR087
 U 1 1 5AFF0470
 P 7450 2550
-F 0 "#PWR085" H 7450 2400 50  0001 C CNN
+F 0 "#PWR087" H 7450 2400 50  0001 C CNN
 F 1 "+3.3V" H 7450 2690 50  0000 C CNN
 F 2 "" H 7450 2550 50  0001 C CNN
@@
 $EndComp
 $Comp
-L GND #PWR086
+L GND #PWR088
 U 1 1 5AFF10BE
 P 3550 3550
-F 0 "#PWR086" H 3550 3300 50  0001 C CNN
+F 0 "#PWR088" H 3550 3300 50  0001 C CNN
 F 1 "GND" H 3550 3400 50  0000 C CNN
 F 2 "" H 3550 3550 50  0001 C CNN
@@
 $EndComp
 $Comp
-L GND #PWR087
+L GND #PWR089
 U 1 1 5AFF2AD6
 P 4150 4150
-F 0 "#PWR087" H 4150 3900 50  0001 C CNN
+F 0 "#PWR089" H 4150 3900 50  0001 C CNN
 F 1 "GND" H 4150 4000 50  0000 C CNN
 F 2 "" H 4150 4150 50  0001 C CNN
@@
 	6200 4300 6350 4300
 $Comp
-L +5V #PWR088
+L +5V #PWR090
 U 1 1 5AFF3AE9
 P 7450 3950
-F 0 "#PWR088" H 7450 3800 50  0001 C CNN
+F 0 "#PWR090" H 7450 3800 50  0001 C CNN
 F 1 "+5V" H 7450 4090 50  0000 C CNN
 F 2 "" H 7450 3950 50  0001 C CNN
@@
 $EndComp
 $Comp
-L GND #PWR089
+L GND #PWR091
 U 1 1 5AFF83AD
 P 2850 5200
-F 0 "#PWR089" H 2850 4950 50  0001 C CNN
+F 0 "#PWR091" H 2850 4950 50  0001 C CNN
 F 1 "GND" H 2850 5050 50  0000 C CNN
 F 2 "" H 2850 5200 50  0001 C CNN
@@
 $EndComp
 $Comp
-L +3.3V #PWR090
+L +3.3V #PWR092
 U 1 1 5AFF8EED
 P 3300 4350
-F 0 "#PWR090" H 3300 4200 50  0001 C CNN
+F 0 "#PWR092" H 3300 4200 50  0001 C CNN
 F 1 "+3.3V" H 3300 4490 50  0000 C CNN
 F 2 "" H 3300 4350 50  0001 C CNN
@@
 	1850 3650 1600 3650
 $Comp
-L +3.3V #PWR092
+L +3.3V #PWR093
 U 1 1 5AFEDBC0
 P 1850 3650
-F 0 "#PWR092" H 1850 3500 50  0001 C CNN
+F 0 "#PWR093" H 1850 3500 50  0001 C CNN
 F 1 "+3.3V" H 1850 3790 50  0000 C CNN
 F 2 "" H 1850 3650 50  0001 C CNN
@@
 $EndComp
 $Comp
-L +5V #PWR093
+L +5V #PWR094
 U 1 1 5AFEDBAA
 P 1850 3350
-F 0 "#PWR093" H 1850 3200 50  0001 C CNN
+F 0 "#PWR094" H 1850 3200 50  0001 C CNN
 F 1 "+5V" H 1850 3490 50  0000 C CNN
 F 2 "" H 1850 3350 50  0001 C CNN
@@
 	1600 3100 1850 3100
 $Comp
-L VCC #PWR094
+L VCC #PWR095
 U 1 1 5AFEDB94
 P 1850 3100
-F 0 "#PWR094" H 1850 2950 50  0001 C CNN
+F 0 "#PWR095" H 1850 2950 50  0001 C CNN
 F 1 "VCC" H 1850 3250 50  0000 C CNN
 F 2 "" H 1850 3100 50  0001 C CNN
