File: KiCad Proyecto/PF_apiner.sch (KiCad schematic (older format))
At the start: 9 parts, among them J1 OBDII Header, J2 Conn_01x05, U11 AZ1117EH-3.3TRG1, U12 +5V_USB, U13 +5V_USB

Commit message: fixed(temp) library problem
Parts:
- C34, C35: symbol OBDII_IoT:C -> C
- D11, D12: symbol OBDII_IoT:D_Schot -> D_Schot
- J1: symbol OBDII_IoT:CONN_2X16_OBDII -> CONN_2X16_OBDII
- J2: symbol Connector:Conn_01x05 -> Conn_01x05
- U11: symbol OBDII_IoT:VOLT_REG -> VOLT_REG
- U12, U13: symbol OBDII_IoT:+5V_USB -> +5V_USB
Changed lines of the file:
@@
 EESchema Schematic File Version 2
-LIBS:power
-LIBS:PF_apiner-cache
+LIBS:OBDII_IoT
+LIBS:Connector
+LIBS:ESP32-footprints-Shem-Lib
+LIBS:ftdi
+LIBS:STN2120
 EELAYER 25 0
 EELAYER END
@@
 	12150 9650 12250 9750
 $Comp
-L OBDII_IoT:GND #PWR01
+L GND #PWR01
 U 1 1 58F8F97A
 P 1550 4150
@@
 $EndComp
 $Comp
-L OBDII_IoT:CONN_2X16_OBDII J1
+L CONN_2X16_OBDII J1
 U 1 1 58F8F983
 P 1250 3350
@@
 $EndSheet
 $Comp
-L OBDII_IoT:VIN #PWR02
+L VIN #PWR02
 U 1 1 58F9B79D
 P 1550 2550
@@
 El UART0 va al USB, el resto hay que configurarlos
 $Comp
-L Connector:Conn_01x05 J2
+L Conn_01x05 J2
 U 1 1 5B87BBB6
 P 9200 2700
@@
 $EndComp
 $Comp
-L OBDII_IoT:C C?
+L C C?
 U 1 1 5B8838EA
 P 10000 1800
@@
 $EndComp
 $Comp
-L OBDII_IoT:VOLT_REG U?
+L VOLT_REG U?
 U 1 1 5B8838F5
 P 9550 1550
@@
 $EndComp
 $Comp
-L OBDII_IoT:C C?
+L C C?
 U 1 1 5B883906
 P 9050 1800
@@
 $EndComp
 $Comp
-L OBDII_IoT:+3.3V #PWR?
+L +3.3V #PWR?
 U 1 1 5B88390D
 P 8500 1450
@@
 $EndComp
 $Comp
-L OBDII_IoT:GND #PWR?
+L GND #PWR?
 U 1 1 5B883913
 P 9550 2050
@@
 $EndComp
 $Comp
-L OBDII_IoT:GND #PWR?
+L GND #PWR?
 U 1 1 5B883919
 P 10000 2050
@@
 $EndComp
 $Comp
-L OBDII_IoT:GND #PWR?
+L GND #PWR?
 U 1 1 5B88391F
 P 9050 2050
@@
 	8950 1550 9100 1550
 $Comp
-L OBDII_IoT:+5V_USB U12
+L +5V_USB U12
 U 1 1 5B88F65F
 P 8900 2400
@@
 Connection ~ 9050 1550
 $Comp
-L OBDII_IoT:+5V #PWR?
+L +5V #PWR?
 U 1 1 5B8A5F5E
 P 10000 1450
@@
 	10650 1550 10650 1450
 $Comp
-L OBDII_IoT:+5V_USB U?
+L +5V_USB U?
 U 1 1 5B8A5F68
 P 10650 1450
@@
 	8500 1550 8750 1550
 $Comp
-L OBDII_IoT:D_Schot D?
+L D_Schot D?
 U 1 1 5B8B67B7
 P 8850 1550
@@
 $EndComp
 $Comp
-L OBDII_IoT:GND #PWR?
+L GND #PWR?
 U 1 1 5B8BA0D1
 P 8900 3050
@@
 	8550 2900 8250 2900
 $Comp
-L OBDII_IoT:D_Schot D?
+L D_Schot D?
 U 1 1 5B8CB262
 P 10350 1550

Commit message: added dual row smd header and 3.3V
Parts:
- removed J2: Conn_01x05, symbol Conn_01x05
- added J?: Conn_01x06, symbol Conn_01x06
- added U? (x2): +3.3V_USB, symbol +3.3V_USB
Connections:
- wire segments 113 -> 115
Other:
- moved on the sheet: C34, C35

Commit message: un cambio que no me acuerdo
Parts:
- D11, D12: footprint (none) -> to-sod-sot:SOD-123
- gave numbers to parts that had none: 3
Changed lines of the file:
@@
 F 0 "D11" H 8800 4430 50  0000 L CNN
 F 1 "MBR0520" H 8730 4250 40  0000 L CNN
-F 2 "" V 8850 4350 50  0000 C CNN
+F 2 "to-sod-sot:SOD-123" V 8850 4350 50  0001 C CNN
 F 3 "" V 8850 4350 50  0000 C CNN
 F 4 "DIODE SCHOTTKY 20V 500MA SOD123" H 8850 4350 50  0001 C CNN "Desc"
@@
 F 0 "D12" H 10300 4430 50  0000 L CNN
 F 1 "MBR0520" H 10230 4250 40  0000 L CNN
-F 2 "" V 10350 4350 50  0000 C CNN
+F 2 "to-sod-sot:SOD-123" V 10350 4350 50  0001 C CNN
 F 3 "" V 10350 4350 50  0000 C CNN
 F 4 "DIODE SCHOTTKY 20V 500MA SOD123" H 10350 4350 50  0001 C CNN "Desc"
@@
 poner schotky de proteccion por el USB?\nen 5V y 3.3V
 $Comp
-L Conn_01x06 J?
+L Conn_01x06 J2
 U 1 1 5B8EE09D
 P 9550 2600
-F 0 "J?" H 9550 2900 50  0000 C CNN
+F 0 "J2" H 9550 2900 50  0000 C CNN
 F 1 "Conn_01x06" H 9550 2200 50  0000 C CNN
 F 2 "" H 9550 2600 50  0001 C CNN
@@
 $EndComp
 $Comp
-L +3.3V_USB U?
+L +3.3V_USB U15
 U 1 1 5B8FA255
 P 9000 2350
-F 0 "U?" H 9000 2500 50  0001 C CNN
+F 0 "U15" H 9000 2500 50  0001 C CNN
 F 1 "+3.3V_USB" H 9000 2450 30  0000 C CNN
 F 2 "" H 9000 2350 50  0001 C CNN
@@
 	9000 2500 9350 2500
 $Comp
-L +3.3V_USB U?
+L +3.3V_USB U16
 U 1 1 5B8FDAFC
 P 9050 4200
-F 0 "U?" H 9050 4350 50  0001 C CNN
+F 0 "U16" H 9050 4350 50  0001 C CNN
 F 1 "+3.3V_USB" H 9050 4300 30  0000 C CNN
 F 2 "" H 9050 4200 50  0001 C CNN

Commit message: added last footprint
Parts:
- J2: value Conn_01x06 -> Conn_02x03; footprint (none) -> conn:Pin_Header_Straight_2x3_SMD; Desc CONN RECEPT 6POS DUAL SMD -> CONN RECEPT 6POS 2MM VERT SMD; Digikey# 609-3704-1-ND -> WM18698-ND; Manf Amphenol FCI -> Molex Connector Corporation; Manf# 20021321-00006C4LF -> 79109-1002
Changed lines of the file:
@@
 LIBS:ftdi
 LIBS:STN2120
+LIBS:PF_apiner-cache
 EELAYER 25 0
 EELAYER END
@@
 P 9550 2600
 F 0 "J2" H 9550 2900 50  0000 C CNN
-F 1 "Conn_01x06" H 9550 2200 50  0000 C CNN
-F 2 "" H 9550 2600 50  0001 C CNN
+F 1 "Conn_02x03" H 9550 2200 50  0000 C CNN
+F 2 "conn:Pin_Header_Straight_2x3_SMD" H 9550 2600 50  0001 C CNN
 F 3 "" H 9550 2600 50  0001 C CNN
-F 4 "CONN RECEPT 6POS DUAL SMD" H 9550 2600 60  0001 C CNN "Desc"
-F 5 "Amphenol FCI" H 9550 2600 60  0001 C CNN "Manf"
-F 6 "20021321-00006C4LF" H 9550 2600 60  0001 C CNN "Manf#"
-F 7 "609-3704-1-ND" H 9550 2600 60  0001 C CNN "Digikey#"
+F 4 "CONN RECEPT 6POS 2MM VERT SMD" H 9550 2600 60  0001 C CNN "Desc"
+F 5 "Molex Connector Corporation" H 9550 2600 60  0001 C CNN "Manf"
+F 6 "79109-1002" H 9550 2600 60  0001 C CNN "Manf#"
+F 7 "WM18698-ND" H 9550 2600 60  0001 C CNN "Digikey#"
 	1    9550 2600
 	1    0    0    -1

Commit message: arreglando manquiadas
Other:
- note added: "Agrandar D1 y cambiar fusible"
Changed lines of the file:
@@
 EESchema Schematic File Version 2
-LIBS:OBDII_IoT
 LIBS:Connector
 LIBS:ESP32-footprints-Shem-Lib
 LIBS:ftdi
+LIBS:OBDII_IoT
 LIBS:STN2120
 LIBS:PF_apiner-cache
@@
 Wire Wire Line
 	9050 4200 9050 4450
+Text Notes 5100 1100 0    60   ~ 0
+Agrandar D1 y cambiar fusible
 $EndSCHEMATC

Commit message: cambios boludos
Connections:
- wire segments 115 -> 116
Changed lines of the file:
@@
 Text Notes 5100 1100 0    60   ~ 0
 Agrandar D1 y cambiar fusible
+$Comp
+L PWR_FLAG #FLG?
+U 1 1 5BA598FF
+P 9350 2200
+F 0 "#FLG?" H 9350 2295 50  0001 C CNN
+F 1 "PWR_FLAG" H 9350 2380 40  0000 C CNN
+F 2 "" H 9350 2200 50  0000 C CNN
+F 3 "" H 9350 2200 50  0000 C CNN
+	1    9350 2200
+	1    0    0    -1
+$EndComp
+Wire Wire Line
+	9350 2400 9350 2200
 $EndSCHEMATC

Commit message: fixed fuse & wrong fields
Parts:
- C34: Desc (none) -> CAP CER 1UF 6.3V X5R 0402; Descripcion CAP CER 1UF 6.3V X5R 0402 -> (none); Digikey# (none) -> 587-1231-1-ND; Digikey/Mouser 587-1231-1-ND -> (none); Fabricante Taiyo Yuden -> (none); Manf (none) -> Taiyo Yuden; Manf# (none) -> JMK105BJ105KV-F; Nro. parte JMK105BJ105KV-F -> (none)
- C35: Desc (none) -> CAP CER 0.1UF 10V X5R 0402; Descripcion CAP CER 0.1UF 10V X5R 0402 -> (none); Digikey# (none) -> 311-1336-1-ND; Digikey/Mouser 311-1336-1-ND -> (none); Fabricante Yageo -> (none); Manf (none) -> Yageo; Manf# (none) -> CC0402KRX5R6BB104; Nro. parte CC0402KRX5R6BB104 -> (none)
- J1: Desc (none) -> OBDII male 90° connector; Descripcion OBDII male 90° connector -> (none); Fabricante Yeahui -> (none); Manf (none) -> Yeahui; Manf# (none) -> YH1012; Nro. parte YH1012 -> (none)
- U11: Desc (none) -> IC REG LDO 3.3V 1A SOT223; Descripcion IC REG LDO 3.3V 1A SOT223 -> (none); Digikey# (none) -> AZ1117EH-3.3TRG1DICT-ND; Digikey/Mouser AZ1117EH-3.3TRG1DICT-ND -> (none); Fabricante Diodes Incorporated -> (none); Manf (none) -> Diodes Incorporated; Manf# (none) -> AZ1117EH-3.3TRG1; Nro. parte AZ1117EH-3.3TRG1 -> (none)
Changed lines of the file:
@@
 F 2 "conn:YH1012" H 1250 3750 50  0001 C CNN
 F 3 "" H 1250 3750 50  0000 C CNN
-F 4 "OBDII male 90° connector" H 1250 3350 60  0001 C CNN "Descripcion"
-F 5 "Yeahui" H 1250 3350 60  0001 C CNN "Fabricante"
-F 6 "YH1012" H 1250 3350 60  0001 C CNN "Nro. parte"
+F 4 "OBDII male 90° connector" H 1250 3350 60  0001 C CNN "Desc"
+F 5 "Yeahui" H 1250 3350 60  0001 C CNN "Manf"
+F 6 "YH1012" H 1250 3350 60  0001 C CNN "Manf#"
 	1    1250 3350
 	-1   0    0    1
@@
 F 2 "chip_rlc:c_0402" H 10038 4450 50  0001 C CNN
 F 3 "" H 10000 4600 50  0000 C CNN
-F 4 "CAP CER 0.1UF 10V X5R 0402" H 10000 4600 60  0001 C CNN "Descripcion"
-F 5 "Yageo" H 10000 4600 60  0001 C CNN "Fabricante"
-F 6 "CC0402KRX5R6BB104" H 10000 4600 60  0001 C CNN "Nro. parte"
-F 7 "311-1336-1-ND" H 10000 4600 60  0001 C CNN "Digikey/Mouser"
+F 4 "CAP CER 0.1UF 10V X5R 0402" H 10000 4600 60  0001 C CNN "Desc"
+F 5 "Yageo" H 10000 4600 60  0001 C CNN "Manf"
+F 6 "CC0402KRX5R6BB104" H 10000 4600 60  0001 C CNN "Manf#"
+F 7 "311-1336-1-ND" H 10000 4600 60  0001 C CNN "Digikey#"
 	1    10000 4600
 	-1   0    0    -1
@@
 F 2 "to-sod-sot:SOT-223" H 2000 -850 40  0001 C CNN
 F 3 "" H 2000 -850 40  0000 C CNN
-F 4 "IC REG LDO 3.3V 1A SOT223" H 9550 4350 60  0001 C CNN "Descripcion"
-F 5 "Diodes Incorporated" H 9550 4350 60  0001 C CNN "Fabricante"
-F 6 "AZ1117EH-3.3TRG1" H 9550 4350 60  0001 C CNN "Nro. parte"
-F 7 "AZ1117EH-3.3TRG1DICT-ND" H 9550 4350 60  0001 C CNN "Digikey/Mouser"
+F 4 "IC REG LDO 3.3V 1A SOT223" H 9550 4350 60  0001 C CNN "Desc"
+F 5 "Diodes Incorporated" H 9550 4350 60  0001 C CNN "Manf"
+F 6 "AZ1117EH-3.3TRG1" H 9550 4350 60  0001 C CNN "Manf#"
+F 7 "AZ1117EH-3.3TRG1DICT-ND" H 9550 4350 60  0001 C CNN "Digikey#"
 	1    9550 4350
 	-1   0    0    -1
@@
 F 2 "chip_rlc:c_0402" H 9088 4450 50  0001 C CNN
 F 3 "" H 9050 4600 50  0000 C CNN
-F 4 "CAP CER 1UF 6.3V X5R 0402" H 9050 4600 60  0001 C CNN "Descripcion"
-F 5 "Taiyo Yuden" H 9050 4600 60  0001 C CNN "Fabricante"
-F 6 "JMK105BJ105KV-F" H 9050 4600 60  0001 C CNN "Nro. parte"
-F 7 "587-1231-1-ND" H 9050 4600 60  0001 C CNN "Digikey/Mouser"
+F 4 "CAP CER 1UF 6.3V X5R 0402" H 9050 4600 60  0001 C CNN "Desc"
+F 5 "Taiyo Yuden" H 9050 4600 60  0001 C CNN "Manf"
+F 6 "JMK105BJ105KV-F" H 9050 4600 60  0001 C CNN "Manf#"
+F 7 "587-1231-1-ND" H 9050 4600 60  0001 C CNN "Digikey#"
 	1    9050 4600
 	-1   0    0    -1
