File: KiCad Proyecto/MicroM4.sch (KiCad schematic (older format))
At the start: 6 parts, among them U14 ESP32-WROOM

Commit message: fixed(temp) library problem
Parts:
- C36, C37, C38: symbol OBDII_IoT:C -> C
- R52, R53: symbol OBDII_IoT:R -> R
- U14: symbol ESP32-footprints-Shem-Lib:ESP32-WROOM -> ESP32-WROOM
Changed lines of the file:
@@
 EESchema Schematic File Version 2
-LIBS:power
-LIBS:PF_apiner-cache
+LIBS:OBDII_IoT
+LIBS:Connector
+LIBS:ESP32-footprints-Shem-Lib
+LIBS:ftdi
+LIBS:STN2120
 EELAYER 25 0
 EELAYER END
@@
 $EndDescr
 $Comp
-L ESP32-footprints-Shem-Lib:ESP32-WROOM U14
+L ESP32-WROOM U14
 U 1 1 5B862489
 P 5650 3400
@@
 $EndComp
 $Comp
-L OBDII_IoT:+3.3V #PWR0120
+L +3.3V #PWR0120
 U 1 1 5B862539
 P 4600 2600
@@
 NoConn ~ 6550 3150
 $Comp
-L OBDII_IoT:GND #PWR0121
+L GND #PWR0121
 U 1 1 5B862710
 P 6750 4100
@@
 Connection ~ 6550 4050
 $Comp
-L OBDII_IoT:GND #PWR0122
+L GND #PWR0122
 U 1 1 5B86275E
 P 5200 4550
@@
 $EndComp
 $Comp
-L OBDII_IoT:GND #PWR0123
+L GND #PWR0123
 U 1 1 5B86276B
 P 4600 4150
@@
 	3600 2450 4000 2450
 $Comp
-L OBDII_IoT:GND #PWR0124
+L GND #PWR0124
 U 1 1 5B862FB4
 P 3800 2450
@@
 	3600 2150 4000 2150
 $Comp
-L OBDII_IoT:+3.3V #PWR0125
+L +3.3V #PWR0125
 U 1 1 5B86325C
 P 3800 2150
@@
 Connection ~ 4250 2900
 $Comp
-L OBDII_IoT:GND #PWR0126
+L GND #PWR0126
 U 1 1 5B8638AE
 P 4250 3200
@@
 PAG 10\nGPIO0 -> 0: DOWNLOAD BOOT\nGPIO0 -> 1: SPI BOOT
 $Comp
-L OBDII_IoT:GND #PWR0127
+L GND #PWR0127
 U 1 1 5B87900D
 P 6000 4600
@@
 RESET
 $Comp
-L OBDII_IoT:C C?
+L C C?
 U 1 1 5B8CBC06
 P 4000 2300
@@
 $EndComp
 $Comp
-L OBDII_IoT:C C?
+L C C?
 U 1 1 5B8CBF7F
 P 4250 3050
@@
 $EndComp
 $Comp
-L OBDII_IoT:R R?
+L R R?
 U 1 1 5B8D142E
 P 6750 2500
@@
 $EndComp
 $Comp
-L OBDII_IoT:+3.3V #PWR?
+L +3.3V #PWR?
 U 1 1 5B8D1435
 P 6750 2300
@@
 Connection ~ 6750 2850
 $Comp
-L OBDII_IoT:C C?
+L C C?
 U 1 1 5B8D3E2F
 P 3600 2300
@@
 $EndComp
 $Comp
-L OBDII_IoT:R R?
+L R R?
 U 1 1 5B8D4B64
 P 4250 2750

Commit message: added dual row smd header and 3.3V
Connections:
- wire segments 22 -> 24
- no-connect marks 23 -> 22
Other:
- note added: "PAG 10\nGPIO 0 -> 0: DOWNLOAD BOOT\nGPIO 0 -> 1: SPI BOOT"
- note removed: "PAG 10\nGPIO0 -> 0: DOWNLOAD BOOT\nGPIO0 -> 1: SPI BOOT"
Changed lines of the file:
@@
 Connection ~ 6550 3950
 Text Notes 7400 4050 0    50   ~ 0
-PAG 10\nGPIO0 -> 0: DOWNLOAD BOOT\nGPIO0 -> 1: SPI BOOT
+PAG 10\nGPIO 0 -> 0: DOWNLOAD BOOT\nGPIO 0 -> 1: SPI BOOT
 $Comp
 L GND #PWR0127
@@
 NoConn ~ 5800 4450
 NoConn ~ 5900 4450
-NoConn ~ 6100 4450
 NoConn ~ 6550 3750
 NoConn ~ 6550 3450
@@
 Text Notes 4400 1900 0    60   ~ 0
 Both ESP32-WROOM-32D and ESP32-WROOM-32U integrate a 4 MB of external SPI flash. The integrated SPI\nflash is connected to GPIO6, GPIO7, GPIO8, GPIO9, GPIO10 and GPIO11. These six pins cannot be used as\nregular GPIOs.
+Wire Wire Line
+	6000 4500 6100 4500
+Wire Wire Line
+	6100 4500 6100 4450
+Connection ~ 6000 4500
 $EndSCHEMATC

Commit message: arreglando manquiadas
Parts:
- removed R53: 1K, chip_rlc:r_0402, symbol R
- added R?: 0, symbol R
- added R?: 100K, symbol R
- added SW? (x2): SW_SPST, symbol SW_SPST
Connections:
- wire segments 24 -> 38
Other:
- note added: "PAG 10\nGPIO15 -> MTDO-> 0 -> U0TXD Silent\ndejarlo sin soldar la resistencia y despues poner una de 0 ohm"
- note added: "PAG 10\npull-up interno\nGPIO 0 -> 0: DOWNLOAD BOOT\nGPIO 0 -> 1: SPI BOOT"
- note removed: "Both ESP32-WROOM-32D and ESP32-WROOM-32U integrate a 4 MB of external SPI flash. The integrated SPI\nflash is connected to GPIO6, GPIO7, GPIO8, GPIO9, GPIO10 and GPIO11. These six pins cannot be used as\nregular GPIOs."
- note removed: "PAG 10\nGPIO 0 -> 0: DOWNLOAD BOOT\nGPIO 0 -> 1: SPI BOOT"
- note removed: "PAG 10\nGPIO15 -> MTDO-> 0 -> U0TXD Silent"
- moved on the sheet: C38, R52

Commit message: cambios boludos
Parts:
- removed R?: 0, symbol R
- SW?: value SW_SPST -> SW_BOOT; footprint (none) -> misc:TACT_SMD_4.5X4.5
- SW?: value SW_SPST -> SW_RESET; footprint (none) -> misc:TACT_SMD_4.5X4.5
Connections:
- wire segments 38 -> 36
Changed lines of the file:
@@
 Connection ~ 6750 4050
-$Comp
-L R R?
-U 1 1 5B9BDF3D
-P 6000 4700
-F 0 "R?" V 6080 4700 50  0000 C CNN
-F 1 "0" V 6000 4700 50  0000 C CNN
-F 2 "" V 5930 4700 50  0000 C CNN
-F 3 "" H 6000 4700 50  0000 C CNN
-F 4 "RES SMD 100K OHM 1% 1/10W 0402" H 6000 4700 60  0001 C CNN "Desc"
-F 5 "Vishay Beyschlag" H 6000 4700 60  0001 C CNN "Manf"
-F 6 "MCS04020C1003FE000" H 6000 4700 60  0001 C CNN "Manf#"
-F 7 "MCS0402-100K-CFCT-ND" H 6000 4700 60  0001 C CNN "Digikey#"
-	1    6000 4700
-	1    0    0    -1
-$EndComp
-Wire Wire Line
-	6000 4550 6000 4450
 $Comp
 L GND #PWR?
 U 1 1 5B9BDFD1
-P 6100 4950
-F 0 "#PWR?" H 6100 4700 50  0001 C CNN
-F 1 "GND" H 6105 4777 50  0001 C CNN
-F 2 "" H 6100 4950 50  0000 C CNN
-F 3 "" H 6100 4950 50  0000 C CNN
-	1    6100 4950
+P 6100 4600
+F 0 "#PWR?" H 6100 4350 50  0001 C CNN
+F 1 "GND" H 6105 4427 50  0001 C CNN
+F 2 "" H 6100 4600 50  0000 C CNN
+F 3 "" H 6100 4600 50  0000 C CNN
+	1    6100 4600
 	1    0    0    -1
 $EndComp
-Wire Wire Line
-	6100 4450 6100 4950
-Wire Wire Line
-	6000 4850 6100 4850
-Connection ~ 6100 4850
 $Comp
 L R R?
@@
 P 7100 4150
 F 0 "SW?" H 7100 4320 50  0000 C CNN
-F 1 "SW_SPST" H 7100 3950 50  0000 C CNN
-F 2 "" H 7100 4150 50  0001 C CNN
+F 1 "SW_BOOT" H 7100 3950 50  0000 C CNN
+F 2 "misc:TACT_SMD_4.5X4.5" H 7100 4150 50  0001 C CNN
 F 3 "" H 7100 4150 50  0001 C CNN
 F 4 "Tactile Switch SPST-NO Top Actuated Surface Mount" H 7100 4150 60  0001 C CNN "Desc"
@@
 P 3450 3250
 F 0 "SW?" H 3450 3420 50  0000 C CNN
-F 1 "SW_SPST" H 3450 3050 50  0000 C CNN
-F 2 "" H 3450 3250 50  0001 C CNN
+F 1 "SW_RESET" H 3450 3050 50  0000 C CNN
+F 2 "misc:TACT_SMD_4.5X4.5" H 3450 3250 50  0001 C CNN
 F 3 "" H 3450 3250 50  0001 C CNN
 F 4 "Tactile Switch SPST-NO Top Actuated Surface Mount" H 3450 3250 60  0001 C CNN "Desc"
@@
 	4250 2950 4250 2900
 Connection ~ 4250 2900
+Wire Wire Line
+	6100 4600 6100 4450
 $EndSCHEMATC

Commit message: fixed fuse & wrong fields
Parts:
- C36: Desc (none) -> CAP CER 10UF 6.3V X5R 0603; Descripcion CAP CER 10UF 6.3V X5R 0603 -> (none); Digikey# (none) -> 587-1256-1-ND; Digikey/Mouser 587-1256-1-ND -> (none); Fabricante Taiyo Yuden -> (none); Manf (none) -> Taiyo Yuden; Manf# (none) -> JMK107BJ106MA-T; Nro. parte JMK107BJ106MA-T -> (none)
- C37, C38: Desc (none) -> CAP CER 0.1UF 10V X5R 0402; Descripcion CAP CER 0.1UF 10V X5R 0402 -> (none); Digikey# (none) -> 311-1336-1-ND; Digikey/Mouser 311-1336-1-ND -> (none); Fabricante Yageo -> (none); Manf (none) -> Yageo; Manf# (none) -> CC0402KRX5R6BB104; Nro. parte CC0402KRX5R6BB104 -> (none)
- R52: Desc (none) -> RES SMD 10K OHM 5% 1/16W 0402; Descripcion RES SMD 10K OHM 5% 1/16W 0402 -> (none); Digikey# (none) -> 311-10KJRCT-ND; Digikey/Mouser 311-10KJRCT-ND -> (none); Fabricante Yageo -> (none); Manf (none) -> Yageo; Manf# (none) -> RC0402JR-0710KL; Nro. parte RC0402JR-0710KL -> (none)
Connections:
- no-connect marks 22 -> 23
Changed lines of the file:
@@
 F 2 "chip_rlc:c_0402" H 4038 2150 50  0001 C CNN
 F 3 "" H 4000 2300 50  0000 C CNN
-F 4 "CAP CER 0.1UF 10V X5R 0402" H 4000 2300 60  0001 C CNN "Descripcion"
-F 5 "Yageo" H 4000 2300 60  0001 C CNN "Fabricante"
-F 6 "CC0402KRX5R6BB104" H 4000 2300 60  0001 C CNN "Nro. parte"
-F 7 "311-1336-1-ND" H 4000 2300 60  0001 C CNN "Digikey/Mouser"
+F 4 "CAP CER 0.1UF 10V X5R 0402" H 4000 2300 60  0001 C CNN "Desc"
+F 5 "Yageo" H 4000 2300 60  0001 C CNN "Manf"
+F 6 "CC0402KRX5R6BB104" H 4000 2300 60  0001 C CNN "Manf#"
+F 7 "311-1336-1-ND" H 4000 2300 60  0001 C CNN "Digikey#"
 	1    4000 2300
 	-1   0    0    -1
@@
 F 2 "chip_rlc:c_0402" H 4288 2950 50  0001 C CNN
 F 3 "" H 4250 3100 50  0000 C CNN
-F 4 "CAP CER 0.1UF 10V X5R 0402" H 4250 3100 60  0001 C CNN "Descripcion"
-F 5 "Yageo" H 4250 3100 60  0001 C CNN "Fabricante"
-F 6 "CC0402KRX5R6BB104" H 4250 3100 60  0001 C CNN "Nro. parte"
-F 7 "311-1336-1-ND" H 4250 3100 60  0001 C CNN "Digikey/Mouser"
+F 4 "CAP CER 0.1UF 10V X5R 0402" H 4250 3100 60  0001 C CNN "Desc"
+F 5 "Yageo" H 4250 3100 60  0001 C CNN "Manf"
+F 6 "CC0402KRX5R6BB104" H 4250 3100 60  0001 C CNN "Manf#"
+F 7 "311-1336-1-ND" H 4250 3100 60  0001 C CNN "Digikey#"
 	1    4250 3100
 	-1   0    0    -1
@@
 F 2 "chip_rlc:c_0603" H 3638 2150 50  0001 C CNN
 F 3 "" H 3600 2300 50  0000 C CNN
-F 4 "CAP CER 10UF 6.3V X5R 0603" H 3600 2300 60  0001 C CNN "Descripcion"
-F 5 "Taiyo Yuden" H 3600 2300 60  0001 C CNN "Fabricante"
-F 6 "JMK107BJ106MA-T" H 3600 2300 60  0001 C CNN "Nro. parte"
-F 7 "587-1256-1-ND" H 3600 2300 60  0001 C CNN "Digikey/Mouser"
+F 4 "CAP CER 10UF 6.3V X5R 0603" H 3600 2300 60  0001 C CNN "Desc"
+F 5 "Taiyo Yuden" H 3600 2300 60  0001 C CNN "Manf"
+F 6 "JMK107BJ106MA-T" H 3600 2300 60  0001 C CNN "Manf#"
+F 7 "587-1256-1-ND" H 3600 2300 60  0001 C CNN "Digikey#"
 	1    3600 2300
 	1    0    0    -1
@@
 F 2 "chip_rlc:r_0402" V 4430 2550 50  0001 C CNN
 F 3 "" H 4500 2550 50  0000 C CNN
-F 4 "Yageo" H 4500 2550 60  0001 C CNN "Fabricante"
-F 5 "RES SMD 10K OHM 5% 1/16W 0402" H 4500 2550 60  0001 C CNN "Descripcion"
-F 6 "RC0402JR-0710KL" H 4500 2550 60  0001 C CNN "Nro. parte"
-F 7 "311-10KJRCT-ND" H 4500 2550 60  0001 C CNN "Digikey/Mouser"
+F 4 "Yageo" H 4500 2550 60  0001 C CNN "Manf"
+F 5 "RES SMD 10K OHM 5% 1/16W 0402" H 4500 2550 60  0001 C CNN "Desc"
+F 6 "RC0402JR-0710KL" H 4500 2550 60  0001 C CNN "Manf#"
+F 7 "311-10KJRCT-ND" H 4500 2550 60  0001 C CNN "Digikey#"
 	1    4500 2550
 	-1   0    0    1
@@
 Wire Wire Line
 	6100 4600 6100 4450
+NoConn ~ 6000 4450
 $EndSCHEMATC

Commit message: wii arrancamos la rev de footprint
Parts:
- R53: renamed from R?; footprint (none) -> chip_rlc:l_0402
- gave numbers to parts that had none: 2
Changed lines of the file:
@@
 $EndComp
 $Comp
-L +3.3V #PWR0120
+L +3.3V #PWR0123
 U 1 1 5B862539
 P 4500 2300
-F 0 "#PWR0120" H 4500 2390 20  0001 C CNN
+F 0 "#PWR0123" H 4500 2390 20  0001 C CNN
 F 1 "+3.3V" H 4496 2428 30  0000 C CNN
 F 2 "" H 4500 2300 60  0000 C CNN
@@
 NoConn ~ 6550 3150
 $Comp
-L GND #PWR0121
+L GND #PWR0124
 U 1 1 5B862710
 P 6750 4100
-F 0 "#PWR0121" H 6750 3850 50  0001 C CNN
+F 0 "#PWR0124" H 6750 3850 50  0001 C CNN
 F 1 "GND" H 6755 3927 50  0001 C CNN
 F 2 "" H 6750 4100 50  0000 C CNN
@@
 	6750 3950 6750 4100
 $Comp
-L GND #PWR0122
+L GND #PWR0125
 U 1 1 5B86275E
 P 5200 4550
-F 0 "#PWR0122" H 5200 4300 50  0001 C CNN
+F 0 "#PWR0125" H 5200 4300 50  0001 C CNN
 F 1 "GND" H 5205 4377 50  0001 C CNN
 F 2 "" H 5200 4550 50  0000 C CNN
@@
 $EndComp
 $Comp
-L GND #PWR0123
+L GND #PWR0126
 U 1 1 5B86276B
 P 4600 4150
-F 0 "#PWR0123" H 4600 3900 50  0001 C CNN
+F 0 "#PWR0126" H 4600 3900 50  0001 C CNN
 F 1 "GND" H 4605 3977 50  0001 C CNN
 F 2 "" H 4600 4150 50  0000 C CNN
@@
 	3600 2450 4000 2450
 $Comp
-L GND #PWR0124
+L GND #PWR0127
 U 1 1 5B862FB4
 P 3800 2450
-F 0 "#PWR0124" H 3800 2200 50  0001 C CNN
+F 0 "#PWR0127" H 3800 2200 50  0001 C CNN
 F 1 "GND" H 3805 2277 50  0001 C CNN
 F 2 "" H 3800 2450 50  0000 C CNN
@@
 	3600 2150 4000 2150
 $Comp
-L +3.3V #PWR0125
+L +3.3V #PWR0128
 U 1 1 5B86325C
 P 3800 2150
-F 0 "#PWR0125" H 3800 2240 20  0001 C CNN
+F 0 "#PWR0128" H 3800 2240 20  0001 C CNN
 F 1 "+3.3V" H 3796 2278 30  0000 C CNN
 F 2 "" H 3800 2150 60  0000 C CNN
@@
 	4700 2350 4700 2800
 $Comp
-L GND #PWR0126
+L GND #PWR0129
 U 1 1 5B8638AE
 P 4250 3250
-F 0 "#PWR0126" H 4250 3000 50  0001 C CNN
+F 0 "#PWR0129" H 4250 3000 50  0001 C CNN
 F 1 "GND" H 4255 3077 50  0001 C CNN
 F 2 "" H 4250 3250 50  0000 C CNN
@@
 	6550 3850 7100 3850
 $Comp
-L GND #PWR?
+L GND #PWR0130
 U 1 1 5B9BDD0C
 P 7000 4450
-F 0 "#PWR?" H 7000 4200 50  0001 C CNN
+F 0 "#PWR0130" H 7000 4200 50  0001 C CNN
 F 1 "GND" H 7005 4277 50  0001 C CNN
 F 2 "" H 7000 4450 50  0000 C CNN
@@
 Connection ~ 6750 4050
 $Comp
-L GND #PWR?
+L GND #PWR0131
 U 1 1 5B9BDFD1
 P 6100 4600
-F 0 "#PWR?" H 6100 4350 50  0001 C CNN
+F 0 "#PWR0131" H 6100 4350 50  0001 C CNN
 F 1 "GND" H 6105 4427 50  0001 C CNN
 F 2 "" H 6100 4600 50  0000 C CNN
@@
 $EndComp
 $Comp
-L R R?
+L R R53
 U 1 1 5B9C04A8
 P 6900 2600
-F 0 "R?" V 6980 2600 50  0000 C CNN
+F 0 "R53" V 6980 2600 50  0000 C CNN
 F 1 "100K" V 6900 2600 50  0000 C CNN
-F 2 "" V 6830 2600 50  0000 C CNN
+F 2 "chip_rlc:l_0402" V 6830 2600 50  0001 C CNN
 F 3 "" H 6900 2600 50  0000 C CNN
 F 4 "RES SMD 100K OHM 1% 1/10W 0402" H 6900 2600 60  0001 C CNN "Desc"
@@
 Connection ~ 6900 2950
 $Comp
-L +3.3V #PWR?
+L +3.3V #PWR0132
 U 1 1 5B9C0576
 P 6900 2350
-F 0 "#PWR?" H 6900 2440 20  0001 C CNN
+F 0 "#PWR0132" H 6900 2440 20  0001 C CNN
 F 1 "+3.3V" H 6896 2478 30  0000 C CNN
 F 2 "" H 6900 2350 60  0000 C CNN
@@
 Connection ~ 3350 2900
 $Comp
-L GND #PWR?
+L GND #PWR0133
 U 1 1 5B9BE7F3
 P 3350 3600
-F 0 "#PWR?" H 3350 3350 50  0001 C CNN
+F 0 "#PWR0133" H 3350 3350 50  0001 C CNN
 F 1 "GND" H 3355 3427 50  0001 C CNN
 F 2 "" H 3350 3600 50  0000 C CNN
@@
 	3350 3600 3350 3500
 $Comp
-L SW_SPST SW?
+L SW_SPST SW2
 U 1 1 5B9C003A
 P 7100 4150
-F 0 "SW?" H 7100 4320 50  0000 C CNN
+F 0 "SW2" H 7100 4320 50  0000 C CNN
 F 1 "SW_BOOT" H 7100 3950 50  0000 C CNN
 F 2 "misc:TACT_SMD_4.5X4.5" H 7100 4150 50  0001 C CNN
@@
 	3450 3600 3350 3600
 $Comp
-L SW_SPST SW?
+L SW_SPST SW1
 U 1 1 5B9C0668
 P 3450 3250
-F 0 "SW?" H 3450 3420 50  0000 C CNN
+F 0 "SW1" H 3450 3420 50  0000 C CNN
 F 1 "SW_RESET" H 3450 3050 50  0000 C CNN
 F 2 "misc:TACT_SMD_4.5X4.5" H 3450 3250 50  0001 C CNN
