File: KiCad Proyecto/CAN_Transceiver.sch (KiCad schematic (older format))
At the start: 24 parts, among them Q6 2N7002, U4 MCP25612FD, U5 TH8056, U6 PESD1CAN, U7 PESD1CAN, U8 PESD1CAN

Commit message: fixed(temp) library problem
Parts:
- C16, C17, C18, C19, C20, C21, C22, C23: symbol OBDII_IoT:C -> C
- Q6: symbol OBDII_IoT:MOS_N -> MOS_N
- R15, R16, R17, R18, R19, R20, R21, R22, R23, R24: symbol OBDII_IoT:R -> R
- U4: symbol OBDII_IoT:MCP25612FD -> MCP25612FD
- U5: symbol OBDII_IoT:TH8056 -> TH8056
- U6, U7, U8: symbol OBDII_IoT:PESD1CAN -> PESD1CAN
Changed lines of the file:
@@
 EESchema Schematic File Version 2
-LIBS:power
-LIBS:PF_apiner-cache
+LIBS:OBDII_IoT
+LIBS:Connector
+LIBS:ESP32-footprints-Shem-Lib
+LIBS:ftdi
+LIBS:STN2120
 EELAYER 25 0
 EELAYER END
 $Descr A4 11693 8268
 encoding utf-8
-Sheet 8 9
+Sheet 6 9
 Title ""
 Date ""
@@
 HS_CAN_RX
 $Comp
-L OBDII_IoT:PESD1CAN U6
+L PESD1CAN U6
 U 1 1 582F34D6
 P 5300 6250
@@
 $EndComp
 $Comp
-L OBDII_IoT:GND #PWR060
+L GND #PWR060
 U 1 1 582F433E
 P 5300 6700
@@
 $EndComp
 $Comp
-L OBDII_IoT:R R21
+L R R21
 U 1 1 58B0A852
 P 5750 5100
@@
 $EndComp
 $Comp
-L OBDII_IoT:MCP25612FD U4
+L MCP25612FD U4
 U 1 1 58EEA34D
 P 3450 5150
@@
 $EndComp
 $Comp
-L OBDII_IoT:TH8056 U5
+L TH8056 U5
 U 1 1 58F03C6E
 P 3700 2950
@@
 SW_CAN_LOAD
 $Comp
-L OBDII_IoT:+5V_SW #PWR061
+L +5V_SW #PWR061
 U 1 1 58FD2521
 P 3150 5100
@@
 $EndComp
 $Comp
-L OBDII_IoT:PESD1CAN U7
+L PESD1CAN U7
 U 1 1 58FD2706
 P 6000 3650
@@
 $EndComp
 $Comp
-L OBDII_IoT:GND #PWR062
+L GND #PWR062
 U 1 1 58FD270C
 P 6000 4050
@@
 $EndComp
 $Comp
-L OBDII_IoT:R R17
+L R R17
 U 1 1 58FD347C
 P 4600 6100
@@
 $EndComp
 $Comp
-L OBDII_IoT:C C19
+L C C19
 U 1 1 58FD3B6F
 P 4600 6450
@@
 $EndComp
 $Comp
-L OBDII_IoT:R R19
+L R R19
 U 1 1 58FD3FA7
 P 4900 6100
@@
 $EndComp
 $Comp
-L OBDII_IoT:C C20
+L C C20
 U 1 1 58FD3FB1
 P 4900 6450
@@
 $EndComp
 $Comp
-L OBDII_IoT:PESD1CAN U8
+L PESD1CAN U8
 U 1 1 58FD4234
 P 6450 6250
@@
 $EndComp
 $Comp
-L OBDII_IoT:GND #PWR063
+L GND #PWR063
 U 1 1 58FD423A
 P 6450 6700
@@
 $EndComp
 $Comp
-L OBDII_IoT:R R22
+L R R22
 U 1 1 58FD4244
 P 5750 6100
@@
 $EndComp
 $Comp
-L OBDII_IoT:C C22
+L C C22
 U 1 1 58FD424E
 P 5750 6450
@@
 $EndComp
 $Comp
-L OBDII_IoT:R R24
+L R R24
 U 1 1 58FD4258
 P 6050 6100
@@
 $EndComp
 $Comp
-L OBDII_IoT:C C23
+L C C23
 U 1 1 58FD4262
 P 6050 6450
@@
 $EndComp
 $Comp
-L OBDII_IoT:GND #PWR064
+L GND #PWR064
 U 1 1 58FD430C
 P 4350 6700
@@
 $EndComp
 $Comp
-L OBDII_IoT:GND #PWR065
+L GND #PWR065
 U 1 1 58FD8A39
 P 4600 6700
@@
 $EndComp
 $Comp
-L OBDII_IoT:GND #PWR066
+L GND #PWR066
 U 1 1 58FD8A60
 P 4900 6700
@@
 $EndComp
 $Comp
-L OBDII_IoT:GND #PWR067
+L GND #PWR067
 U 1 1 58FD8B4B
 P 5750 6700
@@
 $EndComp
 $Comp
-L OBDII_IoT:GND #PWR068
+L GND #PWR068
 U 1 1 58FD8B72
 P 6050 6700
@@
 $EndComp
 $Comp
-L OBDII_IoT:GND #PWR069
+L GND #PWR069
 U 1 1 58FD9262
 P 2500 5700
@@
 $EndComp
 $Comp
-L OBDII_IoT:R R23
+L R R23
 U 1 1 58FDA2D5
 P 6050 5100
@@
 $EndComp
 $Comp
-L OBDII_IoT:C C16
+L C C16
 U 1 1 58FDBFE9
 P 2300 5250
@@
 $EndComp
 $Comp
-L OBDII_IoT:+5V_SW #PWR070
+L +5V_SW #PWR070
 U 1 1 58FDC0F6
 P 2100 5100
@@
 $EndComp
 $Comp
-L OBDII_IoT:C C17
+L C C17
 U 1 1 58FDC125
 P 2300 5550
@@
 $EndComp
 $Comp
-L OBDII_IoT:GND #PWR071
+L GND #PWR071
 U 1 1 58FDC707
 P 3200 6000
@@
 $EndComp
 $Comp
-L OBDII_IoT:+3.3V #PWR072
+L +3.3V #PWR072
 U 1 1 58FDF90E
 P 3200 2550
@@
 $EndComp
 $Comp
-L OBDII_IoT:DLC #PWR073
+L DLC #PWR073
 U 1 1 58FE3EFD
 P 4300 2550
@@
 $EndComp
 $Comp
-L OBDII_IoT:C C18
+L C C18
 U 1 1 58FE50CB
 P 4100 2600
@@
 $EndComp
 $Comp
-L OBDII_IoT:GND #PWR074
+L GND #PWR074
 U 1 1 58FE53E1
 P 3850 2650
@@
 	3850 2650 3850 2600
 $Comp
-L OBDII_IoT:MOS_N Q6
+L MOS_N Q6
 U 1 1 58FE7544
 P 5150 3650
@@
 $EndComp
 $Comp
-L OBDII_IoT:R R16
+L R R16
 U 1 1 58FE76BB
 P 4600 3250
@@
 $EndComp
 $Comp
-L OBDII_IoT:R R20
+L R R20
 U 1 1 58FE7CFE
 P 5250 3250
@@
 $EndComp
 $Comp
-L OBDII_IoT:R R18
+L R R18
 U 1 1 58FEA340
 P 4900 3850
@@
 $EndComp
 $Comp
-L OBDII_IoT:GND #PWR075
+L GND #PWR075
 U 1 1 58FEA42D
 P 5250 4050
@@
 $EndComp
 $Comp
-L OBDII_IoT:C C21
+L C C21
 U 1 1 58FEA778
 P 5550 3550
@@
 $EndComp
 $Comp
-L OBDII_IoT:GND #PWR076
+L GND #PWR076
 U 1 1 58FEAC5F
 P 4300 4050
@@
 	5250 3450 5250 3400
 $Comp
-L OBDII_IoT:GND #PWR077
+L GND #PWR077
 U 1 1 58FEBC1A
 P 5550 4050
@@
 	6000 4000 6000 4050
 $Comp
-L OBDII_IoT:R R15
+L R R15
 U 1 1 58FE8C9D
 P 3200 2750

Commit message: fixed fuse & wrong fields
Parts:
- C16, C17: Desc (none) -> CAP CER 0.1UF 10V X5R 0402; Descripcion CAP CER 0.1UF 10V X5R 0402 -> (none); Digikey# (none) -> 311-1336-1-ND; Digikey/Mouser 311-1336-1-ND -> (none); Fabricante Yageo -> (none); Manf (none) -> Yageo; Manf# (none) -> CC0402KRX5R6BB104; Nro. parte CC0402KRX5R6BB104 -> (none)
- C18: Desc (none) -> CAP CER 10UF 25V X5R 0805; Descripcion CAP CER 10UF 25V X5R 0805 -> (none); Digikey# (none) -> 587-2985-6-ND; Digikey/Mouser 587-2985-6-ND -> (none); Fabricante Taiyo Yuden -> (none); Manf (none) -> Taiyo Yuden; Manf# (none) -> TMK212BBJ106KG-T; Nro. parte TMK212BBJ106KG-T -> (none)
- C19, C20, C22, C23: Desc (none) -> CAP CER 560PF 50V X7R 0402; Descripcion CAP CER 560PF 50V X7R 0402 -> (none); Digikey# (none) -> 311-1029-1-ND; Digikey/Mouser 311-1029-1-ND -> (none); Fabricante Yageo -> (none); Manf (none) -> Yageo; Manf# (none) -> CC0402KRX7R9BB561; Nro. parte CC0402KRX7R9BB561 -> (none)
- C21: Desc (none) -> CAP CER 150PF 50V C0G/NP0 0402; Descripcion CAP CER 150PF 50V C0G/NP0 0402 -> (none); Digikey# (none) -> 490-3229-1-ND; Digikey/Mouser 490-3229-1-ND -> (none); Fabricante Murata -> (none); Manf (none) -> Murata; Manf# (none) -> GRM1555C1H151JA01D; Nro. parte GRM1555C1H151JA01D -> (none)
- Q6: Desc (none) -> MOSFET N-CH 60V 260MA SOT-23; Descripcion MOSFET N-CH 60V 260MA SOT-23 -> (none); Digikey# (none) -> 2N7002ET1GOSCT-ND; Digikey/Mouser 2N7002ET1GOSCT-ND -> (none); Fabricante ON Semiconductor -> (none); Manf (none) -> ON Semiconductor; Manf# (none) -> 2N7002ET1G; Nro. parte 2N7002ET1G -> (none)
- R15: Desc (none) -> RES SMD 1.5K OHM 1% 1/16W 0402; Descripcion RES SMD 1.5K OHM 1% 1/16W 0402 -> (none); Digikey# (none) -> 311-1.50KLRCT-ND; Digikey/Mouser 311-1.50KLRCT-ND -> (none); Fabricante Yageo -> (none); Manf (none) -> Yageo; Manf# (none) -> RC0402FR-071K5L; Nro. parte RC0402FR-071K5L -> (none)
- R16: Desc (none) -> RES SMD 6.49K OHM 1% 1/8W 0805; Descripcion RES SMD 6.49K OHM 1% 1/8W 0805 -> (none); Digikey# (none) -> 311-6.49KCRCT-ND; Digikey/Mouser 311-6.49KCRCT-ND -> (none); Fabricante Yageo -> (none); Manf (none) -> Yageo; Manf# (none) -> RC0805FR-076K49L; Nro. parte RC0805FR-076K49L -> (none)
- R17, R19, R22, R24: Desc (none) -> RES SMD 100 OHM 5% 1/16W 0402; Descripcion RES SMD 100 OHM 5% 1/16W 0402 -> (none); Digikey# (none) -> 311-100JRCT-ND; Digikey/Mouser 311-100JRCT-ND -> (none); Fabricante Yageo -> (none); Manf (none) -> Yageo; Manf# (none) -> RC0402JR-07100RL; Nro. parte RC0402JR-07100RL -> (none)
- R18: Desc (none) -> RES SMD 10K OHM 5% 1/16W 0402; Descripcion RES SMD 10K OHM 5% 1/16W 0402 -> (none); Digikey# (none) -> 311-10KJRCT-ND; Digikey/Mouser 311-10KJRCT-ND -> (none); Fabricante Yageo -> (none); Manf (none) -> Yageo; Manf# (none) -> RC0402JR-0710KL; Nro. parte RC0402JR-0710KL -> (none)
- R20: Desc (none) -> RES SMD 130 OHM 1% 2W 2512; Descripcion RES SMD 130 OHM 1% 2W 2512 -> (none); Digikey# (none) -> A116011CT-ND; Digikey/Mouser A116011CT-ND -> (none); Fabricante TE Connectivity -> (none); Manf (none) -> TE Connectivity; Manf# (none) -> 3521130RFT; Nro. parte 3521130RFT -> (none)
- R21, R23: Desc (none) -> RES SMD 120 OHM 5% 1/16W 0402; Descripcion RES SMD 120 OHM 5% 1/16W 0402 -> (none); Digikey# (none) -> 311-120JRCT-ND; Digikey/Mouser 311-120JRCT-ND -> (none); Fabricante Yageo -> (none); Manf (none) -> Yageo; Manf# (none) -> RC0402JR-07120RL; Nro. parte RC0402JR-07120RL -> (none)
- U4: Desc (none) -> IC TRANSCEIVER CAN HI-SPD 14SOIC; Descripcion IC TRANSCEIVER CAN HI-SPD 14SOIC -> (none); Digikey# (none) -> MCP25612FD-H/SL-ND; Digikey/Mouser MCP25612FD-H/SL-ND -> (none); Fabricante Microchip -> (none); Manf (none) -> Microchip; Manf# (none) -> MCP25612FD-H/SL; Nro. parte MCP25612FD-H/SL -> (none)
- U5: Desc (none) -> IC TXRX CAN 8SOIC; Descripcion IC TXRX CAN 8SOIC -> (none); Digikey# (none) -> TH8056KDC-AAA-008-RETR-ND; Digikey/Mouser TH8056KDC-AAA-008-RETR-ND -> (none); Fabricante Melexis -> (none); Manf (none) -> Melexis; Manf# (none) -> TH8056KDC-AAA-008-RE; Nro. parte TH8056KDC-AAA-008-RE -> (none)
- U6, U7, U8: Desc (none) -> TVS DIODE 24VWM 50VC SC70; Descripcion TVS DIODE 24VWM 50VC SC70 -> (none); Digikey# (none) -> 568-10731-1-ND; Digikey/Mouser 568-10731-1-ND -> (none); Fabricante NXP USA Inc -> (none); Manf (none) -> NXP USA Inc; Manf# (none) -> PESD1CAN-UX; Nro. parte PESD1CAN-UX -> (none)
