File: KiCad Proyecto/ISO_Transceiver.sch (KiCad schematic (older format))
At the start: 16 parts, among them Q4 MMBT3904, Q5 MMBT3904, U3 LM339

Commit message: fixed(temp) library problem
Parts:
- C13, C14, C15: symbol OBDII_IoT:C -> C
- D4, D5: symbol OBDII_IoT:D_Schottky_BAT54SL -> D_Schottky_BAT54SL
- Q4, Q5: symbol OBDII_IoT:NPN -> NPN
- R10, R11, R12, R13, R14, R7, R8, R9: symbol OBDII_IoT:R -> R
- U3: symbol OBDII_IoT:LM339 -> LM339
Changed lines of the file:
@@
 EESchema Schematic File Version 2
-LIBS:power
-LIBS:PF_apiner-cache
+LIBS:OBDII_IoT
+LIBS:Connector
+LIBS:ESP32-footprints-Shem-Lib
+LIBS:ftdi
+LIBS:STN2120
 EELAYER 25 0
 EELAYER END
@@
 K-LINE
 $Comp
-L OBDII_IoT:LM339 U3
+L LM339 U3
 U 1 1 58FAFC7B
 P 4800 4700
@@
 $EndComp
 $Comp
-L OBDII_IoT:R R10
+L R R10
 U 1 1 58FB19FB
 P 4150 2650
@@
 $EndComp
 $Comp
-L OBDII_IoT:NPN Q4
+L NPN Q4
 U 1 1 58FB1A06
 P 4050 3150
@@
 $EndComp
 $Comp
-L OBDII_IoT:R R8
+L R R8
 U 1 1 58FB1A1C
 P 3650 4400
@@
 $EndComp
 $Comp
-L OBDII_IoT:D_Schottky_BAT54SL D4
+L D_Schottky_BAT54SL D4
 U 1 1 58FB2C23
 P 4100 6100
@@
 $EndComp
 $Comp
-L OBDII_IoT:DLC_SW #PWR045
+L DLC_SW #PWR045
 U 1 1 58FB4559
 P 4150 2400
@@
 $EndComp
 $Comp
-L OBDII_IoT:R R7
+L R R7
 U 1 1 58FB45DB
 P 3650 3150
@@
 $EndComp
 $Comp
-L OBDII_IoT:GND #PWR046
+L GND #PWR046
 U 1 1 58FB47BB
 P 4150 3450
@@
 $EndComp
 $Comp
-L OBDII_IoT:R R14
+L R R14
 U 1 1 58FB4DD5
 P 5950 2650
@@
 $EndComp
 $Comp
-L OBDII_IoT:NPN Q5
+L NPN Q5
 U 1 1 58FB4DDF
 P 5850 3150
@@
 $EndComp
 $Comp
-L OBDII_IoT:DLC_SW #PWR047
+L DLC_SW #PWR047
 U 1 1 58FB4DE5
 P 5950 2400
@@
 $EndComp
 $Comp
-L OBDII_IoT:R R13
+L R R13
 U 1 1 58FB4DEF
 P 5450 3150
@@
 $EndComp
 $Comp
-L OBDII_IoT:GND #PWR048
+L GND #PWR048
 U 1 1 58FB4DF5
 P 5950 3450
@@
 $EndComp
 $Comp
-L OBDII_IoT:R R11
+L R R11
 U 1 1 58FB557C
 P 4250 4800
@@
 K-LINE
 $Comp
-L OBDII_IoT:DLC_SW #PWR049
+L DLC_SW #PWR049
 U 1 1 58FB56FF
 P 4700 4200
@@
 $EndComp
 $Comp
-L OBDII_IoT:C C13
+L C C13
 U 1 1 58FB6CF6
 P 4400 6100
@@
 $EndComp
 $Comp
-L OBDII_IoT:DLC_SW #PWR050
+L DLC_SW #PWR050
 U 1 1 58FB717D
 P 6050 4200
@@
 $EndComp
 $Comp
-L OBDII_IoT:C C15
+L C C15
 U 1 1 58FB71A2
 P 6050 4450
@@
 $EndComp
 $Comp
-L OBDII_IoT:GND #PWR051
+L GND #PWR051
 U 1 1 58FB7303
 P 4700 5050
@@
 $EndComp
 $Comp
-L OBDII_IoT:GND #PWR052
+L GND #PWR052
 U 1 1 58FB7392
 P 6050 4700
@@
 Ubicar cerca del LM339
 $Comp
-L OBDII_IoT:R R9
+L R R9
 U 1 1 58FB7561
 P 3650 4800
@@
 $EndComp
 $Comp
-L OBDII_IoT:DLC_SW #PWR053
+L DLC_SW #PWR053
 U 1 1 58FB7632
 P 3650 4200
@@
 $EndComp
 $Comp
-L OBDII_IoT:GND #PWR054
+L GND #PWR054
 U 1 1 58FB7688
 P 3650 5050
@@
 $EndComp
 $Comp
-L OBDII_IoT:GND #PWR055
+L GND #PWR055
 U 1 1 58FB9579
 P 4400 6450
@@
 ISO_RX
 $Comp
-L OBDII_IoT:+3.3V #PWR056
+L +3.3V #PWR056
 U 1 1 58FBB38D
 P 5200 4200
@@
 $EndComp
 $Comp
-L OBDII_IoT:R R12
+L R R12
 U 1 1 58FBB473
 P 5200 4400
@@
 $EndComp
 $Comp
-L OBDII_IoT:DLC #PWR057
+L DLC #PWR057
 U 1 1 58FB941A
 P 4400 5750
@@
 	3450 3150 3500 3150
 $Comp
-L OBDII_IoT:D_Schottky_BAT54SL D5
+L D_Schottky_BAT54SL D5
 U 1 1 59003DD4
 P 5250 6100
@@
 $EndComp
 $Comp
-L OBDII_IoT:C C14
+L C C14
 U 1 1 59003DDE
 P 5550 6100
@@
 $EndComp
 $Comp
-L OBDII_IoT:GND #PWR058
+L GND #PWR058
 U 1 1 59003DE4
 P 5550 6450
@@
 $EndComp
 $Comp
-L OBDII_IoT:DLC #PWR059
+L DLC #PWR059
 U 1 1 59003DEA
 P 5550 5750

Commit message: fixed fuse & wrong fields
Parts:
- C13, C14, C15: Desc (none) -> CAP CER 0.1UF 25V X7R 0603; Descripcion CAP CER 0.1UF 25V X7R 0603 -> (none); Digikey# (none) -> 311-1341-1-ND; Digikey/Mouser 311-1341-1-ND -> (none); Fabricante Yageo -> (none); Manf (none) -> Yageo; Manf# (none) -> CC0603KRX7R8BB104; Nro. parte CC0603KRX7R8BB104 -> (none)
- D4, D5: Desc (none) -> Diode Array 1 Pair Series Connection Schottky 30V 200mA (DC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; Descripcion Diode Array 1 Pair Series Connection Schottky 30V 200mA (DC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 -> (none); Digikey# (none) -> BAT54SLT1GOSCT-ND; Digikey/Mouser BAT54SLT1GOSCT-ND -> (none); Fabricante ON Semiconductor -> (none); Manf (none) -> ON Semiconductor; Manf# (none) -> BAT54SLT1G; Nro. parte BAT54SLT1G -> (none)
- Q4, Q5: Desc (none) -> TRANS NPN 40V 0.2A SOT23; Descripcion TRANS NPN 40V 0.2A SOT23 -> (none); Digikey# (none) -> MMBT3904LT3GOSCT-ND; Digikey/Mouser MMBT3904LT3GOSCT-ND -> (none); Fabricante ON Semiconductor -> (none); Manf (none) -> ON Semiconductor; Manf# (none) -> MMBT3904LT3G; Nro. parte MMBT3904LT3G -> (none)
- R10, R14: Desc (none) -> RES SMD 510 OHM 5% 1/2W 0805; Descripcion RES SMD 510 OHM 5% 1/2W 0805 -> (none); Digikey# (none) -> P510ADCT-ND; Digikey/Mouser P510ADCT-ND -> (none); Fabricante Panasonic Electronic Components -> (none); Manf (none) -> Panasonic Electronic Components; Manf# (none) -> ERJ-P06J511V; Nro. parte ERJ-P06J511V -> (none)
- R11, R12, R8, R9: Desc (none) -> RES SMD 10K OHM 5% 1/16W 0402; Descripcion RES SMD 10K OHM 5% 1/16W 0402 -> (none); Digikey# (none) -> 311-10KJRCT-ND; Digikey/Mouser 311-10KJRCT-ND -> (none); Fabricante Yageo -> (none); Manf (none) -> Yageo; Manf# (none) -> RC0402JR-0710KL; Nro. parte RC0402JR-0710KL -> (none)
- R13, R7: Desc (none) -> RES SMD 1K OHM 5% 1/16W 0402; Descripcion RES SMD 1K OHM 5% 1/16W 0402 -> (none); Digikey# (none) -> 311-1.0KJRCT-ND; Digikey/Mouser 311-1.0KJRCT-ND -> (none); Fabricante Yageo -> (none); Manf (none) -> Yageo; Manf# (none) -> RC0402JR-071KL; Nro. parte RC0402JR-071KL -> (none)
- U3: Desc (none) -> IC QUAD DIFF COMPARATOR 14-TSSOP; Descripcion IC QUAD DIFF COMPARATOR 14-TSSOP -> (none); Digikey# (none) -> 296-6607-1-ND; Digikey/Mouser 296-6607-1-ND -> (none); Fabricante Texas Instruments -> (none); Manf (none) -> Texas Instruments; Manf# (none) -> LM339PWR; Nro. parte LM339PWR -> (none)
