File: KiCad Proyecto/J1850_Transceiver.sch (KiCad schematic (older format))
At the start: 30 parts, among them Q10 2N7002, Q7 2N7002, Q8 2N7002, Q9 BSS314PE, U3 LM339, U9 LM317

Commit message: fixed(temp) library problem
Parts:
- C24, C25, C26, C27: symbol OBDII_IoT:C -> C
- D10, D8, D9: symbol OBDII_IoT:D_Schot -> D_Schot
- D6, D7: symbol OBDII_IoT:D_Schottky_BAT54SL -> D_Schottky_BAT54SL
- Q10, Q7, Q8: symbol OBDII_IoT:MOS_N -> MOS_N
- Q9: symbol OBDII_IoT:MOS_P -> MOS_P
- R25, R26, R27, R28, R29, R30, R31, R32, R33, R34, R35, R36, R37, R38, R39: symbol OBDII_IoT:R -> R
- U3: symbol OBDII_IoT:LM339 -> LM339
- U9: symbol OBDII_IoT:LM317LD -> LM317LD
Changed lines of the file:
@@
 EESchema Schematic File Version 2
-LIBS:power
-LIBS:PF_apiner-cache
+LIBS:OBDII_IoT
+LIBS:Connector
+LIBS:ESP32-footprints-Shem-Lib
+LIBS:ftdi
+LIBS:STN2120
 EELAYER 25 0
 EELAYER END
@@
 J1850_BUS-_TX
 $Comp
-L OBDII_IoT:R R25
+L R R25
 U 1 1 582FD8FC
 P 3900 1850
@@
 $EndComp
 $Comp
-L OBDII_IoT:R R26
+L R R26
 U 1 1 582FDADA
 P 3900 2350
@@
 $EndComp
 $Comp
-L OBDII_IoT:R R27
+L R R27
 U 1 1 5832E14E
 P 3900 2750
@@
 $EndComp
 $Comp
-L OBDII_IoT:LM339 U3
+L LM339 U3
 U 2 1 58FEE375
 P 5850 2100
@@
 $EndComp
 $Comp
-L OBDII_IoT:LM339 U3
+L LM339 U3
 U 3 1 58FEE380
 P 8550 1950
@@
 $EndComp
 $Comp
-L OBDII_IoT:MOS_N Q7
+L MOS_N Q7
 U 1 1 58FF3421
 P 3550 2750
@@
 J1850_BUS+_VH
 $Comp
-L OBDII_IoT:C C25
+L C C25
 U 1 1 58FF9848
 P 2950 1950
@@
 	2950 1600 2950 1800
 $Comp
-L OBDII_IoT:DLC_SW #PWR078
+L DLC_SW #PWR078
 U 1 1 58FFBF93
 P 2950 1600
@@
 Connection ~ 2950 1650
 $Comp
-L OBDII_IoT:V_J1850 #PWR079
+L V_J1850 #PWR079
 U 1 1 58FFC6C3
 P 3900 1600
@@
 Connection ~ 3900 1650
 $Comp
-L OBDII_IoT:GND #PWR080
+L GND #PWR080
 U 1 1 58FFC795
 P 2950 2200
@@
 Connection ~ 3900 2550
 $Comp
-L OBDII_IoT:GND #PWR081
+L GND #PWR081
 U 1 1 58FFC8CF
 P 3900 3000
@@
 	3300 2750 3350 2750
 $Comp
-L OBDII_IoT:R R30
+L R R30
 U 1 1 58FFF46B
 P 5300 2000
@@
 $EndComp
 $Comp
-L OBDII_IoT:D_Schottky_BAT54SL D6
+L D_Schottky_BAT54SL D6
 U 1 1 58FFFF10
 P 1950 4350
@@
 $EndComp
 $Comp
-L OBDII_IoT:C C24
+L C C24
 U 1 1 58FFFF1B
 P 2250 4350
@@
 J1850_BUS-
 $Comp
-L OBDII_IoT:DLC #PWR082
+L DLC #PWR082
 U 1 1 59002768
 P 2250 4000
@@
 $EndComp
 $Comp
-L OBDII_IoT:GND #PWR083
+L GND #PWR083
 U 1 1 5900289A
 P 2250 4700
@@
 Connection ~ 2250 4050
 $Comp
-L OBDII_IoT:D_Schottky_BAT54SL D7
+L D_Schottky_BAT54SL D7
 U 1 1 59002A9E
 P 3100 4350
@@
 $EndComp
 $Comp
-L OBDII_IoT:C C26
+L C C26
 U 1 1 59002AA8
 P 3400 4350
@@
 $EndComp
 $Comp
-L OBDII_IoT:DLC #PWR084
+L DLC #PWR084
 U 1 1 59002AAE
 P 3400 4000
@@
 $EndComp
 $Comp
-L OBDII_IoT:GND #PWR085
+L GND #PWR085
 U 1 1 59002AB4
 P 3400 4700
@@
 	1600 2950 1750 2950
 $Comp
-L OBDII_IoT:R R31
+L R R31
 U 1 1 5900554A
 P 5300 2200
@@
 $EndComp
 $Comp
-L OBDII_IoT:DLC_SW #PWR086
+L DLC_SW #PWR086
 U 1 1 5900675A
 P 5750 1700
@@
 $EndComp
 $Comp
-L OBDII_IoT:GND #PWR087
+L GND #PWR087
 U 1 1 5900679C
 P 5750 2450
@@
 	5750 2400 5750 2450
 $Comp
-L OBDII_IoT:+3.3V #PWR088
+L +3.3V #PWR088
 U 1 1 59006FD8
 P 6250 1700
@@
 $EndComp
 $Comp
-L OBDII_IoT:R R33
+L R R33
 U 1 1 59006FE2
 P 6250 1900
@@
 Connection ~ 6250 2100
 $Comp
-L OBDII_IoT:MOS_N Q8
+L MOS_N Q8
 U 1 1 59007FAD
 P 5150 4100
@@
 $EndComp
 $Comp
-L OBDII_IoT:MOS_P Q9
+L MOS_P Q9
 U 1 1 5900CF77
 P 5500 3550
@@
 $EndComp
 $Comp
-L OBDII_IoT:R R28
+L R R28
 U 1 1 5900D39E
 P 4900 4300
@@
 $EndComp
 $Comp
-L OBDII_IoT:GND #PWR089
+L GND #PWR089
 U 1 1 5900D50B
 P 5250 4500
@@
 $EndComp
 $Comp
-L OBDII_IoT:R R29
+L R R29
 U 1 1 5900D718
 P 5250 3650
@@
 $EndComp
 $Comp
-L OBDII_IoT:D_Schot D8
+L D_Schot D8
 U 1 1 5900E8B5
 P 5950 3450
@@
 J1850_BUS+
 $Comp
-L OBDII_IoT:D_Schot D9
+L D_Schot D9
 U 1 1 5900EFC2
 P 6150 4250
@@
 $EndComp
 $Comp
-L OBDII_IoT:R R32
+L R R32
 U 1 1 5900F3D6
 P 6150 3850
@@
 $EndComp
 $Comp
-L OBDII_IoT:GND #PWR090
+L GND #PWR090
 U 1 1 5900F564
 P 6150 4500
@@
 	5250 3400 5250 3500
 $Comp
-L OBDII_IoT:V_J1850 #PWR091
+L V_J1850 #PWR091
 U 1 1 5900FFB7
 P 5250 3400
@@
 	6150 4500 6150 4350
 $Comp
-L OBDII_IoT:+3.3V #PWR092
+L +3.3V #PWR092
 U 1 1 59011723
 P 8950 1550
@@
 $EndComp
 $Comp
-L OBDII_IoT:R R39
+L R R39
 U 1 1 5901172D
 P 8950 1750
@@
 	8950 1600 8950 1550
 $Comp
-L OBDII_IoT:DLC_SW #PWR093
+L DLC_SW #PWR093
 U 1 1 5901176C
 P 8450 1550
@@
 	8450 1550 8450 1650
 $Comp
-L OBDII_IoT:R R35
+L R R35
 U 1 1 59011805
 P 7350 2250
@@
 $EndComp
 $Comp
-L OBDII_IoT:R R34
+L R R34
 U 1 1 590118B7
 P 7350 1850
@@
 $EndComp
 $Comp
-L OBDII_IoT:R R37
+L R R37
 U 1 1 590119B2
 P 8050 1850
@@
 Connection ~ 7350 2050
 $Comp
-L OBDII_IoT:+5V_SW #PWR094
+L +5V_SW #PWR094
 U 1 1 590137AA
 P 7350 1550
@@
 	7350 1550 7350 1700
 $Comp
-L OBDII_IoT:GND #PWR095
+L GND #PWR095
 U 1 1 5901397C
 P 7350 2450
@@
 	7350 2450 7350 2400
 $Comp
-L OBDII_IoT:GND #PWR096
+L GND #PWR096
 U 1 1 59013A21
 P 8450 2450
@@
 Connection ~ 8950 1950
 $Comp
-L OBDII_IoT:+5V_SW #PWR097
+L +5V_SW #PWR097
 U 1 1 590144CF
 P 8200 3400
@@
 $EndComp
 $Comp
-L OBDII_IoT:D_Schot D10
+L D_Schot D10
 U 1 1 590146A5
 P 8200 3550
@@
 $EndComp
 $Comp
-L OBDII_IoT:R R38
+L R R38
 U 1 1 590146AF
 P 8200 3850
@@
 $EndComp
 $Comp
-L OBDII_IoT:MOS_N Q10
+L MOS_N Q10
 U 1 1 590147AD
 P 8100 4300
@@
 $EndComp
 $Comp
-L OBDII_IoT:R R36
+L R R36
 U 1 1 59015277
 P 7850 3850
@@
 	7800 4300 7900 4300
 $Comp
-L OBDII_IoT:GND #PWR098
+L GND #PWR098
 U 1 1 590155AC
 P 8200 4550
@@
 $EndComp
 $Comp
-L OBDII_IoT:+5V_SW #PWR099
+L +5V_SW #PWR099
 U 1 1 59015925
 P 7850 3400
@@
 	8200 4550 8200 4500
 $Comp
-L OBDII_IoT:LM317LD U9
+L LM317LD U9
 U 1 1 58F8CA15
 P 3400 1650
@@
 $EndComp
 $Comp
-L OBDII_IoT:C C27
+L C C27
 U 1 1 58FD532B
 P 4150 1850
@@
 $EndComp
 $Comp
-L OBDII_IoT:GND #PWR0100
+L GND #PWR0100
 U 1 1 58FD55BE
 P 4150 2150

Commit message: fixed fuse & wrong fields
Parts:
- C24, C25, C26, C27: Desc (none) -> CAP CER 0.1UF 25V X7R 0603; Descripcion CAP CER 0.1UF 25V X7R 0603 -> (none); Digikey# (none) -> 311-1341-1-ND; Digikey/Mouser 311-1341-1-ND -> (none); Fabricante Yageo -> (none); Manf (none) -> Yageo; Manf# (none) -> CC0603KRX7R8BB104; Nro. parte CC0603KRX7R8BB104 -> (none)
- D10, D8, D9: Desc (none) -> Diode Schottky 30V 200mA Surface Mount SMini2-F5-B; Descripcion Diode Schottky 30V 200mA Surface Mount SMini2-F5-B -> (none); Digikey# (none) -> DB2J31000LCT-ND; Digikey/Mouser DB2J31000LCT-ND -> (none); Fabricante Panasonic Electronic Components -> (none); Manf (none) -> Panasonic Electronic Components; Manf# (none) -> DB2J31000L; Nro. parte DB2J31000L -> (none)
- D6, D7: Desc (none) -> Diode Array 1 Pair Series Connection Schottky 30V 200mA (DC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; Descripcion Diode Array 1 Pair Series Connection Schottky 30V 200mA (DC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 -> (none); Digikey# (none) -> BAT54SLT1GOSCT-ND; Digikey/Mouser BAT54SLT1GOSCT-ND -> (none); Fabricante ON Semiconductor -> (none); Manf (none) -> ON Semiconductor; Manf# (none) -> BAT54SLT1G; Nro. parte BAT54SLT1G -> (none)
- Q10, Q7, Q8: Desc (none) -> MOSFET N-CH 60V 260MA SOT-23; Descripcion MOSFET N-CH 60V 260MA SOT-23 -> (none); Digikey# (none) -> 2N7002ET1GOSCT-ND; Digikey/Mouser 2N7002ET1GOSCT-ND -> (none); Fabricante ON Semiconductor -> (none); Manf (none) -> ON Semiconductor; Manf# (none) -> 2N7002ET1G; Nro. parte 2N7002ET1G -> (none)
- Q9: Desc (none) -> MOSFET P-CH 30V 1.5A SOT23; Descripcion MOSFET P-CH 30V 1.5A SOT23 -> (none); Digikey# (none) -> BSS314PE H6327CT-ND; Digikey/Mouser BSS314PE H6327CT-ND -> (none); Fabricante Infineon -> (none); Manf (none) -> Infineon; Manf# (none) -> BSS314PE H6327; Nro. parte BSS314PE H6327 -> (none)
- R25: Desc (none) -> RES SMD 240 OHM 1% 1/16W 0402; Descripcion RES SMD 240 OHM 1% 1/16W 0402 -> (none); Digikey# (none) -> 311-240LRCT-ND; Digikey/Mouser 311-240LRCT-ND -> (none); Fabricante Yageo -> (none); Manf (none) -> Yageo; Manf# (none) -> RC0402FR-07240RL; Nro. parte RC0402FR-07240RL -> (none)
- R26: Desc (none) -> RES SMD 866 OHM 1% 1/16W 0402; Descripcion RES SMD 866 OHM 1% 1/16W 0402 -> (none); Digikey# (none) -> YAG3248CT-ND; Digikey/Mouser YAG3248CT-ND -> (none); Fabricante Yaego -> (none); Manf (none) -> Yaego; Manf# (none) -> RC0402FR-07866RL; Nro. parte RC0402FR-07866RL -> (none)
- R27: Desc (none) -> RES SMD 374 OHM 1% 1/16W 0402; Descripcion RES SMD 374 OHM 1% 1/16W 0402 -> (none); Digikey# (none) -> YAG3137CT-ND; Digikey/Mouser YAG3137CT-ND -> (none); Fabricante Yageo -> (none); Manf (none) -> Yageo; Manf# (none) -> RC0402FR-07374RL; Nro. parte RC0402FR-07374RL -> (none)
- R28, R29, R30, R31, R32, R33, R35, R36, R37, R38, R39: Desc (none) -> RES SMD 10K OHM 5% 1/16W 0402; Descripcion RES SMD 10K OHM 5% 1/16W 0402 -> (none); Digikey# (none) -> 311-10KJRCT-ND; Digikey/Mouser 311-10KJRCT-ND -> (none); Fabricante Yageo -> (none); Manf (none) -> Yageo; Manf# (none) -> RC0402JR-0710KL; Nro. parte RC0402JR-0710KL -> (none)
- R34: Desc (none) -> RES SMD 2.7K OHM 5% 1/16W 0402; Descripcion RES SMD 2.7K OHM 5% 1/16W 0402 -> (none); Digikey# (none) -> 311-2.7KJRCT-ND; Digikey/Mouser 311-2.7KJRCT-ND -> (none); Fabricante Yageo -> (none); Manf (none) -> Yageo; Manf# (none) -> RC0402JR-072K7L; Nro. parte RC0402JR-072K7L -> (none)
- U3: Desc (none) -> IC QUAD DIFF COMPARATOR 14-TSSOP; Descripcion IC QUAD DIFF COMPARATOR 14-TSSOP -> (none); Digikey# (none) -> 296-6607-1-ND; Digikey/Mouser 296-6607-1-ND -> (none); Fabricante Texas Instruments -> (none); Manf (none) -> Texas Instruments; Manf# (none) -> LM339PWR; Nro. parte LM339PWR -> (none)
- U9: Desc (none) -> IC REG LINEAR ADJ 0.1A SOT89-3; Descripcion IC REG LINEAR ADJ 0.1A SOT89-3 -> (none); Digikey# (none) -> 296-26093-1-ND; Digikey/Mouser 296-26093-1-ND -> (none); Fabricante Texas Instruments -> (none); Manf (none) -> Texas Instruments; Manf# (none) -> LM317LCPK; Nro. parte LM317LCPK -> (none)

Commit message: added screw holes
Other:
- note added: "revizar este footprint"
Changed lines of the file:
@@
 Wire Wire Line
 	4150 1650 4150 1700
+Text Notes 2950 1250 0    60   ~ 0
+revizar este footprint
 $EndSCHEMATC
