File: KiCad Proyecto/OBD_UART_Interface.sch (KiCad schematic (older format))
At the start: 20 parts, among them U10 STN2120, Y1 16M

Commit message: fixed(temp) library problem
Parts:
- C28, C29, C30, C31, C32, C33: symbol OBDII_IoT:C -> C
- R40, R41, R42, R43, R44, R45, R46, R47, R48, R49, R50, R51: symbol OBDII_IoT:R -> R
- U10: symbol STN2120:STN2120 -> STN2120
- Y1: symbol OBDII_IoT:XTAL-4 -> XTAL-4
Changed lines of the file:
@@
 EESchema Schematic File Version 2
-LIBS:power
-LIBS:PF_apiner-cache
+LIBS:OBDII_IoT
+LIBS:Connector
+LIBS:ESP32-footprints-Shem-Lib
+LIBS:ftdi
+LIBS:STN2120
 EELAYER 25 0
 EELAYER END
@@
 UART_RX
 $Comp
-L STN2120:STN2120 U10
+L STN2120 U10
 U 1 1 58EDBBC5
 P 5200 3200
@@
 SW_CAN_LOAD
 $Comp
-L OBDII_IoT:XTAL-4 Y1
+L XTAL-4 Y1
 U 1 1 5903DC2F
 P 7000 2850
@@
 $EndComp
 $Comp
-L OBDII_IoT:C C33
+L C C33
 U 1 1 5903DF35
 P 7200 3100
@@
 $EndComp
 $Comp
-L OBDII_IoT:C C32
+L C C32
 U 1 1 5903E0C3
 P 6800 3100
@@
 $EndComp
 $Comp
-L OBDII_IoT:GND #PWR0101
+L GND #PWR0101
 U 1 1 5903E766
 P 7000 3350
@@
 PWR_SAVE
 $Comp
-L OBDII_IoT:C C29
+L C C29
 U 1 1 5904189F
 P 3700 2150
@@
 $EndComp
 $Comp
-L OBDII_IoT:R R45
+L R R45
 U 1 1 590439DA
 P 3700 1700
@@
 $EndComp
 $Comp
-L OBDII_IoT:C C28
+L C C28
 U 1 1 59044C3A
 P 3700 1850
@@
 $EndComp
 $Comp
-L OBDII_IoT:+3.3V #PWR0102
+L +3.3V #PWR0102
 U 1 1 59046CC9
 P 3500 1650
@@
 $EndComp
 $Comp
-L OBDII_IoT:GND #PWR0103
+L GND #PWR0103
 U 1 1 5904707A
 P 3500 1900
@@
 $EndComp
 $Comp
-L OBDII_IoT:+3.3V #PWR0104
+L +3.3V #PWR0104
 U 1 1 59047136
 P 3900 2350
@@
 $EndComp
 $Comp
-L OBDII_IoT:GND #PWR0105
+L GND #PWR0105
 U 1 1 590471E5
 P 3500 2200
@@
 $EndComp
 $Comp
-L OBDII_IoT:+5V_SW #PWR0106
+L +5V_SW #PWR0106
 U 1 1 59048A8B
 P 3250 2150
@@
 $EndComp
 $Comp
-L OBDII_IoT:PWR_FLAG #FLG0107
+L PWR_FLAG #FLG0107
 U 1 1 59048B35
 P 3950 1700
@@
 $EndComp
 $Comp
-L OBDII_IoT:R R44
+L R R44
 U 1 1 59049DD7
 P 3250 2350
@@
 $EndComp
 $Comp
-L OBDII_IoT:R R43
+L R R43
 U 1 1 5904A952
 P 3050 2350
@@
 $EndComp
 $Comp
-L OBDII_IoT:R R41
+L R R41
 U 1 1 5904B0AE
 P 2850 2350
@@
 $EndComp
 $Comp
-L OBDII_IoT:+3.3V #PWR0108
+L +3.3V #PWR0108
 U 1 1 5904B391
 P 3050 2150
@@
 $EndComp
 $Comp
-L OBDII_IoT:R R40
+L R R40
 U 1 1 5904B9FE
 P 2650 2350
@@
 $EndComp
 $Comp
-L OBDII_IoT:+5V_SW #PWR0109
+L +5V_SW #PWR0109
 U 1 1 5904BD19
 P 2850 2150
@@
 $EndComp
 $Comp
-L OBDII_IoT:+3.3V #PWR0110
+L +3.3V #PWR0110
 U 1 1 5904BD78
 P 2650 2150
@@
 $EndComp
 $Comp
-L OBDII_IoT:GND #PWR0111
+L GND #PWR0111
 U 1 1 5904BFE6
 P 3950 3600
@@
 $EndComp
 $Comp
-L OBDII_IoT:R R42
+L R R42
 U 1 1 5904CEC6
 P 2850 3350
@@
 $EndComp
 $Comp
-L OBDII_IoT:+3.3V #PWR0112
+L +3.3V #PWR0112
 U 1 1 5904D311
 P 2850 3150
@@
 $EndComp
 $Comp
-L OBDII_IoT:GND #PWR0113
+L GND #PWR0113
 U 1 1 5904D529
 P 6450 2500
@@
 $EndComp
 $Comp
-L OBDII_IoT:R R46
+L R R46
 U 1 1 58F97F7C
 P 6550 3300
@@
 $EndComp
 $Comp
-L OBDII_IoT:+3.3V #PWR0114
+L +3.3V #PWR0114
 U 1 1 58F97F82
 P 6550 3100
@@
 $EndComp
 $Comp
-L OBDII_IoT:R R47
+L R R47
 U 1 1 58F988CB
 P 7500 3250
@@
 $EndComp
 $Comp
-L OBDII_IoT:+3.3V #PWR0115
+L +3.3V #PWR0115
 U 1 1 58F988D1
 P 7500 2900
@@
 $EndComp
 $Comp
-L OBDII_IoT:R R48
+L R R48
 U 1 1 58F989BA
 P 7600 3250
@@
 	8200 4850 6350 4850
 $Comp
-L OBDII_IoT:+5V_SW #PWR0116
+L +5V_SW #PWR0116
 U 1 1 58F9D419
 P 7750 2900
@@
 	7850 4050 7850 3400
 $Comp
-L OBDII_IoT:R R51
+L R R51
 U 1 1 58F9E41D
 P 7950 3250
@@
 Connection ~ 7750 3950
 $Comp
-L OBDII_IoT:+3.3V #PWR0117
+L +3.3V #PWR0117
 U 1 1 58FA1833
 P 4900 1450
@@
 $EndComp
 $Comp
-L OBDII_IoT:C C30
+L C C30
 U 1 1 58FA1876
 P 5150 1500
@@
 $EndComp
 $Comp
-L OBDII_IoT:C C31
+L C C31
 U 1 1 58FA1951
 P 5150 1700
@@
 $EndComp
 $Comp
-L OBDII_IoT:GND #PWR0118
+L GND #PWR0118
 U 1 1 58FA1B98
 P 5400 1750
@@
 NoConn ~ 6350 3250
 $Comp
-L OBDII_IoT:R R49
+L R R49
 U 1 1 58FE6DAD
 P 7750 3250
@@
 $EndComp
 $Comp
-L OBDII_IoT:R R50
+L R R50
 U 1 1 58FE6FBE
 P 7850 3250
@@
 	7750 2950 7850 2950
 $Comp
-L OBDII_IoT:+5V #PWR0119
+L +5V #PWR0119
 U 1 1 5903F151
 P 7950 2900

Commit message: arreglando manquiadas
Parts:
- R42: value 1K -> 10K
Changed lines of the file:
@@
 EESchema Schematic File Version 2
-LIBS:OBDII_IoT
 LIBS:Connector
 LIBS:ESP32-footprints-Shem-Lib
 LIBS:ftdi
+LIBS:OBDII_IoT
 LIBS:STN2120
 LIBS:PF_apiner-cache
@@
 P 2850 3350
 F 0 "R42" V 2930 3350 50  0000 C CNN
-F 1 "1K" V 2850 3350 50  0000 C CNN
+F 1 "10K" V 2850 3350 50  0000 C CNN
 F 2 "chip_rlc:r_0402" V 2780 3350 50  0001 C CNN
 F 3 "" H 2850 3350 50  0000 C CNN

Commit message: cambios boludos
Other:
- note added: "revizar footprint"
Changed lines of the file:
@@
 	1    0    0    -1
 $EndComp
+Text Notes 2500 2950 0    60   ~ 0
+revizar footprint
 $EndSCHEMATC

Commit message: fixed fuse & wrong fields
Parts:
- C28, C30, C31: Desc (none) -> CAP CER 1UF 6.3V X5R 0402; Descripcion CAP CER 1UF 6.3V X5R 0402 -> (none); Digikey# (none) -> 587-1231-1-ND; Digikey/Mouser 587-1231-1-ND -> (none); Fabricante Taiyo Yuden -> (none); Manf (none) -> Taiyo Yuden; Manf# (none) -> JMK105BJ105KV-F; Nro. parte JMK105BJ105KV-F -> (none)
- C29: Desc (none) -> CAP CER 10UF 6.3V X5R 0603; Descripcion CAP CER 10UF 6.3V X5R 0603 -> (none); Digikey# (none) -> 587-1256-1-ND; Digikey/Mouser 587-1256-1-ND -> (none); Fabricante Taiyo Yuden -> (none); Manf (none) -> Taiyo Yuden; Manf# (none) -> JMK107BJ106MA-T; Nro. parte JMK107BJ106MA-T -> (none)
- C32, C33: Desc (none) -> CAP CER 16PF 50V C0G/NP0 0402; Descripcion CAP CER 16PF 50V C0G/NP0 0402 -> (none); Digikey# (none) -> 490-5926-1-ND; Digikey/Mouser 490-5926-1-ND -> (none); Fabricante Murata -> (none); Manf (none) -> Murata; Manf# (none) -> GRM1555C1H160JA01D; Nro. parte GRM1555C1H160JA01D -> (none)
- R40, R43, R46, R47, R48: Desc (none) -> RES SMD 100K OHM 1% 1/16W 0402; Descripcion RES SMD 100K OHM 1% 1/16W 0402 -> (none); Digikey# (none) -> 311-100KLRCT-ND; Digikey/Mouser 311-100KLRCT-ND -> (none); Fabricante Yageo -> (none); Manf (none) -> Yageo; Manf# (none) -> RC0402FR-07100KL; Nro. parte RC0402FR-07100KL -> (none)
- R41, R42: Desc (none) -> RES SMD 1K OHM 5% 1/16W 0402; Descripcion RES SMD 1K OHM 5% 1/16W 0402 -> (none); Digikey# (none) -> 311-1.0KJRCT-ND; Digikey/Mouser 311-1.0KJRCT-ND -> (none); Fabricante Yageo -> (none); Manf (none) -> Yageo; Manf# (none) -> RC0402JR-071KL; Nro. parte RC0402JR-071KL -> (none)
- R44, R51: Desc (none) -> RES SMD 1.5K OHM 1% 1/16W 0402; Descripcion RES SMD 1.5K OHM 1% 1/16W 0402 -> (none); Digikey# (none) -> 311-1.50KLRCT-ND; Digikey/Mouser 311-1.50KLRCT-ND -> (none); Fabricante Yageo -> (none); Manf (none) -> Yageo; Manf# (none) -> RC0402FR-071K5L; Nro. parte RC0402FR-071K5L -> (none)
- R45: Desc (none) -> RES SMD 10 OHM 5% 1/16W 0402; Descripcion RES SMD 10 OHM 5% 1/16W 0402 -> (none); Digikey# (none) -> 311-10JRCT-ND; Digikey/Mouser 311-10JRCT-ND -> (none); Fabricante Yageo -> (none); Manf (none) -> Yageo; Manf# (none) -> RC0402JR-0710RL; Nro. parte RC0402JR-0710RL -> (none)
- R49, R50: Desc (none) -> RES SMD 10K OHM 5% 1/16W 0402; Descripcion RES SMD 10K OHM 5% 1/16W 0402 -> (none); Digikey# (none) -> 311-10KJRCT-ND; Digikey/Mouser 311-10KJRCT-ND -> (none); Fabricante Yageo -> (none); Manf (none) -> Yageo; Manf# (none) -> RC0402JR-0710KL; Nro. parte RC0402JR-0710KL -> (none)
- U10: Desc (none) -> OBD-II, SW-CAN, MS-CAN Interpreter IC; Descripcion OBD-II, SW-CAN, MS-CAN Interpreter IC -> (none); Fabricante OBD Solutions -> (none); Manf (none) -> OBD Solutions; Manf# (none) -> STN2120; Nro. parte STN2120 -> (none)
- Y1: Desc (none) -> CRYSTAL 16.0000MHZ 8PF SMD; Descripcion CRYSTAL 16.0000MHZ 8PF SMD -> (none); Digikey# (none) -> 887-2555-1-ND; Digikey/Mouser 887-2555-1-ND -> (none); Fabricante TXC -> (none); Manf (none) -> TXC; Manf# (none) -> 7M-16.000MAHV-T; Nro. parte 7M-16.000MAHV-T -> (none)
