File: KiCad Proyecto/Power_CRTL.sch (KiCad schematic (older format))
At the start: 5 parts, among them Q1 2N7002, Q2 BSS314PE, Q3 BSS314PE

Commit message: fixed(temp) library problem
Parts:
- Q1: symbol OBDII_IoT:MOS_N -> MOS_N
- Q2, Q3: symbol OBDII_IoT:MOS_P -> MOS_P
- R3, R4: symbol OBDII_IoT:R -> R
Changed lines of the file:
@@
 EESchema Schematic File Version 2
-LIBS:power
-LIBS:PF_apiner-cache
+LIBS:OBDII_IoT
+LIBS:Connector
+LIBS:ESP32-footprints-Shem-Lib
+LIBS:ftdi
+LIBS:STN2120
 EELAYER 25 0
 EELAYER END
@@
 PWR_SAVE
 $Comp
-L OBDII_IoT:DLC #PWR029
+L DLC #PWR029
 U 1 1 5833D47C
 P 5350 4600
@@
 $EndComp
 $Comp
-L OBDII_IoT:DLC_SW #PWR030
+L DLC_SW #PWR030
 U 1 1 5833D496
 P 5950 4600
@@
 $EndComp
 $Comp
-L OBDII_IoT:+5V_SW #PWR031
+L +5V_SW #PWR031
 U 1 1 5833D581
 P 6900 4600
@@
 	5000 4300 5000 4450
 $Comp
-L OBDII_IoT:DLC #PWR032
+L DLC #PWR032
 U 1 1 5833D8D2
 P 5000 3900
@@
 	5000 3900 5000 4000
 $Comp
-L OBDII_IoT:GND #PWR033
+L GND #PWR033
 U 1 1 5833D90C
 P 5000 4950
@@
 Connection ~ 5650 4400
 $Comp
-L OBDII_IoT:PWR_FLAG #FLG034
+L PWR_FLAG #FLG034
 U 1 1 584984F2
 P 5350 5000
@@
 $EndComp
 $Comp
-L OBDII_IoT:PWR_FLAG #FLG035
+L PWR_FLAG #FLG035
 U 1 1 58498516
 P 5950 5000
@@
 $EndComp
 $Comp
-L OBDII_IoT:PWR_FLAG #FLG036
+L PWR_FLAG #FLG036
 U 1 1 5849858A
 P 6900 5000
@@
 Connection ~ 6900 4850
 $Comp
-L OBDII_IoT:R R3
+L R R3
 U 1 1 58FA0F0C
 P 4600 4150
@@
 $EndComp
 $Comp
-L OBDII_IoT:+3.3V #PWR037
+L +3.3V #PWR037
 U 1 1 58FA0FB6
 P 4600 3900
@@
 	4600 3900 4600 4000
 $Comp
-L OBDII_IoT:R R4
+L R R4
 U 1 1 58FA1022
 P 5000 4150
@@
 $EndComp
 $Comp
-L OBDII_IoT:MOS_P Q2
+L MOS_P Q2
 U 1 1 58FA2395
 P 5650 4750
@@
 $EndComp
 $Comp
-L OBDII_IoT:MOS_N Q1
+L MOS_N Q1
 U 1 1 58FA23A0
 P 4900 4650
@@
 $EndComp
 $Comp
-L OBDII_IoT:+5V #PWR038
+L +5V #PWR038
 U 1 1 58FA6825
 P 6300 4600
@@
 	6300 4600 6300 5000
 $Comp
-L OBDII_IoT:PWR_FLAG #FLG039
+L PWR_FLAG #FLG039
 U 1 1 58FA7137
 P 6300 5000
@@
 	6600 4400 5000 4400
 $Comp
-L OBDII_IoT:MOS_P Q3
+L MOS_P Q3
 U 1 1 59009220
 P 6600 4750

Commit message: fixed fuse & wrong fields
Parts:
- Q1: Desc (none) -> MOSFET N-CH 60V 260MA SOT-23; Descripcion MOSFET N-CH 60V 260MA SOT-23 -> (none); Digikey# (none) -> 2N7002ET1GOSCT-ND; Digikey/Mouser 2N7002ET1GOSCT-ND -> (none); Fabricante ON Semiconductor -> (none); Manf (none) -> ON Semiconductor; Manf# (none) -> 2N7002ET1G; Nro. parte 2N7002ET1G -> (none)
- Q2, Q3: Desc (none) -> MOSFET P-CH 30V 1.5A SOT23; Descripcion MOSFET P-CH 30V 1.5A SOT23 -> (none); Digikey# (none) -> BSS314PE H6327CT-ND; Digikey/Mouser BSS314PE H6327CT-ND -> (none); Fabricante Infineon -> (none); Manf (none) -> Infineon; Manf# (none) -> BSS314PE H6327; Nro. parte BSS314PE H6327 -> (none)
- R3, R4: Desc (none) -> RES SMD 100K OHM 1% 1/16W 0402; Descripcion RES SMD 100K OHM 1% 1/16W 0402 -> (none); Digikey# (none) -> 311-100KLRCT-ND; Digikey/Mouser 311-100KLRCT-ND -> (none); Fabricante Yageo -> (none); Manf (none) -> Yageo; Manf# (none) -> RC0402FR-07100KL; Nro. parte RC0402FR-07100KL -> (none)
Changed lines of the file:
@@
 F 2 "chip_rlc:r_0402" V 4530 4150 50  0001 C CNN
 F 3 "" H 4600 4150 50  0000 C CNN
-F 4 "RES SMD 100K OHM 1% 1/16W 0402" H 4600 4150 60  0001 C CNN "Descripcion"
-F 5 "Yageo" H 4600 4150 60  0001 C CNN "Fabricante"
-F 6 "RC0402FR-07100KL" H 4600 4150 60  0001 C CNN "Nro. parte"
-F 7 "311-100KLRCT-ND" H 4600 4150 60  0001 C CNN "Digikey/Mouser"
+F 4 "RES SMD 100K OHM 1% 1/16W 0402" H 4600 4150 60  0001 C CNN "Desc"
+F 5 "Yageo" H 4600 4150 60  0001 C CNN "Manf"
+F 6 "RC0402FR-07100KL" H 4600 4150 60  0001 C CNN "Manf#"
+F 7 "311-100KLRCT-ND" H 4600 4150 60  0001 C CNN "Digikey#"
 	1    4600 4150
 	1    0    0    -1
@@
 F 2 "chip_rlc:r_0402" V 4930 4150 50  0001 C CNN
 F 3 "" H 5000 4150 50  0000 C CNN
-F 4 "RES SMD 100K OHM 1% 1/16W 0402" H 5000 4150 60  0001 C CNN "Descripcion"
-F 5 "Yageo" H 5000 4150 60  0001 C CNN "Fabricante"
-F 6 "RC0402FR-07100KL" H 5000 4150 60  0001 C CNN "Nro. parte"
-F 7 "311-100KLRCT-ND" H 5000 4150 60  0001 C CNN "Digikey/Mouser"
+F 4 "RES SMD 100K OHM 1% 1/16W 0402" H 5000 4150 60  0001 C CNN "Desc"
+F 5 "Yageo" H 5000 4150 60  0001 C CNN "Manf"
+F 6 "RC0402FR-07100KL" H 5000 4150 60  0001 C CNN "Manf#"
+F 7 "311-100KLRCT-ND" H 5000 4150 60  0001 C CNN "Digikey#"
 	1    5000 4150
 	1    0    0    -1
@@
 F 2 "to-sod-sot:SOT-23" H 5650 4750 60  0001 C CNN
 F 3 "" H 5650 4750 60  0000 C CNN
-F 4 "MOSFET P-CH 30V 1.5A SOT23" H 5650 4750 60  0001 C CNN "Descripcion"
-F 5 "Infineon" H 5650 4750 60  0001 C CNN "Fabricante"
-F 6 "BSS314PE H6327" H 5650 4750 60  0001 C CNN "Nro. parte"
-F 7 "BSS314PE H6327CT-ND" H 5650 4750 60  0001 C CNN "Digikey/Mouser"
+F 4 "MOSFET P-CH 30V 1.5A SOT23" H 5650 4750 60  0001 C CNN "Desc"
+F 5 "Infineon" H 5650 4750 60  0001 C CNN "Manf"
+F 6 "BSS314PE H6327" H 5650 4750 60  0001 C CNN "Manf#"
+F 7 "BSS314PE H6327CT-ND" H 5650 4750 60  0001 C CNN "Digikey#"
 	1    5650 4750
 	0    1    1    0
@@
 F 2 "to-sod-sot:SOT-23" H 4900 4650 60  0001 C CNN
 F 3 "" H 4900 4650 60  0000 C CNN
-F 4 "MOSFET N-CH 60V 260MA SOT-23" H 4900 4650 60  0001 C CNN "Descripcion"
-F 5 "ON Semiconductor" H 4900 4650 60  0001 C CNN "Fabricante"
-F 6 "2N7002ET1G" H 4900 4650 60  0001 C CNN "Nro. parte"
-F 7 "2N7002ET1GOSCT-ND" H 4900 4650 60  0001 C CNN "Digikey/Mouser"
+F 4 "MOSFET N-CH 60V 260MA SOT-23" H 4900 4650 60  0001 C CNN "Desc"
+F 5 "ON Semiconductor" H 4900 4650 60  0001 C CNN "Manf"
+F 6 "2N7002ET1G" H 4900 4650 60  0001 C CNN "Manf#"
+F 7 "2N7002ET1GOSCT-ND" H 4900 4650 60  0001 C CNN "Digikey#"
 	1    4900 4650
 	1    0    0    -1
@@
 F 2 "to-sod-sot:SOT-23" H 6600 4750 60  0001 C CNN
 F 3 "" H 6600 4750 60  0000 C CNN
-F 4 "MOSFET P-CH 30V 1.5A SOT23" H 6600 4750 60  0001 C CNN "Descripcion"
-F 5 "Infineon" H 6600 4750 60  0001 C CNN "Fabricante"
-F 6 "BSS314PE H6327" H 6600 4750 60  0001 C CNN "Nro. parte"
-F 7 "BSS314PE H6327CT-ND" H 6600 4750 60  0001 C CNN "Digikey/Mouser"
+F 4 "MOSFET P-CH 30V 1.5A SOT23" H 6600 4750 60  0001 C CNN "Desc"
+F 5 "Infineon" H 6600 4750 60  0001 C CNN "Manf"
+F 6 "BSS314PE H6327" H 6600 4750 60  0001 C CNN "Manf#"
+F 7 "BSS314PE H6327CT-ND" H 6600 4750 60  0001 C CNN "Digikey#"
 	1    6600 4750
 	0    1    1    0
