File: KiCad Proyecto/Power_Supplies.sch (KiCad schematic (older format))
At the start: 19 parts, among them U1 TPS54202, U2 AZ1117EH-3.3TRG1

Commit message: fixed(temp) library problem
Parts:
- C1, C10, C11, C2, C3, C4, C5, C6, C7, C8, C9: symbol OBDII_IoT:C -> C
- D1: symbol OBDII_IoT:TVS -> TVS
- D2: symbol OBDII_IoT:D -> D
- F1: symbol OBDII_IoT:FUSE -> FUSE
- L1: symbol OBDII_IoT:L -> L
- R1, R2: symbol OBDII_IoT:R -> R
- U1: symbol OBDII_IoT:TPS54202 -> TPS54202
- U2: symbol OBDII_IoT:VOLT_REG -> VOLT_REG
Changed lines of the file:
@@
 EESchema Schematic File Version 2
-LIBS:power
-LIBS:PF_apiner-cache
+LIBS:OBDII_IoT
+LIBS:Connector
+LIBS:ESP32-footprints-Shem-Lib
+LIBS:ftdi
+LIBS:STN2120
 EELAYER 25 0
 EELAYER END
@@
 $EndDescr
 $Comp
-L OBDII_IoT:DLC_RAW #PWR09
+L DLC_RAW #PWR09
 U 1 1 5835BB34
 P 4950 2400
@@
 $EndComp
 $Comp
-L OBDII_IoT:C C1
+L C C1
 U 1 1 5835BB57
 P 4300 2700
@@
 $EndComp
 $Comp
-L OBDII_IoT:DLC #PWR010
+L DLC #PWR010
 U 1 1 5835BBB8
 P 5900 2400
@@
 $EndComp
 $Comp
-L OBDII_IoT:C C4
+L C C4
 U 1 1 5835BBD5
 P 5300 2700
@@
 $EndComp
 $Comp
-L OBDII_IoT:GND #PWR011
+L GND #PWR011
 U 1 1 5835BE13
 P 4300 2950
@@
 $EndComp
 $Comp
-L OBDII_IoT:TVS D1
+L TVS D1
 U 1 1 5835C003
 P 4950 2750
@@
 $EndComp
 $Comp
-L OBDII_IoT:D D2
+L D D2
 U 1 1 5835C0B1
 P 5150 2500
@@
 $EndComp
 $Comp
-L OBDII_IoT:FUSE F1
+L FUSE F1
 U 1 1 5835F7DA
 P 4600 2500
@@
 $EndComp
 $Comp
-L OBDII_IoT:TPS54202 U1
+L TPS54202 U1
 U 1 1 5835C29D
 P 4500 3800
@@
 $EndComp
 $Comp
-L OBDII_IoT:DLC #PWR012
+L DLC #PWR012
 U 1 1 5835C416
 P 3950 3550
@@
 $EndComp
 $Comp
-L OBDII_IoT:L L1
+L L L1
 U 1 1 5835C9FC
 P 5500 3650
@@
 $EndComp
 $Comp
-L OBDII_IoT:C C8
+L C C8
 U 1 1 5835CACB
 P 5700 3850
@@
 $EndComp
 $Comp
-L OBDII_IoT:+5V #PWR013
+L +5V #PWR013
 U 1 1 5836344D
 P 6000 3500
@@
 	4050 2500 4350 2500
 $Comp
-L OBDII_IoT:C C3
+L C C3
 U 1 1 588025EB
 P 5150 3650
@@
 $EndComp
 $Comp
-L OBDII_IoT:C C10
+L C C10
 U 1 1 589356C6
 P 6200 4050
@@
 Connection ~ 6200 4500
 $Comp
-L OBDII_IoT:R R1
+L R R1
 U 1 1 58A271C0
 P 6000 3850
@@
 $EndComp
 $Comp
-L OBDII_IoT:GND #PWR014
+L GND #PWR014
 U 1 1 58F7E73C
 P 4950 2950
@@
 $EndComp
 $Comp
-L OBDII_IoT:GND #PWR015
+L GND #PWR015
 U 1 1 58F7E773
 P 5900 2950
@@
 	5900 2950 5900 2850
 $Comp
-L OBDII_IoT:GND #PWR016
+L GND #PWR016
 U 1 1 58F7F16E
 P 5700 2950
@@
 $EndComp
 $Comp
-L OBDII_IoT:GND #PWR017
+L GND #PWR017
 U 1 1 58F7F1A5
 P 5500 2950
@@
 $EndComp
 $Comp
-L OBDII_IoT:GND #PWR018
+L GND #PWR018
 U 1 1 58F7F1DC
 P 5300 2950
@@
 	5700 2950 5700 2850
 $Comp
-L OBDII_IoT:C C6
+L C C6
 U 1 1 58F7FBBA
 P 5500 2700
@@
 $EndComp
 $Comp
-L OBDII_IoT:C C7
+L C C7
 U 1 1 58F7FBFE
 P 5700 2700
@@
 $EndComp
 $Comp
-L OBDII_IoT:C C9
+L C C9
 U 1 1 58F7FC44
 P 5900 2700
@@
 $EndComp
 $Comp
-L OBDII_IoT:C C2
+L C C2
 U 1 1 58F80648
 P 4450 5200
@@
 $EndComp
 $Comp
-L OBDII_IoT:C C11
+L C C11
 U 1 1 58F81C6B
 P 6450 4050
@@
 $EndComp
 $Comp
-L OBDII_IoT:GND #PWR019
+L GND #PWR019
 U 1 1 58F81EC8
 P 3950 4100
@@
 $EndComp
 $Comp
-L OBDII_IoT:GND #PWR020
+L GND #PWR020
 U 1 1 58F81EFF
 P 6000 4550
@@
 $EndComp
 $Comp
-L OBDII_IoT:VOLT_REG U2
+L VOLT_REG U2
 U 1 1 58F82CD2
 P 4900 4950
@@
 $EndComp
 $Comp
-L OBDII_IoT:+5V #PWR021
+L +5V #PWR021
 U 1 1 58F82E5C
 P 4450 4900
@@
 $EndComp
 $Comp
-L OBDII_IoT:C C5
+L C C5
 U 1 1 58F85AE2
 P 5400 5200
@@
 $EndComp
 $Comp
-L OBDII_IoT:+3.3V #PWR022
+L +3.3V #PWR022
 U 1 1 58F85D19
 P 5400 4900
@@
 $EndComp
 $Comp
-L OBDII_IoT:GND #PWR023
+L GND #PWR023
 U 1 1 58F85EE0
 P 4900 5450
@@
 $EndComp
 $Comp
-L OBDII_IoT:GND #PWR024
+L GND #PWR024
 U 1 1 58F85FA0
 P 4450 5450
@@
 $EndComp
 $Comp
-L OBDII_IoT:GND #PWR025
+L GND #PWR025
 U 1 1 58F85FD1
 P 5400 5450
@@
 Connection ~ 5400 4950
 $Comp
-L OBDII_IoT:R R2
+L R R2
 U 1 1 58F89868
 P 6000 4300
@@
 	4300 2400 4300 2550
 $Comp
-L OBDII_IoT:VIN #PWR026
+L VIN #PWR026
 U 1 1 58F9A73A
 P 4300 2400
@@
 	3950 3650 4050 3650
 $Comp
-L OBDII_IoT:PWR_FLAG #FLG027
+L PWR_FLAG #FLG027
 U 1 1 590B622B
 P 4050 2500
@@
 $EndComp
 $Comp
-L OBDII_IoT:PWR_FLAG #FLG028
+L PWR_FLAG #FLG028
 U 1 1 590B82D6
 P 4050 2850

Commit message: arreglando manquiadas
Other:
- note removed: "poner schotky de proteccion por el USB?\nen 5V y 3.3V"
Changed lines of the file:
@@
 EESchema Schematic File Version 2
-LIBS:OBDII_IoT
 LIBS:Connector
 LIBS:ESP32-footprints-Shem-Lib
 LIBS:ftdi
+LIBS:OBDII_IoT
 LIBS:STN2120
 LIBS:PF_apiner-cache
@@
 	4050 2900 4300 2900
 Connection ~ 4300 2900
-Text Notes 5350 3300 0    50   ~ 0
-poner schotky de proteccion por el USB?\nen 5V y 3.3V
 $EndSCHEMATC

Commit message: fixed fuse & wrong fields
Parts:
- C1: Desc (none) -> CAP CER 10000PF 25V C0G 0603; Descripcion CAP CER 10000PF 25V C0G 0603 -> (none); Digikey/Mouser 445-2664-1-ND -> (none); Fabricante TDK Corporation -> (none); Manf (none) -> TDK Corporation; Manf# (none) -> 445-2664-1-ND; Nro. parte C1608C0G1E103J080AA -> (none)
- C10, C11: Desc (none) -> CAP CER 10UF 6.3V X5R 0603; Descripcion CAP CER 10UF 6.3V X5R 0603 -> (none); Digikey/Mouser 587-1256-1-ND -> (none); Fabricante Taiyo Yuden -> (none); Manf (none) -> Taiyo Yuden; Manf# (none) -> 587-1256-1-ND; Nro. parte JMK107BJ106MA-T -> (none)
- C2, C3: Desc (none) -> CAP CER 0.1UF 10V X5R 0402; Descripcion CAP CER 0.1UF 10V X5R 0402 -> (none); Digikey/Mouser 311-1336-1-ND -> (none); Fabricante Yageo -> (none); Manf (none) -> Yageo; Manf# (none) -> 311-1336-1-ND; Nro. parte CC0402KRX5R6BB104 -> (none)
- C4, C6, C7, C9: Desc (none) -> 47µF ±20% 25V Ceramic Capacitor X5R 1206 (3216 Metric); Descripcion 47µF ±20% 25V Ceramic Capacitor X5R 1206 (3216 Metric) -> (none); Digikey/Mouser 445-8047-1-ND -> (none); Fabricante TDK Corporation -> (none); Manf (none) -> TDK Corporation; Manf# (none) -> 445-8047-1-ND; Nro. parte C3216X5R1E476M160AC -> (none)
- C5: Desc (none) -> CAP CER 1UF 6.3V X5R 0402; Descripcion CAP CER 1UF 6.3V X5R 0402 -> (none); Digikey/Mouser 587-1231-1-ND -> (none); Fabricante Taiyo Yuden -> (none); Manf (none) -> Taiyo Yuden; Manf# (none) -> 587-1231-1-ND; Nro. parte JMK105BJ105KV-F -> (none)
- C8: Desc (none) -> CAP CER 62PF 50V C0G/NPO 0402; Descripcion CAP CER 62PF 50V C0G/NPO 0402 -> (none); Digikey/Mouser 311-1674-1-ND -> (none); Fabricante Yageo -> (none); Manf (none) -> Yageo; Manf# (none) -> 311-1674-1-ND; Nro. parte CC0402JRNPO9BN620 -> (none)
- D1: Desc (none) -> TVS DIODE 14VWM 23.2VC SOD-123FL; Descripcion TVS DIODE 14VWM 23.2VC SOD-123FL -> (none); Digikey/Mouser SMF14A-TPMSCT-ND -> (none); Fabricante Micro Commercial Co -> (none); Manf (none) -> Micro Commercial Co; Manf# (none) -> SMF14A-TPMSCT-ND; Nro. parte SMF14A-TP -> (none)
- D2: Desc (none) -> DIODE SBR 30V 2A POWERDI123; Descripcion DIODE SBR 30V 2A POWERDI123 -> (none); Digikey/Mouser SBR2U30P1DICT-ND -> (none); Fabricante Diodes Incorporated -> (none); Manf (none) -> Diodes Incorporated; Manf# (none) -> SBR2U30P1DICT-ND; Nro. parte SBR2U30P1-7 -> (none)
- F1: Desc (none) -> FUSE BOARD MNT 2A 63VAC/VDC 1206; Descripcion FUSE BOARD MOUNT 2A 63VDC 1206 -> (none); Digikey# (none) -> F2570CT-ND; Digikey/Mouser 1206SFF200F/63-2CT-ND -> (none); Fabricante Littelfuse -> (none); Manf (none) -> Littelfuse Inc.; Manf# (none) -> 0468002.NR; Nro. parte 1206SFF200F/63-2 -> (none)
- L1: Desc (none) -> 10µH Shielded Wirewound Inductor 2.5A 58.6 mOhm Max Nonstan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; Descripcion 10µH Shielded Wirewound Inductor 2.5A 58.6 mOhm Max Nonstan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 -> (none); Digikey/Mouser SRN6045-100MCT-ND -> (none); Fabricante Bourns Inc -> (none); Manf (none) -> Bourns Inc; Manf# (none) -> SRN6045-100MCT-ND; Nro. parte SRN6045-100M -> (none)
- R1: Desc (none) -> RES SMD 100K OHM 1% 1/16W 0402; Descripcion RES SMD 100K OHM 1% 1/16W 0402 -> (none); Digikey/Mouser 311-100KLRCT-ND -> (none); Fabricante Yageo -> (none); Manf (none) -> Yageo; Manf# (none) -> 311-100KLRCT-ND; Nro. parte RC0402FR-07100KL -> (none)
- R2: Desc (none) -> RES SMD 13.7K OHM 1% 1/16W 0402; Descripcion RES SMD 13.7K OHM 1% 1/16W 0402 -> (none); Digikey/Mouser 311-13.7KLRCT-ND -> (none); Fabricante Yageo -> (none); Manf (none) -> Yageo; Manf# (none) -> 311-13.7KLRCT-ND; Nro. parte RC0402FR-0713K7L -> (none)
- U1: Desc (none) -> Buck Switching Regulator IC Positive Adjustable 0.596V 1 Ou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; Descripcion Buck Switching Regulator IC Positive Adjustable 0.596V 1 Ou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 -> (none); Digikey/Mouser 296-44151-1-ND -> (none); Fabricante Texas Instruments -> (none); Manf (none) -> Texas Instruments; Manf# (none) -> 296-44151-1-ND; Nro. parte TPS54202DDCT -> (none)
- U2: Desc (none) -> IC REG LDO 3.3V 1A SOT223; Descripcion IC REG LDO 3.3V 1A SOT223 -> (none); Digikey/Mouser AZ1117EH-3.3TRG1DICT-ND -> (none); Fabricante Diodes Incorporated -> (none); Manf (none) -> Diodes Incorporated; Manf# (none) -> AZ1117EH-3.3TRG1DICT-ND; Nro. parte AZ1117EH-3.3TRG1 -> (none)

Commit message: added screw holes
Parts:
- U1: Digikey# (none) -> 296-44396-1-ND; Manf# 296-44151-1-ND -> TPS54202DDCT
Other:
- note added: "poner infinitas vias\ndata tps #21"
Changed lines of the file:
@@
 F 2 "to-sod-sot:SOT-23-6" H 4500 4200 60  0001 C CNN
 F 3 "" H 4500 4200 60  0000 C CNN
-F 4 "Texas Instruments" H 4500 3800 60  0001 C CNN "Manf"
-F 5 "Buck Switching Regulator IC Positive Adjustable 0.596V 1 Output 2A SOT-23-6 Thin, TSOT-23-6" H 4500 3800 60  0001 C CNN "Desc"
+F 4 "Buck Switching Regulator IC Positive Adjustable 0.596V 1 Output 2A SOT-23-6 Thin, TSOT-23-6" H 4500 3800 60  0001 C CNN "Desc"
+F 5 "Texas Instruments" H 4500 3800 60  0001 C CNN "Manf"
 F 6 "TPS54202DDCT" H 4500 3800 60  0001 C CNN "Manf#"
-F 7 "296-44151-1-ND" H 4500 3800 60  0001 C CNN "Manf#"
+F 7 "296-44396-1-ND" H 4500 3800 60  0001 C CNN "Digikey#"
 	1    4500 3800
 	1    0    0    -1
@@
 	4050 2900 4300 2900
 Connection ~ 4300 2900
+Text Notes 5200 3300 0    60   ~ 0
+poner infinitas vias\ndata tps #21
 $EndSCHEMATC
