File: KiCad Proyecto/Voltage_Sense.sch (KiCad schematic (older format))
At the start: 4 parts

Commit message: fixed(temp) library problem
Parts:
- C12: symbol OBDII_IoT:C -> C
- D3: symbol OBDII_IoT:D_Schottky_BAT54SL -> D_Schottky_BAT54SL
- R5, R6: symbol OBDII_IoT:R -> R
Changed lines of the file:
@@
 EESchema Schematic File Version 2
-LIBS:power
-LIBS:PF_apiner-cache
+LIBS:OBDII_IoT
+LIBS:Connector
+LIBS:ESP32-footprints-Shem-Lib
+LIBS:ftdi
+LIBS:STN2120
 EELAYER 25 0
 EELAYER END
@@
 $EndDescr
 $Comp
-L OBDII_IoT:DLC_RAW #PWR040
+L DLC_RAW #PWR040
 U 1 1 582F295A
 P 5150 3350
@@
 $EndComp
 $Comp
-L OBDII_IoT:R R5
+L R R5
 U 1 1 582F3539
 P 5150 3650
@@
 $EndComp
 $Comp
-L OBDII_IoT:GND #PWR041
+L GND #PWR041
 U 1 1 582F35F0
 P 5150 4450
@@
 $EndComp
 $Comp
-L OBDII_IoT:GND #PWR042
+L GND #PWR042
 U 1 1 582F3A7C
 P 5650 4450
@@
 	5650 4200 5650 4450
 $Comp
-L OBDII_IoT:D_Schottky_BAT54SL D3
+L D_Schottky_BAT54SL D3
 U 1 1 583A9D5F
 P 5650 3900
@@
 Connection ~ 5350 3900
 $Comp
-L OBDII_IoT:R R6
+L R R6
 U 1 1 583AB1A6
 P 5150 4150
@@
 $EndComp
 $Comp
-L OBDII_IoT:PWR_FLAG #FLG043
+L PWR_FLAG #FLG043
 U 1 1 58498D94
 P 4900 3350
@@
 Connection ~ 5150 3400
 $Comp
-L OBDII_IoT:C C12
+L C C12
 U 1 1 58F8BB88
 P 4850 4150
@@
 $EndComp
 $Comp
-L OBDII_IoT:+3.3V #PWR044
+L +3.3V #PWR044
 U 1 1 58F8C1FD
 P 5650 3350

Commit message: fixed fuse & wrong fields
Parts:
- C12: Desc (none) -> CAP CER 0.1UF 10V X5R 0402; Descripcion CAP CER 0.1UF 10V X5R 0402 -> (none); Digikey# (none) -> 311-1336-1-ND; Digikey/Mouser 311-1336-1-ND -> (none); Fabricante Yageo -> (none); Manf (none) -> Yageo; Manf# (none) -> CC0402KRX5R6BB104; Nro. parte CC0402KRX5R6BB104 -> (none)
- D3: Desc (none) -> Diode Array 1 Pair Series Connection Schottky 30V 200mA (DC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; Descripcion Diode Array 1 Pair Series Connection Schottky 30V 200mA (DC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 -> (none); Digikey# (none) -> BAT54SLT1GOSCT-ND; Digikey/Mouser BAT54SLT1GOSCT-ND -> (none); Fabricante ON Semiconductor -> (none); Manf (none) -> ON Semiconductor; Manf# (none) -> BAT54SLT1G; Nro. parte BAT54SLT1G -> (none)
- R5: Desc (none) -> RES SMD 62K OHM 1% 1/16W 0402; Descripcion RES SMD 62K OHM 1% 1/16W 0402 -> (none); Digikey# (none) -> 311-62.0KLRCT-ND; Digikey/Mouser 311-62.0KLRCT-ND -> (none); Fabricante Yageo -> (none); Manf (none) -> Yageo; Manf# (none) -> RC0402FR-0762KL; Nro. parte RC0402FR-0762KL -> (none)
- R6: Desc (none) -> RES SMD 10K OHM 1% 1/16W 0402; Descripcion RES SMD 10K OHM 1% 1/16W 0402 -> (none); Digikey# (none) -> 311-10.0KLRCT-ND; Digikey/Mouser 311-10.0KLRCT-ND -> (none); Fabricante Yaego -> (none); Manf (none) -> Yaego; Manf# (none) -> RC0402FR-0710KL; Nro. parte RC0402FR-0710KL -> (none)
Changed lines of the file:
@@
 F 2 "chip_rlc:r_0402" V 5080 3650 50  0001 C CNN
 F 3 "" H 5150 3650 50  0000 C CNN
-F 4 "RES SMD 62K OHM 1% 1/16W 0402" H 5150 3650 60  0001 C CNN "Descripcion"
-F 5 "Yageo" H 5150 3650 60  0001 C CNN "Fabricante"
-F 6 "RC0402FR-0762KL" H 5150 3650 60  0001 C CNN "Nro. parte"
-F 7 "311-62.0KLRCT-ND" H 5150 3650 60  0001 C CNN "Digikey/Mouser"
+F 4 "RES SMD 62K OHM 1% 1/16W 0402" H 5150 3650 60  0001 C CNN "Desc"
+F 5 "Yageo" H 5150 3650 60  0001 C CNN "Manf"
+F 6 "RC0402FR-0762KL" H 5150 3650 60  0001 C CNN "Manf#"
+F 7 "311-62.0KLRCT-ND" H 5150 3650 60  0001 C CNN "Digikey#"
 	1    5150 3650
 	-1   0    0    1
@@
 F 2 "to-sod-sot:SOT-23" H 5650 3900 50  0001 C CNN
 F 3 "" H 5650 3900 50  0000 C CNN
-F 4 "Diode Array 1 Pair Series Connection Schottky 30V 200mA (DC) Surface Mount TO-236-3, SC-59, SOT-23-3" H 5650 3900 60  0001 C CNN "Descripcion"
-F 5 "ON Semiconductor" H 5650 3900 60  0001 C CNN "Fabricante"
-F 6 "BAT54SLT1G" H 5650 3900 60  0001 C CNN "Nro. parte"
-F 7 "BAT54SLT1GOSCT-ND" H 5650 3900 60  0001 C CNN "Digikey/Mouser"
+F 4 "Diode Array 1 Pair Series Connection Schottky 30V 200mA (DC) Surface Mount TO-236-3, SC-59, SOT-23-3" H 5650 3900 60  0001 C CNN "Desc"
+F 5 "ON Semiconductor" H 5650 3900 60  0001 C CNN "Manf"
+F 6 "BAT54SLT1G" H 5650 3900 60  0001 C CNN "Manf#"
+F 7 "BAT54SLT1GOSCT-ND" H 5650 3900 60  0001 C CNN "Digikey#"
 	1    5650 3900
 	0    1    -1   0
@@
 F 2 "chip_rlc:r_0402" V 5080 4150 50  0001 C CNN
 F 3 "" H 5150 4150 50  0000 C CNN
-F 4 "RES SMD 10K OHM 1% 1/16W 0402" H 5150 4150 60  0001 C CNN "Descripcion"
-F 5 "Yaego" H 5150 4150 60  0001 C CNN "Fabricante"
-F 6 "RC0402FR-0710KL" H 5150 4150 60  0001 C CNN "Nro. parte"
-F 7 "311-10.0KLRCT-ND" H 5150 4150 60  0001 C CNN "Digikey/Mouser"
+F 4 "RES SMD 10K OHM 1% 1/16W 0402" H 5150 4150 60  0001 C CNN "Desc"
+F 5 "Yaego" H 5150 4150 60  0001 C CNN "Manf"
+F 6 "RC0402FR-0710KL" H 5150 4150 60  0001 C CNN "Manf#"
+F 7 "311-10.0KLRCT-ND" H 5150 4150 60  0001 C CNN "Digikey#"
 	1    5150 4150
 	1    0    0    -1
@@
 F 2 "chip_rlc:c_0402" H 4888 4000 50  0001 C CNN
 F 3 "" H 4850 4150 50  0000 C CNN
-F 4 "CAP CER 0.1UF 10V X5R 0402" H 4850 4150 60  0001 C CNN "Descripcion"
-F 5 "Yageo" H 4850 4150 60  0001 C CNN "Fabricante"
-F 6 "CC0402KRX5R6BB104" H 4850 4150 60  0001 C CNN "Nro. parte"
-F 7 "311-1336-1-ND" H 4850 4150 60  0001 C CNN "Digikey/Mouser"
+F 4 "CAP CER 0.1UF 10V X5R 0402" H 4850 4150 60  0001 C CNN "Desc"
+F 5 "Yageo" H 4850 4150 60  0001 C CNN "Manf"
+F 6 "CC0402KRX5R6BB104" H 4850 4150 60  0001 C CNN "Manf#"
+F 7 "311-1336-1-ND" H 4850 4150 60  0001 C CNN "Digikey#"
 	1    4850 4150
 	1    0    0    -1
