File: KiCad_Proyecto/PF_apiner.sch (KiCad schematic (older format))
At the start: 8 parts, among them J1 OBDII Header, J2 Conn_01x05

Commit message: se viene
Connections:
- net MicroM4/UART0_RX: now also J2.2 (Pin_2); no longer J2.3 (Pin_3)
- net MicroM4/UART0_TX: now also J2.3 (Pin_3); no longer J2.2 (Pin_2)
- no-connect marks 4 -> 8
Changed lines of the file:
@@
 F0 "MicroM4" 40
 F1 "MicroM4.sch" 40
-F2 "UART0_TX" O R 8250 2600 50
+F2 "UART0_TX" O R 8250 2700 50
 F3 "UART1_TX" O L 7050 3150 50
-F4 "UART0_RX" I R 8250 2700 50
+F4 "UART0_RX" I R 8250 2600 50
 F5 "UART1_RX" I L 7050 3050 50
 F6 "STN_SLEEP" O L 7050 2900 50
@@
 	8900 2900 8900 3050
 Wire Wire Line
-	8250 2600 9350 2600
-Wire Wire Line
-	8250 2700 9350 2700
-Wire Wire Line
 	8550 2800 9350 2800
 Wire Wire Line
@@
 	1    0    0    -1
 $EndComp
+NoConn ~ 10050 3200
+NoConn ~ 10050 3350
+NoConn ~ 10050 3500
+NoConn ~ 10050 3650
+Wire Wire Line
+	8250 2600 9350 2600
+Wire Wire Line
+	9350 2700 8250 2700
 $EndSCHEMATC
