File: KiCad_Proyecto/PF_apiner.sch (KiCad schematic (older format))
At the start: 8 parts, among them J1 OBDII Header, J2 Conn_01x05

Commit message: todos los .sch arreglados
Parts:
- C35: symbol PF_apiner-rescue:C-OBDII_IoT1 -> OBDII_IoT:C
- D12: symbol PF_apiner-rescue:D_Schot-OBDII_IoT1 -> OBDII_IoT:D_Schot
- H1, H2, H3, H4: symbol PF_apiner-rescue:PCB_HOLE-OBDII_IoT1 -> OBDII_IoT:PCB_HOLE
- J1: symbol PF_apiner-rescue:CONN_2X16_OBDII-OBDII_IoT1 -> OBDII_IoT:CONN_2X16_OBDII
- J2: symbol PF_apiner-rescue:Conn_01x05-Connector1 -> Connector:Conn_01x05
Changed lines of the file:
@@
 EESchema Schematic File Version 4
 LIBS:PF_apiner-cache
-EELAYER 29 0
+EELAYER 26 0
 EELAYER END
 $Descr A4 11693 8268
@@
 	12150 9650 12250 9750
 $Comp
-L PF_apiner-rescue:GND-OBDII_IoT1 #PWR01
+L OBDII_IoT:GND #PWR01
 U 1 1 58F8F97A
 P 1550 4150
@@
 $EndComp
 $Comp
-L PF_apiner-rescue:CONN_2X16_OBDII-OBDII_IoT1 J1
+L OBDII_IoT:CONN_2X16_OBDII J1
 U 1 1 58F8F983
 P 1250 3350
@@
 $EndSheet
 $Comp
-L PF_apiner-rescue:VIN-OBDII_IoT1 #PWR02
+L OBDII_IoT:VIN #PWR02
 U 1 1 58F9B79D
 P 1550 2550
@@
 El UART0 va al USB, el resto hay que configurarlos
 $Comp
-L PF_apiner-rescue:C-OBDII_IoT1 C?
+L OBDII_IoT:C C?
 U 1 1 5B8838EA
 P 10000 4600
@@
 $EndComp
 $Comp
-L PF_apiner-rescue:GND-OBDII_IoT1 #PWR?
+L OBDII_IoT:GND #PWR?
 U 1 1 5B883919
 P 10000 4850
@@
 $EndComp
 $Comp
-L PF_apiner-rescue:+5V_USB-OBDII_IoT1 #U04
+L OBDII_IoT:+5V_USB #U04
 U 1 1 5B88F65F
 P 9250 2300
@@
 $EndComp
 $Comp
-L PF_apiner-rescue:+5V-OBDII_IoT1 #PWR?
+L OBDII_IoT:+5V #PWR?
 U 1 1 5B8A5F5E
 P 10000 4250
@@
 $EndComp
 $Comp
-L PF_apiner-rescue:+5V_USB-OBDII_IoT1 U?
+L OBDII_IoT:+5V_USB U?
 U 1 1 5B8A5F68
 P 10650 4250
@@
 $EndComp
 $Comp
-L PF_apiner-rescue:GND-OBDII_IoT1 #PWR?
+L OBDII_IoT:GND #PWR?
 U 1 1 5B8BA0D1
 P 8900 3050
@@
 $EndComp
 $Comp
-L PF_apiner-rescue:D_Schot-OBDII_IoT1 D?
+L OBDII_IoT:D_Schot D?
 U 1 1 5B8CB262
 P 10350 4350
@@
 $EndComp
 $Comp
-L PF_apiner-rescue:PWR_FLAG-OBDII_IoT1 #FLG08
+L OBDII_IoT:PWR_FLAG #FLG08
 U 1 1 5BA598FF
 P 9350 2200
@@
 	9350 2200 9350 2400
 $Comp
-L PF_apiner-rescue:Conn_01x05-Connector1 J2
+L Connector:Conn_01x05 J2
 U 1 1 5BCA1F49
 P 9550 2700
@@
 	10000 4350 10250 4350
 $Comp
-L PF_apiner-rescue:PCB_HOLE-OBDII_IoT1 H4
+L OBDII_IoT:PCB_HOLE H4
 U 1 1 5BDBC2D4
 P 10050 3650
@@
 $EndComp
 $Comp
-L PF_apiner-rescue:PCB_HOLE-OBDII_IoT1 H3
+L OBDII_IoT:PCB_HOLE H3
 U 1 1 5BDBD6A0
 P 10050 3500
@@
 $EndComp
 $Comp
-L PF_apiner-rescue:PCB_HOLE-OBDII_IoT1 H2
+L OBDII_IoT:PCB_HOLE H2
 U 1 1 5BDBD82A
 P 10050 3350
@@
 $EndComp
 $Comp
-L PF_apiner-rescue:PCB_HOLE-OBDII_IoT1 H1
+L OBDII_IoT:PCB_HOLE H1
 U 1 1 5BDBD9BA
 P 10050 3200
