File: KiCad_Proyecto/MicroM4.sch (KiCad schematic (older format))
At the start: 8 parts, among them SW1 SW_RESET, SW2 SW_BOOT, U14 ESP32-WROOM

Commit message: se viene
Parts:
- added R54: 10K, chip_rlc:r_0402, symbol R
Connections:
- net +3.3V: now also R54.2
- net BOOT: now reaches SW2.1 (A), SW2.2 (B), U14.25 (IO0)
- net BOOT: now also R54.1
Other:
- moved on the sheet: SW2
Changed lines of the file:
@@
 Text HLabel 4350 3600 0    50   Output ~ 0
 STN_RESET
-Text Label 6850 3550 0    50   ~ 0
+Text Label 6650 3550 0    50   ~ 0
 UART2_TX
-Text Label 6850 3650 0    50   ~ 0
+Text Label 6650 3650 0    50   ~ 0
 UART2_RX
-Text Notes 7400 4050 0    50   ~ 0
+Text Notes 8600 4000 0    50   ~ 0
 PAG 10\npull-up interno\nGPIO 0 -> 0: DOWNLOAD BOOT\nGPIO 0 -> 1: SPI BOOT
 Text Notes 6250 4800 0    50   ~ 0
@@
 NoConn ~ 5900 4450
 NoConn ~ 6550 3750
-NoConn ~ 6550 3450
 NoConn ~ 6550 3350
 NoConn ~ 6550 3250
@@
 Wire Wire Line
 	4350 3500 4700 3500
-Wire Wire Line
-	6550 3850 7100 3850
 $Comp
 L GND #PWR0127
 U 1 1 5B9BDD0C
-P 7000 4450
-F 0 "#PWR0127" H 7000 4200 50  0001 C CNN
-F 1 "GND" H 7005 4277 50  0001 C CNN
-F 2 "" H 7000 4450 50  0000 C CNN
-F 3 "" H 7000 4450 50  0000 C CNN
-	1    7000 4450
+P 8200 4400
+F 0 "#PWR0127" H 8200 4150 50  0001 C CNN
+F 1 "GND" H 8205 4227 50  0001 C CNN
+F 2 "" H 8200 4400 50  0000 C CNN
+F 3 "" H 8200 4400 50  0000 C CNN
+	1    8200 4400
 	1    0    0    -1
 $EndComp
@@
 L SW_SPST SW2
 U 1 1 5B9C003A
-P 7100 4150
-F 0 "SW2" H 7100 4320 50  0000 C CNN
-F 1 "SW_BOOT" H 7100 3950 50  0000 C CNN
-F 2 "misc:TACT_SMD_4.5X4.5" H 7100 4150 50  0001 C CNN
-F 3 "" H 7100 4150 50  0001 C CNN
-F 4 "Tactile Switch SPST-NO Top Actuated Surface Mount" H 7100 4150 60  0001 C CNN "Desc"
-F 5 "E-Switch" H 7100 4150 60  0001 C CNN "Manf"
-F 6 "TL3305AF160QG" H 7100 4150 60  0001 C CNN "Manf#"
-F 7 "EG5350CT-ND" H 7100 4150 60  0001 C CNN "Digikey#"
-	1    7100 4150
+P 8300 4100
+F 0 "SW2" H 8300 4270 50  0000 C CNN
+F 1 "SW_BOOT" H 8300 3900 50  0000 C CNN
+F 2 "misc:TACT_SMD_4.5X4.5" H 8300 4100 50  0001 C CNN
+F 3 "" H 8300 4100 50  0001 C CNN
+F 4 "Tactile Switch SPST-NO Top Actuated Surface Mount" H 8300 4100 60  0001 C CNN "Desc"
+F 5 "E-Switch" H 8300 4100 60  0001 C CNN "Manf"
+F 6 "TL3305AF160QG" H 8300 4100 60  0001 C CNN "Manf#"
+F 7 "EG5350CT-ND" H 8300 4100 60  0001 C CNN "Digikey#"
+	1    8300 4100
 	0    1    1    0
 $EndComp
 Wire Wire Line
-	7000 3850 7000 3900
-Wire Wire Line
-	7100 3850 7100 3900
-Connection ~ 7000 3850
-Wire Wire Line
-	7000 4400 7000 4450
-Wire Wire Line
-	7000 4450 7100 4450
-Wire Wire Line
-	7100 4450 7100 4400
+	8300 3700 8300 3850
+Wire Wire Line
+	8200 4350 8200 4400
+Wire Wire Line
+	8200 4400 8300 4400
+Wire Wire Line
+	8300 4400 8300 4350
 Wire Wire Line
 	3350 3000 3350 2900
@@
 	6100 4600 6100 4450
 NoConn ~ 6000 4450
+$Comp
+L +3.3V #PWR0131
+U 1 1 5BE1DF37
+P 8300 3300
+F 0 "#PWR0131" H 8300 3390 20  0001 C CNN
+F 1 "+3.3V" H 8296 3428 30  0000 C CNN
+F 2 "" H 8300 3300 60  0000 C CNN
+F 3 "" H 8300 3300 60  0000 C CNN
+	1    8300 3300
+	1    0    0    -1
+$EndComp
+Wire Wire Line
+	8300 3300 8300 3400
+$Comp
+L R R54
+U 1 1 5BE20C64
+P 8300 3550
+F 0 "R54" V 8350 3350 50  0000 C CNN
+F 1 "10K" V 8300 3550 50  0000 C CNN
+F 2 "chip_rlc:r_0402" V 8230 3550 50  0001 C CNN
+F 3 "" H 8300 3550 50  0000 C CNN
+F 4 "Yageo" H 8300 3550 60  0001 C CNN "Manf"
+F 5 "RES SMD 10K OHM 5% 1/16W 0402" H 8300 3550 60  0001 C CNN "Desc"
+F 6 "RC0402JR-0710KL" H 8300 3550 60  0001 C CNN "Manf#"
+F 7 "311-10KJRCT-ND" H 8300 3550 60  0001 C CNN "Digikey#"
+	1    8300 3550
+	-1   0    0    1
+$EndComp
+Text Label 6650 3850 0    50   ~ 0
+BOOT
+Wire Wire Line
+	6550 3850 6650 3850
+Wire Wire Line
+	8050 3750 8300 3750
+Wire Wire Line
+	8200 3750 8200 3850
+Connection ~ 8300 3750
+Text Label 8050 3750 2    50   ~ 0
+BOOT
+Connection ~ 8200 3750
+NoConn ~ 6550 3450
 $EndSCHEMATC

Commit message: ruteado terminado listo para rev
Connections:
- net PWR_SAVE: now also U14.28 (IO17); no longer U14.8 (IO32)
- net STN_SLEEP: now also U14.33 (IO21); no longer U14.9 (IO33)
Changed lines of the file:
@@
 Wire Wire Line
 	5500 4450 5500 4850
-Text HLabel 4350 3400 0    50   Input ~ 0
+Text HLabel 7050 3550 2    50   Input ~ 0
 PWR_SAVE
-Text HLabel 4350 3500 0    50   Output ~ 0
+Text HLabel 7000 3050 2    50   Output ~ 0
 STN_SLEEP
 Text HLabel 4350 3600 0    50   Output ~ 0
 STN_RESET
-Text Label 6650 3550 0    50   ~ 0
-UART2_TX
-Text Label 6650 3650 0    50   ~ 0
-UART2_RX
 Text Notes 8600 4000 0    50   ~ 0
 PAG 10\npull-up interno\nGPIO 0 -> 0: DOWNLOAD BOOT\nGPIO 0 -> 1: SPI BOOT
@@
 $EndComp
 Wire Wire Line
-	4350 3400 4700 3400
-Wire Wire Line
 	4350 3600 4700 3600
 NoConn ~ 4700 3000
@@
 NoConn ~ 6550 3350
 NoConn ~ 6550 3250
-NoConn ~ 6550 3050
 NoConn ~ 6550 2750
 NoConn ~ 6550 2650
-NoConn ~ 6550 3550
 NoConn ~ 6550 3650
-Wire Wire Line
-	4350 3500 4700 3500
 $Comp
 L GND #PWR0127
@@
 Connection ~ 8200 3750
 NoConn ~ 6550 3450
+Wire Wire Line
+	6550 3050 7000 3050
+NoConn ~ 4700 3400
+Wire Wire Line
+	6550 3550 7050 3550
+NoConn ~ 4700 3500
 $EndSCHEMATC
