File: KiCad_Proyecto/MicroM4.sch (KiCad schematic (older format))
At the start: 12 parts, among them SW1 SW_RESET, SW2 SW_BOOT, U14 ESP32-WROOM

Commit message: todos los .sch arreglados
Parts:
- C34: symbol C -> OBDII_IoT:C
- C36, C37, C38: symbol PF_apiner-rescue:C-OBDII_IoT1 -> OBDII_IoT:C
- DS1: symbol LED -> OBDII_IoT:LED
- R52, R53, R54: symbol PF_apiner-rescue:R-OBDII_IoT1 -> OBDII_IoT:R
- R55: symbol R -> OBDII_IoT:R
- SW1, SW2: symbol PF_apiner-rescue:SW_SPST-OBDII_IoT1 -> OBDII_IoT:SW_SPST
- U14: symbol PF_apiner-rescue:ESP32-WROOM-ESP32-footprints-Shem-Lib1 -> ESP32-footprints-Shem-Lib:ESP32-WROOM
Connections:
- wire segments 44 -> 58
Changed lines of the file:
@@
 EESchema Schematic File Version 4
 LIBS:PF_apiner-cache
-EELAYER 29 0
+EELAYER 26 0
 EELAYER END
 $Descr A4 11693 8268
@@
 $EndDescr
 $Comp
-L PF_apiner-rescue:ESP32-WROOM-ESP32-footprints-Shem-Lib1 U14
+L ESP32-footprints-Shem-Lib:ESP32-WROOM U14
 U 1 1 5B862489
 P 5650 3400
@@
 $EndComp
 $Comp
-L PF_apiner-rescue:+3.3V-OBDII_IoT1 #PWR0120
+L OBDII_IoT:+3.3V #PWR0120
 U 1 1 5B862539
 P 4500 2300
@@
 NoConn ~ 6550 3150
 $Comp
-L PF_apiner-rescue:GND-OBDII_IoT1 #PWR0121
+L OBDII_IoT:GND #PWR0121
 U 1 1 5B862710
 P 6750 4100
@@
 	6550 4050 6750 4050
 Wire Wire Line
-	6750 3950 6750 4100
-$Comp
-L PF_apiner-rescue:GND-OBDII_IoT1 #PWR0122
+	6750 3950 6750 4050
+$Comp
+L OBDII_IoT:GND #PWR0122
 U 1 1 5B86275E
 P 5200 4550
@@
 $EndComp
 $Comp
-L PF_apiner-rescue:GND-OBDII_IoT1 #PWR0123
+L OBDII_IoT:GND #PWR0123
 U 1 1 5B86276B
 P 4600 4150
@@
 $EndComp
 Wire Wire Line
-	4600 4000 4600 4150
+	4600 4000 4600 4100
 Wire Wire Line
 	4600 4100 4700 4100
@@
 	6550 2850 7000 2850
 Wire Wire Line
-	6550 2950 7000 2950
-Wire Wire Line
-	3600 2450 4000 2450
-$Comp
-L PF_apiner-rescue:GND-OBDII_IoT1 #PWR0124
+	6550 2950 6900 2950
+$Comp
+L OBDII_IoT:GND #PWR0124
 U 1 1 5B862FB4
-P 3800 2450
-F 0 "#PWR0124" H 3800 2200 50  0001 C CNN
-F 1 "GND" H 3805 2277 50  0001 C CNN
-F 2 "" H 3800 2450 50  0000 C CNN
-F 3 "" H 3800 2450 50  0000 C CNN
-	1    3800 2450
-	1    0    0    -1
-$EndComp
-Connection ~ 3800 2450
-Wire Wire Line
-	3600 2150 4000 2150
-$Comp
-L PF_apiner-rescue:+3.3V-OBDII_IoT1 #PWR0125
+P 3800 2500
+F 0 "#PWR0124" H 3800 2250 50  0001 C CNN
+F 1 "GND" H 3805 2327 50  0001 C CNN
+F 2 "" H 3800 2500 50  0000 C CNN
+F 3 "" H 3800 2500 50  0000 C CNN
+	1    3800 2500
+	1    0    0    -1
+$EndComp
+$Comp
+L OBDII_IoT:+3.3V #PWR0125
 U 1 1 5B86325C
-P 3800 2150
-F 0 "#PWR0125" H 3800 2240 20  0001 C CNN
-F 1 "+3.3V" H 3796 2278 30  0000 C CNN
-F 2 "" H 3800 2150 60  0000 C CNN
-F 3 "" H 3800 2150 60  0000 C CNN
-	1    3800 2150
-	1    0    0    -1
-$EndComp
-Connection ~ 3800 2150
+P 3800 2050
+F 0 "#PWR0125" H 3800 2140 20  0001 C CNN
+F 1 "+3.3V" H 3796 2178 30  0000 C CNN
+F 2 "" H 3800 2050 60  0000 C CNN
+F 3 "" H 3800 2050 60  0000 C CNN
+	1    3800 2050
+	1    0    0    -1
+$EndComp
 Wire Wire Line
 	4700 2350 4700 2800
 $Comp
-L PF_apiner-rescue:GND-OBDII_IoT1 #PWR0126
+L OBDII_IoT:GND #PWR0126
 U 1 1 5B8638AE
 P 4250 3250
@@
 $EndComp
 Wire Wire Line
-	3050 2900 4700 2900
+	3050 2900 3350 2900
 Text HLabel 7000 2850 2    50   Output ~ 0
 UART0_TX
@@
 RESET
 $Comp
-L PF_apiner-rescue:C-OBDII_IoT1 C?
+L OBDII_IoT:C C?
 U 1 1 5B8CBC06
 P 4000 2300
@@
 $EndComp
 $Comp
-L PF_apiner-rescue:C-OBDII_IoT1 C?
+L OBDII_IoT:C C?
 U 1 1 5B8CBF7F
 P 4250 3100
@@
 $EndComp
 $Comp
-L PF_apiner-rescue:C-OBDII_IoT1 C?
+L OBDII_IoT:C C?
 U 1 1 5B8D3E2F
 P 3600 2300
@@
 $EndComp
 $Comp
-L PF_apiner-rescue:R-OBDII_IoT1 R?
+L OBDII_IoT:R R?
 U 1 1 5B8D4B64
 P 4500 2550
@@
 NoConn ~ 6550 3650
 $Comp
-L PF_apiner-rescue:GND-OBDII_IoT1 #PWR0127
+L OBDII_IoT:GND #PWR0127
 U 1 1 5B9BDD0C
 P 8200 4400
@@
 Connection ~ 6750 4050
 $Comp
-L PF_apiner-rescue:GND-OBDII_IoT1 #PWR0128
+L OBDII_IoT:GND #PWR0128
 U 1 1 5B9BDFD1
 P 6100 4600
@@
 $EndComp
 $Comp
-L PF_apiner-rescue:R-OBDII_IoT1 R53
+L OBDII_IoT:R R53
 U 1 1 5B9C04A8
 P 6900 2600
@@
 Connection ~ 6900 2950
 $Comp
-L PF_apiner-rescue:+3.3V-OBDII_IoT1 #PWR0129
+L OBDII_IoT:+3.3V #PWR0129
 U 1 1 5B9C0576
 P 6900 2350
@@
 Connection ~ 3350 2900
 $Comp
-L PF_apiner-rescue:GND-OBDII_IoT1 #PWR0130
+L OBDII_IoT:GND #PWR0130
 U 1 1 5B9BE7F3
 P 3350 3600
@@
 	3350 3600 3350 3500
 $Comp
-L PF_apiner-rescue:SW_SPST-OBDII_IoT1 SW2
+L OBDII_IoT:SW_SPST SW2
 U 1 1 5B9C003A
 P 8300 4100
@@
 $EndComp
 Wire Wire Line
-	8300 3700 8300 3850
+	8300 3700 8300 3750
 Wire Wire Line
 	8200 4350 8200 4400
 Wire Wire Line
-	8200 4400 8650 4400
+	8200 4400 8300 4400
 Wire Wire Line
 	8300 4400 8300 4350
@@
 	3450 3600 3350 3600
 $Comp
-L PF_apiner-rescue:SW_SPST-OBDII_IoT1 SW1
+L OBDII_IoT:SW_SPST SW1
 U 1 1 5B9C0668
 P 3450 3250
@@
 $EndComp
 Wire Wire Line
-	4500 2300 4500 2400
+	4500 2300 4500 2350
 Wire Wire Line
 	4500 2350 4700 2350
@@
 NoConn ~ 6000 4450
 $Comp
-L PF_apiner-rescue:+3.3V-OBDII_IoT1 #PWR0131
+L OBDII_IoT:+3.3V #PWR0131
 U 1 1 5BE1DF37
 P 8300 3300
@@
 	8300 3300 8300 3400
 $Comp
-L PF_apiner-rescue:R-OBDII_IoT1 R54
+L OBDII_IoT:R R54
 U 1 1 5BE20C64
 P 8300 3550
@@
 	6550 3850 6650 3850
 Wire Wire Line
-	8050 3750 8650 3750
+	8050 3750 8200 3750
 Wire Wire Line
 	8200 3750 8200 3850
@@
 NoConn ~ 4700 3500
 $Comp
-L C C34
+L OBDII_IoT:C C34
 U 1 1 5D48B20D
 P 8650 4100
@@
 Connection ~ 8300 4400
 $Comp
-L R R55
+L OBDII_IoT:R R55
 U 1 1 5D491F3F
 P 3950 4900
@@
 $EndComp
 $Comp
-L LED DS1
+L OBDII_IoT:LED DS1
 U 1 1 5D491FC2
 P 3950 5250
@@
 $EndComp
 $Comp
-L GND #PWR0132
+L OBDII_IoT:GND #PWR0132
 U 1 1 5D492137
 P 3950 5450
@@
 Text Label 3950 4650 0    60   ~ 0
 Led_Status
+Wire Wire Line
+	4600 4100 4600 4150
+Wire Wire Line
+	6750 4050 6750 4100
+Wire Wire Line
+	6900 2950 7000 2950
+Wire Wire Line
+	3350 2900 3450 2900
+Wire Wire Line
+	3450 2900 4250 2900
+Wire Wire Line
+	4500 2350 4500 2400
+Wire Wire Line
+	4500 2900 4700 2900
+Wire Wire Line
+	4250 2900 4500 2900
+Wire Wire Line
+	8300 3750 8300 3850
+Wire Wire Line
+	8300 3750 8650 3750
+Wire Wire Line
+	8200 3750 8300 3750
+Wire Wire Line
+	8300 4400 8650 4400
+Wire Wire Line
+	3600 2450 4000 2450
+Wire Wire Line
+	3600 2150 3800 2150
+Wire Wire Line
+	3800 2050 3800 2150
+Connection ~ 3800 2150
+Wire Wire Line
+	3800 2150 4000 2150
 $EndSCHEMATC
