File: KiCad_Proyecto/ISO_Transceiver.sch (KiCad schematic (older format))
At the start: 16 parts, among them Q4 MMBT3904, Q5 MMBT3904, U3 LM339

Commit message: todos los .sch arreglados
Parts:
- C13, C14, C15: symbol PF_apiner-rescue:C-OBDII_IoT1 -> OBDII_IoT:C
- D4, D5: symbol PF_apiner-rescue:D_Schottky_BAT54SL-OBDII_IoT1 -> OBDII_IoT:D_Schottky_BAT54SL
- Q4, Q5: symbol PF_apiner-rescue:NPN-OBDII_IoT1 -> OBDII_IoT:NPN
- R10, R11, R12, R13, R14, R7, R8, R9: symbol PF_apiner-rescue:R-OBDII_IoT1 -> OBDII_IoT:R
- U3: symbol PF_apiner-rescue:LM339-OBDII_IoT1 -> OBDII_IoT:LM339
Changed lines of the file:
@@
 EESchema Schematic File Version 4
 LIBS:PF_apiner-cache
-EELAYER 29 0
+EELAYER 26 0
 EELAYER END
 $Descr A4 11693 8268
@@
 K-LINE
 $Comp
-L PF_apiner-rescue:LM339-OBDII_IoT1 U3
+L OBDII_IoT:LM339 U3
 U 1 1 58FAFC7B
 P 4800 4700
@@
 $EndComp
 $Comp
-L PF_apiner-rescue:R-OBDII_IoT1 R10
+L OBDII_IoT:R R10
 U 1 1 58FB19FB
 P 4150 2650
@@
 $EndComp
 $Comp
-L PF_apiner-rescue:NPN-OBDII_IoT1 Q4
+L OBDII_IoT:NPN Q4
 U 1 1 58FB1A06
 P 4050 3150
@@
 $EndComp
 $Comp
-L PF_apiner-rescue:R-OBDII_IoT1 R8
+L OBDII_IoT:R R8
 U 1 1 58FB1A1C
 P 3650 4400
@@
 $EndComp
 $Comp
-L PF_apiner-rescue:D_Schottky_BAT54SL-OBDII_IoT1 D4
+L OBDII_IoT:D_Schottky_BAT54SL D4
 U 1 1 58FB2C23
 P 4100 6100
@@
 $EndComp
 $Comp
-L PF_apiner-rescue:DLC_SW-OBDII_IoT1 #PWR045
+L OBDII_IoT:DLC_SW #PWR045
 U 1 1 58FB4559
 P 4150 2400
@@
 $EndComp
 $Comp
-L PF_apiner-rescue:R-OBDII_IoT1 R7
+L OBDII_IoT:R R7
 U 1 1 58FB45DB
 P 3650 3150
@@
 $EndComp
 $Comp
-L PF_apiner-rescue:GND-OBDII_IoT1 #PWR046
+L OBDII_IoT:GND #PWR046
 U 1 1 58FB47BB
 P 4150 3450
@@
 $EndComp
 $Comp
-L PF_apiner-rescue:R-OBDII_IoT1 R14
+L OBDII_IoT:R R14
 U 1 1 58FB4DD5
 P 5950 2650
@@
 $EndComp
 $Comp
-L PF_apiner-rescue:NPN-OBDII_IoT1 Q5
+L OBDII_IoT:NPN Q5
 U 1 1 58FB4DDF
 P 5850 3150
@@
 $EndComp
 $Comp
-L PF_apiner-rescue:DLC_SW-OBDII_IoT1 #PWR047
+L OBDII_IoT:DLC_SW #PWR047
 U 1 1 58FB4DE5
 P 5950 2400
@@
 $EndComp
 $Comp
-L PF_apiner-rescue:R-OBDII_IoT1 R13
+L OBDII_IoT:R R13
 U 1 1 58FB4DEF
 P 5450 3150
@@
 $EndComp
 $Comp
-L PF_apiner-rescue:GND-OBDII_IoT1 #PWR048
+L OBDII_IoT:GND #PWR048
 U 1 1 58FB4DF5
 P 5950 3450
@@
 $EndComp
 $Comp
-L PF_apiner-rescue:R-OBDII_IoT1 R11
+L OBDII_IoT:R R11
 U 1 1 58FB557C
 P 4250 4800
@@
 K-LINE
 $Comp
-L PF_apiner-rescue:DLC_SW-OBDII_IoT1 #PWR049
+L OBDII_IoT:DLC_SW #PWR049
 U 1 1 58FB56FF
 P 4700 4200
@@
 $EndComp
 $Comp
-L PF_apiner-rescue:C-OBDII_IoT1 C13
+L OBDII_IoT:C C13
 U 1 1 58FB6CF6
 P 4400 6100
@@
 $EndComp
 $Comp
-L PF_apiner-rescue:DLC_SW-OBDII_IoT1 #PWR050
+L OBDII_IoT:DLC_SW #PWR050
 U 1 1 58FB717D
 P 6050 4200
@@
 $EndComp
 $Comp
-L PF_apiner-rescue:C-OBDII_IoT1 C15
+L OBDII_IoT:C C15
 U 1 1 58FB71A2
 P 6050 4450
@@
 $EndComp
 $Comp
-L PF_apiner-rescue:GND-OBDII_IoT1 #PWR051
+L OBDII_IoT:GND #PWR051
 U 1 1 58FB7303
 P 4700 5050
@@
 $EndComp
 $Comp
-L PF_apiner-rescue:GND-OBDII_IoT1 #PWR052
+L OBDII_IoT:GND #PWR052
 U 1 1 58FB7392
 P 6050 4700
@@
 Ubicar cerca del LM339
 $Comp
-L PF_apiner-rescue:R-OBDII_IoT1 R9
+L OBDII_IoT:R R9
 U 1 1 58FB7561
 P 3650 4800
@@
 $EndComp
 $Comp
-L PF_apiner-rescue:DLC_SW-OBDII_IoT1 #PWR053
+L OBDII_IoT:DLC_SW #PWR053
 U 1 1 58FB7632
 P 3650 4200
@@
 $EndComp
 $Comp
-L PF_apiner-rescue:GND-OBDII_IoT1 #PWR054
+L OBDII_IoT:GND #PWR054
 U 1 1 58FB7688
 P 3650 5050
@@
 $EndComp
 $Comp
-L PF_apiner-rescue:GND-OBDII_IoT1 #PWR055
+L OBDII_IoT:GND #PWR055
 U 1 1 58FB9579
 P 4400 6450
@@
 ISO_RX
 $Comp
-L PF_apiner-rescue:+3.3V-OBDII_IoT1 #PWR056
+L OBDII_IoT:+3.3V #PWR056
 U 1 1 58FBB38D
 P 5200 4200
@@
 $EndComp
 $Comp
-L PF_apiner-rescue:R-OBDII_IoT1 R12
+L OBDII_IoT:R R12
 U 1 1 58FBB473
 P 5200 4400
@@
 $EndComp
 $Comp
-L PF_apiner-rescue:DLC-OBDII_IoT1 #PWR057
+L OBDII_IoT:DLC #PWR057
 U 1 1 58FB941A
 P 4400 5750
@@
 	3450 3150 3500 3150
 $Comp
-L PF_apiner-rescue:D_Schottky_BAT54SL-OBDII_IoT1 D5
+L OBDII_IoT:D_Schottky_BAT54SL D5
 U 1 1 59003DD4
 P 5250 6100
@@
 $EndComp
 $Comp
-L PF_apiner-rescue:C-OBDII_IoT1 C14
+L OBDII_IoT:C C14
 U 1 1 59003DDE
 P 5550 6100
@@
 $EndComp
 $Comp
-L PF_apiner-rescue:GND-OBDII_IoT1 #PWR058
+L OBDII_IoT:GND #PWR058
 U 1 1 59003DE4
 P 5550 6450
@@
 $EndComp
 $Comp
-L PF_apiner-rescue:DLC-OBDII_IoT1 #PWR059
+L OBDII_IoT:DLC #PWR059
 U 1 1 59003DEA
 P 5550 5750
