File: KiCad_Proyecto/J1850_Transceiver.sch (KiCad schematic (older format))
At the start: 30 parts, among them Q10 2N7002, Q7 2N7002, Q8 2N7002, Q9 BSS314PE, U3 LM339, U9 LM317

Commit message: todos los .sch arreglados
Parts:
- C24, C25, C26, C27: symbol PF_apiner-rescue:C-OBDII_IoT1 -> OBDII_IoT:C
- D10, D8, D9: symbol PF_apiner-rescue:D_Schot-OBDII_IoT1 -> OBDII_IoT:D_Schot
- D6, D7: symbol PF_apiner-rescue:D_Schottky_BAT54SL-OBDII_IoT1 -> OBDII_IoT:D_Schottky_BAT54SL
- Q10, Q7, Q8: symbol PF_apiner-rescue:MOS_N-OBDII_IoT1 -> OBDII_IoT:MOS_N
- Q9: symbol PF_apiner-rescue:MOS_P-OBDII_IoT1 -> OBDII_IoT:MOS_P
- R25, R26, R27, R28, R29, R30, R31, R32, R33, R34, R35, R36, R37, R38, R39: symbol PF_apiner-rescue:R-OBDII_IoT1 -> OBDII_IoT:R
- U3: symbol PF_apiner-rescue:LM339-OBDII_IoT1 -> OBDII_IoT:LM339
- U9: symbol PF_apiner-rescue:LM317LD-OBDII_IoT1 -> OBDII_IoT:LM317LD
Changed lines of the file:
@@
 EESchema Schematic File Version 4
 LIBS:PF_apiner-cache
-EELAYER 29 0
+EELAYER 26 0
 EELAYER END
 $Descr A4 11693 8268
@@
 J1850_BUS-_TX
 $Comp
-L PF_apiner-rescue:R-OBDII_IoT1 R25
+L OBDII_IoT:R R25
 U 1 1 582FD8FC
 P 3900 1850
@@
 $EndComp
 $Comp
-L PF_apiner-rescue:R-OBDII_IoT1 R26
+L OBDII_IoT:R R26
 U 1 1 582FDADA
 P 3900 2350
@@
 $EndComp
 $Comp
-L PF_apiner-rescue:R-OBDII_IoT1 R27
+L OBDII_IoT:R R27
 U 1 1 5832E14E
 P 3900 2750
@@
 $EndComp
 $Comp
-L PF_apiner-rescue:LM339-OBDII_IoT1 U3
+L OBDII_IoT:LM339 U3
 U 2 1 58FEE375
 P 5850 2100
@@
 $EndComp
 $Comp
-L PF_apiner-rescue:LM339-OBDII_IoT1 U3
+L OBDII_IoT:LM339 U3
 U 3 1 58FEE380
 P 8550 1950
@@
 $EndComp
 $Comp
-L PF_apiner-rescue:MOS_N-OBDII_IoT1 Q7
+L OBDII_IoT:MOS_N Q7
 U 1 1 58FF3421
 P 3550 2750
@@
 J1850_BUS+_VH
 $Comp
-L PF_apiner-rescue:C-OBDII_IoT1 C25
+L OBDII_IoT:C C25
 U 1 1 58FF9848
 P 2950 1950
@@
 	2950 1600 2950 1800
 $Comp
-L PF_apiner-rescue:DLC_SW-OBDII_IoT1 #PWR078
+L OBDII_IoT:DLC_SW #PWR078
 U 1 1 58FFBF93
 P 2950 1600
@@
 Connection ~ 2950 1650
 $Comp
-L PF_apiner-rescue:V_J1850-OBDII_IoT1 #PWR079
+L OBDII_IoT:V_J1850 #PWR079
 U 1 1 58FFC6C3
 P 3900 1600
@@
 Connection ~ 3900 1650
 $Comp
-L PF_apiner-rescue:GND-OBDII_IoT1 #PWR080
+L OBDII_IoT:GND #PWR080
 U 1 1 58FFC795
 P 2950 2200
@@
 Connection ~ 3900 2550
 $Comp
-L PF_apiner-rescue:GND-OBDII_IoT1 #PWR081
+L OBDII_IoT:GND #PWR081
 U 1 1 58FFC8CF
 P 3900 3000
@@
 	3300 2750 3350 2750
 $Comp
-L PF_apiner-rescue:R-OBDII_IoT1 R30
+L OBDII_IoT:R R30
 U 1 1 58FFF46B
 P 5300 2000
@@
 $EndComp
 $Comp
-L PF_apiner-rescue:D_Schottky_BAT54SL-OBDII_IoT1 D6
+L OBDII_IoT:D_Schottky_BAT54SL D6
 U 1 1 58FFFF10
 P 1950 4350
@@
 $EndComp
 $Comp
-L PF_apiner-rescue:C-OBDII_IoT1 C24
+L OBDII_IoT:C C24
 U 1 1 58FFFF1B
 P 2250 4350
@@
 J1850_BUS-
 $Comp
-L PF_apiner-rescue:DLC-OBDII_IoT1 #PWR082
+L OBDII_IoT:DLC #PWR082
 U 1 1 59002768
 P 2250 4000
@@
 $EndComp
 $Comp
-L PF_apiner-rescue:GND-OBDII_IoT1 #PWR083
+L OBDII_IoT:GND #PWR083
 U 1 1 5900289A
 P 2250 4700
@@
 Connection ~ 2250 4050
 $Comp
-L PF_apiner-rescue:D_Schottky_BAT54SL-OBDII_IoT1 D7
+L OBDII_IoT:D_Schottky_BAT54SL D7
 U 1 1 59002A9E
 P 3100 4350
@@
 $EndComp
 $Comp
-L PF_apiner-rescue:C-OBDII_IoT1 C26
+L OBDII_IoT:C C26
 U 1 1 59002AA8
 P 3400 4350
@@
 $EndComp
 $Comp
-L PF_apiner-rescue:DLC-OBDII_IoT1 #PWR084
+L OBDII_IoT:DLC #PWR084
 U 1 1 59002AAE
 P 3400 4000
@@
 $EndComp
 $Comp
-L PF_apiner-rescue:GND-OBDII_IoT1 #PWR085
+L OBDII_IoT:GND #PWR085
 U 1 1 59002AB4
 P 3400 4700
@@
 	1600 2950 1750 2950
 $Comp
-L PF_apiner-rescue:R-OBDII_IoT1 R31
+L OBDII_IoT:R R31
 U 1 1 5900554A
 P 5300 2200
@@
 $EndComp
 $Comp
-L PF_apiner-rescue:DLC_SW-OBDII_IoT1 #PWR086
+L OBDII_IoT:DLC_SW #PWR086
 U 1 1 5900675A
 P 5750 1700
@@
 $EndComp
 $Comp
-L PF_apiner-rescue:GND-OBDII_IoT1 #PWR087
+L OBDII_IoT:GND #PWR087
 U 1 1 5900679C
 P 5750 2450
@@
 	5750 2400 5750 2450
 $Comp
-L PF_apiner-rescue:+3.3V-OBDII_IoT1 #PWR088
+L OBDII_IoT:+3.3V #PWR088
 U 1 1 59006FD8
 P 6250 1700
@@
 $EndComp
 $Comp
-L PF_apiner-rescue:R-OBDII_IoT1 R33
+L OBDII_IoT:R R33
 U 1 1 59006FE2
 P 6250 1900
@@
 Connection ~ 6250 2100
 $Comp
-L PF_apiner-rescue:MOS_N-OBDII_IoT1 Q8
+L OBDII_IoT:MOS_N Q8
 U 1 1 59007FAD
 P 5150 4100
@@
 $EndComp
 $Comp
-L PF_apiner-rescue:MOS_P-OBDII_IoT1 Q9
+L OBDII_IoT:MOS_P Q9
 U 1 1 5900CF77
 P 5500 3550
@@
 $EndComp
 $Comp
-L PF_apiner-rescue:R-OBDII_IoT1 R28
+L OBDII_IoT:R R28
 U 1 1 5900D39E
 P 4900 4300
@@
 $EndComp
 $Comp
-L PF_apiner-rescue:GND-OBDII_IoT1 #PWR089
+L OBDII_IoT:GND #PWR089
 U 1 1 5900D50B
 P 5250 4500
@@
 $EndComp
 $Comp
-L PF_apiner-rescue:R-OBDII_IoT1 R29
+L OBDII_IoT:R R29
 U 1 1 5900D718
 P 5250 3650
@@
 $EndComp
 $Comp
-L PF_apiner-rescue:D_Schot-OBDII_IoT1 D8
+L OBDII_IoT:D_Schot D8
 U 1 1 5900E8B5
 P 5950 3450
@@
 J1850_BUS+
 $Comp
-L PF_apiner-rescue:D_Schot-OBDII_IoT1 D9
+L OBDII_IoT:D_Schot D9
 U 1 1 5900EFC2
 P 6150 4250
@@
 $EndComp
 $Comp
-L PF_apiner-rescue:R-OBDII_IoT1 R32
+L OBDII_IoT:R R32
 U 1 1 5900F3D6
 P 6150 3850
@@
 $EndComp
 $Comp
-L PF_apiner-rescue:GND-OBDII_IoT1 #PWR090
+L OBDII_IoT:GND #PWR090
 U 1 1 5900F564
 P 6150 4500
@@
 	5250 3400 5250 3500
 $Comp
-L PF_apiner-rescue:V_J1850-OBDII_IoT1 #PWR091
+L OBDII_IoT:V_J1850 #PWR091
 U 1 1 5900FFB7
 P 5250 3400
@@
 	6150 4500 6150 4350
 $Comp
-L PF_apiner-rescue:+3.3V-OBDII_IoT1 #PWR092
+L OBDII_IoT:+3.3V #PWR092
 U 1 1 59011723
 P 8950 1550
@@
 $EndComp
 $Comp
-L PF_apiner-rescue:R-OBDII_IoT1 R39
+L OBDII_IoT:R R39
 U 1 1 5901172D
 P 8950 1750
@@
 	8950 1600 8950 1550
 $Comp
-L PF_apiner-rescue:DLC_SW-OBDII_IoT1 #PWR093
+L OBDII_IoT:DLC_SW #PWR093
 U 1 1 5901176C
 P 8450 1550
@@
 	8450 1550 8450 1650
 $Comp
-L PF_apiner-rescue:R-OBDII_IoT1 R35
+L OBDII_IoT:R R35
 U 1 1 59011805
 P 7350 2250
@@
 $EndComp
 $Comp
-L PF_apiner-rescue:R-OBDII_IoT1 R34
+L OBDII_IoT:R R34
 U 1 1 590118B7
 P 7350 1850
@@
 $EndComp
 $Comp
-L PF_apiner-rescue:R-OBDII_IoT1 R37
+L OBDII_IoT:R R37
 U 1 1 590119B2
 P 8050 1850
@@
 Connection ~ 7350 2050
 $Comp
-L PF_apiner-rescue:+5V_SW-OBDII_IoT1 #PWR094
+L OBDII_IoT:+5V_SW #PWR094
 U 1 1 590137AA
 P 7350 1550
@@
 	7350 1550 7350 1700
 $Comp
-L PF_apiner-rescue:GND-OBDII_IoT1 #PWR095
+L OBDII_IoT:GND #PWR095
 U 1 1 5901397C
 P 7350 2450
@@
 	7350 2450 7350 2400
 $Comp
-L PF_apiner-rescue:GND-OBDII_IoT1 #PWR096
+L OBDII_IoT:GND #PWR096
 U 1 1 59013A21
 P 8450 2450
@@
 Connection ~ 8950 1950
 $Comp
-L PF_apiner-rescue:+5V_SW-OBDII_IoT1 #PWR097
+L OBDII_IoT:+5V_SW #PWR097
 U 1 1 590144CF
 P 8200 3400
@@
 $EndComp
 $Comp
-L PF_apiner-rescue:D_Schot-OBDII_IoT1 D10
+L OBDII_IoT:D_Schot D10
 U 1 1 590146A5
 P 8200 3550
@@
 $EndComp
 $Comp
-L PF_apiner-rescue:R-OBDII_IoT1 R38
+L OBDII_IoT:R R38
 U 1 1 590146AF
 P 8200 3850
@@
 $EndComp
 $Comp
-L PF_apiner-rescue:MOS_N-OBDII_IoT1 Q10
+L OBDII_IoT:MOS_N Q10
 U 1 1 590147AD
 P 8100 4300
@@
 $EndComp
 $Comp
-L PF_apiner-rescue:R-OBDII_IoT1 R36
+L OBDII_IoT:R R36
 U 1 1 59015277
 P 7850 3850
@@
 	7800 4300 7900 4300
 $Comp
-L PF_apiner-rescue:GND-OBDII_IoT1 #PWR098
+L OBDII_IoT:GND #PWR098
 U 1 1 590155AC
 P 8200 4550
@@
 $EndComp
 $Comp
-L PF_apiner-rescue:+5V_SW-OBDII_IoT1 #PWR099
+L OBDII_IoT:+5V_SW #PWR099
 U 1 1 59015925
 P 7850 3400
@@
 	8200 4550 8200 4500
 $Comp
-L PF_apiner-rescue:LM317LD-OBDII_IoT1 U9
+L OBDII_IoT:LM317LD U9
 U 1 1 58F8CA15
 P 3400 1650
@@
 $EndComp
 $Comp
-L PF_apiner-rescue:C-OBDII_IoT1 C27
+L OBDII_IoT:C C27
 U 1 1 58FD532B
 P 4150 1850
@@
 $EndComp
 $Comp
-L PF_apiner-rescue:GND-OBDII_IoT1 #PWR0100
+L OBDII_IoT:GND #PWR0100
 U 1 1 58FD55BE
 P 4150 2150
