File: KiCad_Proyecto/Power_CRTL.sch (KiCad schematic (older format))
At the start: 5 parts, among them Q1 2N7002, Q2 BSS314PE, Q3 BSS314PE

Commit message: todos los .sch arreglados
Parts:
- Q1: symbol PF_apiner-rescue:MOS_N-OBDII_IoT1 -> OBDII_IoT:MOS_N
- Q2, Q3: symbol PF_apiner-rescue:MOS_P-OBDII_IoT1 -> OBDII_IoT:MOS_P
- R3, R4: symbol PF_apiner-rescue:R-OBDII_IoT1 -> OBDII_IoT:R
Changed lines of the file:
@@
 EESchema Schematic File Version 4
 LIBS:PF_apiner-cache
-EELAYER 29 0
+EELAYER 26 0
 EELAYER END
 $Descr A4 11693 8268
@@
 PWR_SAVE
 $Comp
-L PF_apiner-rescue:DLC-OBDII_IoT1 #PWR029
+L OBDII_IoT:DLC #PWR029
 U 1 1 5833D47C
 P 5350 4600
@@
 $EndComp
 $Comp
-L PF_apiner-rescue:DLC_SW-OBDII_IoT1 #PWR030
+L OBDII_IoT:DLC_SW #PWR030
 U 1 1 5833D496
 P 5950 4600
@@
 $EndComp
 $Comp
-L PF_apiner-rescue:+5V_SW-OBDII_IoT1 #PWR031
+L OBDII_IoT:+5V_SW #PWR031
 U 1 1 5833D581
 P 6900 4600
@@
 	5000 4300 5000 4450
 $Comp
-L PF_apiner-rescue:DLC-OBDII_IoT1 #PWR032
+L OBDII_IoT:DLC #PWR032
 U 1 1 5833D8D2
 P 5000 3900
@@
 	5000 3900 5000 4000
 $Comp
-L PF_apiner-rescue:GND-OBDII_IoT1 #PWR033
+L OBDII_IoT:GND #PWR033
 U 1 1 5833D90C
 P 5000 4950
@@
 Connection ~ 5650 4400
 $Comp
-L PF_apiner-rescue:PWR_FLAG-OBDII_IoT1 #FLG034
+L OBDII_IoT:PWR_FLAG #FLG034
 U 1 1 584984F2
 P 5350 5000
@@
 $EndComp
 $Comp
-L PF_apiner-rescue:PWR_FLAG-OBDII_IoT1 #FLG035
+L OBDII_IoT:PWR_FLAG #FLG035
 U 1 1 58498516
 P 5950 5000
@@
 $EndComp
 $Comp
-L PF_apiner-rescue:PWR_FLAG-OBDII_IoT1 #FLG036
+L OBDII_IoT:PWR_FLAG #FLG036
 U 1 1 5849858A
 P 6900 5000
@@
 Connection ~ 6900 4850
 $Comp
-L PF_apiner-rescue:R-OBDII_IoT1 R3
+L OBDII_IoT:R R3
 U 1 1 58FA0F0C
 P 4600 4150
@@
 $EndComp
 $Comp
-L PF_apiner-rescue:+3.3V-OBDII_IoT1 #PWR037
+L OBDII_IoT:+3.3V #PWR037
 U 1 1 58FA0FB6
 P 4600 3900
@@
 	4600 3900 4600 4000
 $Comp
-L PF_apiner-rescue:R-OBDII_IoT1 R4
+L OBDII_IoT:R R4
 U 1 1 58FA1022
 P 5000 4150
@@
 $EndComp
 $Comp
-L PF_apiner-rescue:MOS_P-OBDII_IoT1 Q2
+L OBDII_IoT:MOS_P Q2
 U 1 1 58FA2395
 P 5650 4750
@@
 $EndComp
 $Comp
-L PF_apiner-rescue:MOS_N-OBDII_IoT1 Q1
+L OBDII_IoT:MOS_N Q1
 U 1 1 58FA23A0
 P 4900 4650
@@
 $EndComp
 $Comp
-L PF_apiner-rescue:+5V-OBDII_IoT1 #PWR038
+L OBDII_IoT:+5V #PWR038
 U 1 1 58FA6825
 P 6300 4600
@@
 	6300 4600 6300 5000
 $Comp
-L PF_apiner-rescue:PWR_FLAG-OBDII_IoT1 #FLG039
+L OBDII_IoT:PWR_FLAG #FLG039
 U 1 1 58FA7137
 P 6300 5000
@@
 	6600 4400 5000 4400
 $Comp
-L PF_apiner-rescue:MOS_P-OBDII_IoT1 Q3
+L OBDII_IoT:MOS_P Q3
 U 1 1 59009220
 P 6600 4750
