File: KiCad_Proyecto/Power_Supplies.sch (KiCad schematic (older format))
At the start: 19 parts, among them U1 TPS54202, U2 AZ1117EH-3.3TRG1

Commit message: todos los .sch arreglados
Parts:
- C1, C10, C11, C2, C3, C4, C5, C6, C7, C8, C9: symbol PF_apiner-rescue:C-OBDII_IoT1 -> OBDII_IoT:C
- D1: symbol PF_apiner-rescue:TVS-OBDII_IoT1 -> OBDII_IoT:TVS
- D2: symbol PF_apiner-rescue:D-OBDII_IoT1 -> OBDII_IoT:D
- F1: symbol PF_apiner-rescue:FUSE-OBDII_IoT1 -> OBDII_IoT:FUSE
- L1: symbol PF_apiner-rescue:L-OBDII_IoT1 -> OBDII_IoT:L
- R1, R2: symbol PF_apiner-rescue:R-OBDII_IoT1 -> OBDII_IoT:R
- U1: symbol PF_apiner-rescue:TPS54202-OBDII_IoT1 -> OBDII_IoT:TPS54202
- U2: symbol PF_apiner-rescue:VOLT_REG-OBDII_IoT1 -> OBDII_IoT:VOLT_REG
Changed lines of the file:
@@
 EESchema Schematic File Version 4
 LIBS:PF_apiner-cache
-EELAYER 29 0
+EELAYER 26 0
 EELAYER END
 $Descr A4 11693 8268
@@
 $EndDescr
 $Comp
-L PF_apiner-rescue:DLC_RAW-OBDII_IoT1 #PWR09
+L OBDII_IoT:DLC_RAW #PWR09
 U 1 1 5835BB34
 P 4950 2400
@@
 $EndComp
 $Comp
-L PF_apiner-rescue:C-OBDII_IoT1 C1
+L OBDII_IoT:C C1
 U 1 1 5835BB57
 P 4300 2700
@@
 $EndComp
 $Comp
-L PF_apiner-rescue:DLC-OBDII_IoT1 #PWR010
+L OBDII_IoT:DLC #PWR010
 U 1 1 5835BBB8
 P 5900 2400
@@
 $EndComp
 $Comp
-L PF_apiner-rescue:C-OBDII_IoT1 C4
+L OBDII_IoT:C C4
 U 1 1 5835BBD5
 P 5300 2700
@@
 $EndComp
 $Comp
-L PF_apiner-rescue:GND-OBDII_IoT1 #PWR011
+L OBDII_IoT:GND #PWR011
 U 1 1 5835BE13
 P 4300 2950
@@
 $EndComp
 $Comp
-L PF_apiner-rescue:TVS-OBDII_IoT1 D1
+L OBDII_IoT:TVS D1
 U 1 1 5835C003
 P 4950 2750
@@
 $EndComp
 $Comp
-L PF_apiner-rescue:D-OBDII_IoT1 D2
+L OBDII_IoT:D D2
 U 1 1 5835C0B1
 P 5150 2500
@@
 $EndComp
 $Comp
-L PF_apiner-rescue:FUSE-OBDII_IoT1 F1
+L OBDII_IoT:FUSE F1
 U 1 1 5835F7DA
 P 4600 2500
@@
 $EndComp
 $Comp
-L PF_apiner-rescue:TPS54202-OBDII_IoT1 U1
+L OBDII_IoT:TPS54202 U1
 U 1 1 5835C29D
 P 4500 3800
@@
 $EndComp
 $Comp
-L PF_apiner-rescue:DLC-OBDII_IoT1 #PWR012
+L OBDII_IoT:DLC #PWR012
 U 1 1 5835C416
 P 3950 3550
@@
 $EndComp
 $Comp
-L PF_apiner-rescue:L-OBDII_IoT1 L1
+L OBDII_IoT:L L1
 U 1 1 5835C9FC
 P 5500 3650
@@
 $EndComp
 $Comp
-L PF_apiner-rescue:C-OBDII_IoT1 C8
+L OBDII_IoT:C C8
 U 1 1 5835CACB
 P 5700 3850
@@
 $EndComp
 $Comp
-L PF_apiner-rescue:+5V-OBDII_IoT1 #PWR013
+L OBDII_IoT:+5V #PWR013
 U 1 1 5836344D
 P 6000 3500
@@
 	4050 2500 4350 2500
 $Comp
-L PF_apiner-rescue:C-OBDII_IoT1 C3
+L OBDII_IoT:C C3
 U 1 1 588025EB
 P 5150 3650
@@
 $EndComp
 $Comp
-L PF_apiner-rescue:C-OBDII_IoT1 C10
+L OBDII_IoT:C C10
 U 1 1 589356C6
 P 6200 4050
@@
 Connection ~ 6200 4500
 $Comp
-L PF_apiner-rescue:R-OBDII_IoT1 R1
+L OBDII_IoT:R R1
 U 1 1 58A271C0
 P 6000 3850
@@
 $EndComp
 $Comp
-L PF_apiner-rescue:GND-OBDII_IoT1 #PWR014
+L OBDII_IoT:GND #PWR014
 U 1 1 58F7E73C
 P 4950 2950
@@
 $EndComp
 $Comp
-L PF_apiner-rescue:GND-OBDII_IoT1 #PWR015
+L OBDII_IoT:GND #PWR015
 U 1 1 58F7E773
 P 5900 2950
@@
 	5900 2950 5900 2850
 $Comp
-L PF_apiner-rescue:GND-OBDII_IoT1 #PWR016
+L OBDII_IoT:GND #PWR016
 U 1 1 58F7F16E
 P 5700 2950
@@
 $EndComp
 $Comp
-L PF_apiner-rescue:GND-OBDII_IoT1 #PWR017
+L OBDII_IoT:GND #PWR017
 U 1 1 58F7F1A5
 P 5500 2950
@@
 $EndComp
 $Comp
-L PF_apiner-rescue:GND-OBDII_IoT1 #PWR018
+L OBDII_IoT:GND #PWR018
 U 1 1 58F7F1DC
 P 5300 2950
@@
 	5700 2950 5700 2850
 $Comp
-L PF_apiner-rescue:C-OBDII_IoT1 C6
+L OBDII_IoT:C C6
 U 1 1 58F7FBBA
 P 5500 2700
@@
 $EndComp
 $Comp
-L PF_apiner-rescue:C-OBDII_IoT1 C7
+L OBDII_IoT:C C7
 U 1 1 58F7FBFE
 P 5700 2700
@@
 $EndComp
 $Comp
-L PF_apiner-rescue:C-OBDII_IoT1 C9
+L OBDII_IoT:C C9
 U 1 1 58F7FC44
 P 5900 2700
@@
 $EndComp
 $Comp
-L PF_apiner-rescue:C-OBDII_IoT1 C2
+L OBDII_IoT:C C2
 U 1 1 58F80648
 P 4450 5200
@@
 $EndComp
 $Comp
-L PF_apiner-rescue:C-OBDII_IoT1 C11
+L OBDII_IoT:C C11
 U 1 1 58F81C6B
 P 6450 4050
@@
 $EndComp
 $Comp
-L PF_apiner-rescue:GND-OBDII_IoT1 #PWR019
+L OBDII_IoT:GND #PWR019
 U 1 1 58F81EC8
 P 3950 4100
@@
 $EndComp
 $Comp
-L PF_apiner-rescue:GND-OBDII_IoT1 #PWR020
+L OBDII_IoT:GND #PWR020
 U 1 1 58F81EFF
 P 6000 4550
@@
 $EndComp
 $Comp
-L PF_apiner-rescue:VOLT_REG-OBDII_IoT1 U2
+L OBDII_IoT:VOLT_REG U2
 U 1 1 58F82CD2
 P 4900 4950
@@
 $EndComp
 $Comp
-L PF_apiner-rescue:+5V-OBDII_IoT1 #PWR021
+L OBDII_IoT:+5V #PWR021
 U 1 1 58F82E5C
 P 4450 4900
@@
 $EndComp
 $Comp
-L PF_apiner-rescue:C-OBDII_IoT1 C5
+L OBDII_IoT:C C5
 U 1 1 58F85AE2
 P 5400 5200
@@
 $EndComp
 $Comp
-L PF_apiner-rescue:+3.3V-OBDII_IoT1 #PWR022
+L OBDII_IoT:+3.3V #PWR022
 U 1 1 58F85D19
 P 5400 4900
@@
 $EndComp
 $Comp
-L PF_apiner-rescue:GND-OBDII_IoT1 #PWR023
+L OBDII_IoT:GND #PWR023
 U 1 1 58F85EE0
 P 4900 5450
@@
 $EndComp
 $Comp
-L PF_apiner-rescue:GND-OBDII_IoT1 #PWR024
+L OBDII_IoT:GND #PWR024
 U 1 1 58F85FA0
 P 4450 5450
@@
 $EndComp
 $Comp
-L PF_apiner-rescue:GND-OBDII_IoT1 #PWR025
+L OBDII_IoT:GND #PWR025
 U 1 1 58F85FD1
 P 5400 5450
@@
 Connection ~ 5400 4950
 $Comp
-L PF_apiner-rescue:R-OBDII_IoT1 R2
+L OBDII_IoT:R R2
 U 1 1 58F89868
 P 6000 4300
@@
 	4300 2400 4300 2550
 $Comp
-L PF_apiner-rescue:VIN-OBDII_IoT1 #PWR026
+L OBDII_IoT:VIN #PWR026
 U 1 1 58F9A73A
 P 4300 2400
@@
 	3950 3650 4050 3650
 $Comp
-L PF_apiner-rescue:PWR_FLAG-OBDII_IoT1 #FLG027
+L OBDII_IoT:PWR_FLAG #FLG027
 U 1 1 590B622B
 P 4050 2500
@@
 $EndComp
 $Comp
-L PF_apiner-rescue:PWR_FLAG-OBDII_IoT1 #FLG028
+L OBDII_IoT:PWR_FLAG #FLG028
 U 1 1 590B82D6
 P 4050 2850
