File: KiCad_Proyecto/Voltage_Sense.sch (KiCad schematic (older format))
At the start: 4 parts

Commit message: todos los .sch arreglados
Parts:
- C12: symbol PF_apiner-rescue:C-OBDII_IoT1 -> OBDII_IoT:C
- D3: symbol PF_apiner-rescue:D_Schottky_BAT54SL-OBDII_IoT1 -> OBDII_IoT:D_Schottky_BAT54SL
- R5, R6: symbol PF_apiner-rescue:R-OBDII_IoT1 -> OBDII_IoT:R
Changed lines of the file:
@@
 EESchema Schematic File Version 4
 LIBS:PF_apiner-cache
-EELAYER 29 0
+EELAYER 26 0
 EELAYER END
 $Descr A4 11693 8268
@@
 $EndDescr
 $Comp
-L PF_apiner-rescue:DLC_RAW-OBDII_IoT1 #PWR040
+L OBDII_IoT:DLC_RAW #PWR040
 U 1 1 582F295A
 P 5150 3350
@@
 $EndComp
 $Comp
-L PF_apiner-rescue:R-OBDII_IoT1 R5
+L OBDII_IoT:R R5
 U 1 1 582F3539
 P 5150 3650
@@
 $EndComp
 $Comp
-L PF_apiner-rescue:GND-OBDII_IoT1 #PWR041
+L OBDII_IoT:GND #PWR041
 U 1 1 582F35F0
 P 5150 4450
@@
 $EndComp
 $Comp
-L PF_apiner-rescue:GND-OBDII_IoT1 #PWR042
+L OBDII_IoT:GND #PWR042
 U 1 1 582F3A7C
 P 5650 4450
@@
 	5650 4200 5650 4450
 $Comp
-L PF_apiner-rescue:D_Schottky_BAT54SL-OBDII_IoT1 D3
+L OBDII_IoT:D_Schottky_BAT54SL D3
 U 1 1 583A9D5F
 P 5650 3900
@@
 Connection ~ 5350 3900
 $Comp
-L PF_apiner-rescue:R-OBDII_IoT1 R6
+L OBDII_IoT:R R6
 U 1 1 583AB1A6
 P 5150 4150
@@
 $EndComp
 $Comp
-L PF_apiner-rescue:PWR_FLAG-OBDII_IoT1 #FLG043
+L OBDII_IoT:PWR_FLAG #FLG043
 U 1 1 58498D94
 P 4900 3350
@@
 Connection ~ 5150 3400
 $Comp
-L PF_apiner-rescue:C-OBDII_IoT1 C12
+L OBDII_IoT:C C12
 U 1 1 58F8BB88
 P 4850 4150
@@
 $EndComp
 $Comp
-L PF_apiner-rescue:+3.3V-OBDII_IoT1 #PWR044
+L OBDII_IoT:+3.3V #PWR044
 U 1 1 58F8C1FD
 P 5650 3350
