File: KiCad_Proyecto/PF_apiner.kicad_pcb (KiCad board)
At the start: 4 copper layers, 50 x 40.5 mm, 133 parts, among them J1 OBDII Header, J2 Conn_01x05, Q1 2N7002, Q10 2N7002, Q2 BSS314PE, Q3 BSS314PE, Q4 MMBT3904, Q5 MMBT3904, Q6 2N7002, Q7 2N7002, Q8 2N7002, Q9 BSS314PE, SW1 SW_RESET, SW2 SW_BOOT, U1 TPS54202, U10 STN2120, U14 ESP32-WROOM, U2 AZ1117EH-3.3TRG1, U3 LM339, U4 MCP25612FD, U5 TH8056, U6 PESD1CAN, U7 PESD1CAN, U8 PESD1CAN, U9 LM317, Y1 16M

Commit message: se viene
Parts:
- added R54: 10K, chip_rlc:r_0402, B.Cu at (84.8, 64.5)
- C10, C38: moved to B.Cu
- C19, C21, Q6, R17, R18, R20, R34, R35, R39, R49, R50, R51: moved to F.Cu
- moved R30 47.1 mm to (111.5, 48.8), turned to 180 degrees
- moved R12 45.8 mm to (107.8, 49.8), turned to 0 degrees
- moved C15 45.6 mm to (108.0, 48.2), turned to 0 degrees
- moved R33 44.2 mm to (107.8, 51.0), turned to 0 degrees
- moved D10 39.0 mm to (104.9, 44.2), turned to 0 degrees
- moved R37 38.3 mm to (111.5, 50.0), turned to 180 degrees
- moved R9 35.2 mm to (99.8, 52.8)
- moved R8 35.1 mm to (99.8, 54.0)
- moved R11 35.1 mm to (99.8, 55.2)
- moved R31 32.9 mm to (107.8, 47.0), turned to 180 degrees
- moved R15 31.9 mm to (110.2, 54.0), turned to 180 degrees
- moved R28 31.5 mm to (102.0, 66.0), turned to 90 degrees
- moved R38 31.2 mm to (108.0, 44.2), turned to 180 degrees
- moved C27 31.0 mm to (93.5, 76.2), turned to 180 degrees
- moved R4 30.6 mm to (95.5, 45.0), turned to 0 degrees
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Connections:
- net /CAN_Transceiver/HS_CAN_HI renamed /HS_CAN_P
- net /CAN_Transceiver/HS_CAN_LO renamed /HS_CAN_N
- net /CAN_Transceiver/MS_CAN_HI renamed /MS_CAN_P
- net /CAN_Transceiver/MS_CAN_LO renamed /MS_CAN_N
- net /CAN_Transceiver/SW_CAN renamed /SW_CAN
- net /ISO_Transceiver/K-LINE renamed /K-LINE
- net /ISO_Transceiver/L-LINE renamed /L-LINE
- net /J1850_Transceiver/J1850_BUS+ renamed /J1850_BUS+
- net /J1850_Transceiver/J1850_BUS- renamed /J1850_BUS-
- net Net-(SW2-Pad1) renamed /MicroM4/BOOT
- J2 pad 2: /MicroM4/UART0_TX -> /MicroM4/UART0_RX
- J2 pad 3: /MicroM4/UART0_RX -> /MicroM4/UART0_TX
Routing:
- net /HS_CAN_P: track 0.00 -> 52.1 mm, vias 0 -> 1
- net /HS_CAN_N: track 0.00 -> 50.5 mm, vias 0 -> 1
- net /MS_CAN_N: track 0.00 -> 39.5 mm, vias 0 -> 1
- net /MS_CAN_P: track 0.00 -> 38.8 mm, vias 0 -> 1
- net /K-LINE: track 0.00 -> 27.7 mm
- net /J1850_Transceiver/VPW_RX: track 0.00 -> 26.7 mm, vias 0 -> 2
- net /CAN_Transceiver/SW_CAN_LOAD: track 0.00 -> 25.3 mm, vias 0 -> 3
- net /ISO_Transceiver/ISO_RX: track 0.00 -> 24.5 mm, vias 0 -> 2
- net /MicroM4/RESET: track 0.00 -> 23.9 mm
- net /SW_CAN: track 0.00 -> 22.6 mm, vias 0 -> 1
- net /CAN_Transceiver/SW_CAN_MODE1: track 0.00 -> 21.7 mm, vias 0 -> 3
- net /CAN_Transceiver/SW_CAN_MODE0: track 0.00 -> 21.0 mm, vias 0 -> 3
- net /ISO_Transceiver/ISO_K_TX: track 0.00 -> 20.8 mm, vias 0 -> 2
- net /J1850_BUS+: track 0.00 -> 20.1 mm
- net /ISO_Transceiver/ISO_L_TX: track 0.00 -> 20.0 mm, vias 0 -> 2
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- added copper zone on F.Cu, net +3.3V
- added copper zone on F.Cu, net +5V
- added copper zone on F.Cu, net DLC
- added copper zone on F.Cu, net DLC_RAW
- added copper zone on F.Cu, net VIN

Commit message: es viernes
Parts:
- R52: moved to B.Cu
- moved C7 9.26 mm to (83.0, 48.0), turned to 180 degrees
- moved D1 8.25 mm to (91.8, 49.2), turned to 180 degrees
- moved R52 5.51 mm to (126.2, 62.8), turned to 0 degrees
- moved R26 1.50 mm to (90.0, 69.5)
- moved C4 0.75 mm to (83.0, 50.8)
- moved C6 0.75 mm to (83.0, 50.8)
- moved C9 0.75 mm to (83.0, 48.0)
- moved R15 0.50 mm to (110.8, 54.0)
- moved R42 0.50 mm to (110.8, 55.0)
Routing:
- net DLC_RAW: track 0.00 -> 48.5 mm, vias 0 -> 3
- net GND: track 19.9 -> 39.5 mm, vias 0 -> 4
- net Net-(Q1-Pad3): track 0.00 -> 16.1 mm
- net +3.3V: track 6.57 -> 20.5 mm
- net /MicroM4/RESET: track 23.9 -> 37.7 mm
- net DLC: track 0.65 -> 12.5 mm, vias 0 -> 4
- net Net-(R37-Pad2): track 0.00 -> 11.9 mm, vias 0 -> 2
- net Net-(R30-Pad2): track 0.00 -> 11.4 mm, vias 0 -> 2
- net DLC_SW: track 5.35 -> 16.3 mm, vias 0 -> 4
- net +5V: track 4.97 -> 15.6 mm, vias 0 -> 1
- net Net-(C3-Pad1): track 5.35 -> 12.9 mm, vias 0 -> 2
- net /CAN_Transceiver/SW_CAN_TX: track 13.2 -> 19.6 mm
- net V_J1850: track 11.4 -> 15.5 mm
- net /MicroM4/UART1_RX: track 13.5 -> 10.9 mm
- net /CAN_Transceiver/SW_CAN_RX: track 17.4 -> 14.8 mm
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
Commit message: ruteado terminado listo para rev
Parts:
- C16, C17, C38, R52: moved to F.Cu
- moved R52 8.85 mm to (120.2, 69.2), turned to 270 degrees
- moved R25 7.30 mm to (96.5, 71.8)
- moved C2 6.82 mm to (90.8, 62.8)
- moved C17 5.49 mm to (121.0, 63.5)
- moved C16 5.37 mm to (122.0, 63.5)
- moved C37 4.61 mm to (121.0, 73.5)
- moved C36 4.56 mm to (119.3, 73.7)
- moved C10 3.95 mm to (92.0, 61.0), turned to 0 degrees
- moved C27 3.61 mm to (96.5, 74.2), turned to 270 degrees
- moved U9 3.07 mm to (94.1, 73.5), turned to 270 degrees
- moved R54 2.76 mm to (82.0, 64.8), turned to 270 degrees
- moved R26 2.37 mm to (92.2, 70.2), turned to 0 degrees
- moved R7 2.26 mm to (91.5, 52.8), turned to 90 degrees
- moved R48 1.65 mm to (115.1, 64.7)
- moved C25 1.50 mm to (88.5, 75.0)
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Connections:
- U14 pad 28: Net-(U14-Pad28) -> /MicroM4/PWR_SAVE
- U14 pad 33: Net-(U14-Pad33) -> /MicroM4/STN_SLEEP
- U14 pad 8: /MicroM4/PWR_SAVE -> Net-(U14-Pad8)
- U14 pad 9: /MicroM4/STN_SLEEP -> Net-(U14-Pad9)
Routing:
- net GND: track 39.5 -> 178.7 mm, vias 4 -> 67
- net +3.3V: track 20.5 -> 147.5 mm, vias 0 -> 13
- net +5V_SW: track 1.25 -> 93.0 mm, vias 0 -> 7
- net +5V: track 15.6 -> 90.4 mm, vias 1 -> 10
- net DLC: track 12.5 -> 84.7 mm, vias 4 -> 9
- net DLC_SW: track 16.3 -> 67.6 mm
- net /MicroM4/BOOT: track 0.00 -> 34.2 mm, vias 0 -> 2
- net /J1850_BUS+: track 20.1 -> 45.5 mm, vias 0 -> 2
- net /SW_CAN: track 22.6 -> 35.9 mm, vias 1 -> 2
- net /MicroM4/PWR_SAVE: track 13.4 -> 19.5 mm, vias 1 -> 2
- net /MicroM4/STN_SLEEP: track 0.00 -> 5.53 mm, vias 0 -> 1
- net V_J1850: track 15.5 -> 11.2 mm
- net Net-(R25-Pad1): track 8.44 -> 4.29 mm
- net /MicroM4/RESET: track 37.7 -> 40.6 mm
- net /MicroM4/UART1_RX: track 10.9 -> 13.2 mm
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- added copper zone on PWR, net +3.3V
- added copper zone on F.Cu, net GND
- added copper zone on GND, net GND

Commit message: lalala
Routing:
- net VIN: track 2.50 -> 6.39 mm
- net DLC_RAW: track 49.2 -> 47.8 mm
- removed copper zone on F.Cu, net VIN

Commit message: .net y pcb final
Parts:
- added C34: 0.1uF, chip_rlc:c_0402, F.Cu at (87.8, 69.0)
- added DS1: LED, misc:LED-0603, F.Cu at (116.2, 47.2)
- added R55: 100, chip_rlc:r_0402, F.Cu at (117.2, 49.8)
Connections:
- C36 pad 2: GND -> Net-(C36-Pad2)
- C37 pad 2: GND -> Net-(C36-Pad2)
- U14 pad 13: Net-(U14-Pad13) -> /MicroM4/Led_Status
Routing:
- net /MicroM4/Led_Status: track 0.00 -> 8.02 mm
- net /MicroM4/BOOT: track 34.2 -> 37.4 mm
- net Net-(C36-Pad2): track 0.00 -> 2.82 mm, vias 0 -> 1
- net Net-(DS1-Pad1): track 0.00 -> 2.60 mm
- net GND: track 178.7 -> 178.5 mm, vias 67 -> 66
